File: hv_signal_generator.sch (KiCad schematic (older format))
At the start: 23 parts, among them IC1 ATMEG328PU, J2 CONN_01X10, J3 BNC, P1 CONN_01X06, P2 CONN_01X06, SW1 Switch_DPST, X1 16MHz

Commit message: Complete layout
Parts:
- removed C2, C4: 33uF, symbol CP1
- removed C6: 0.1uF, symbol C
- removed C7: 0.01uF, symbol C
- removed DS2: VCC, symbol LED
- removed J3: BNC, symbol BNC
- removed R127: 1k, symbol R
- added C1: 10uF, Capacitors_Tantalum_SMD:TantalC_SizeD_EIA-7343_Reflow, symbol CP
- added C12, C5, C8: 0.1uF, Capacitors_SMD:C_1206, symbol C
- added C2: 0.1uF, Capacitors_SMD:C_1206, symbol CP
- added C4: 0.1uF, Capacitors_SMD:C_1812, symbol C_Small
- added C6: 100uF,35V, Capacitors_Tantalum_SMD:TantalC_SizeE_EIA-7360_Reflow, symbol CP
- added C7: 4u7,250V, Capacitors_SMD:c_elec_8x10.5, symbol CP
- added C9: 100nF,250V, Capacitors_SMD:C_1812, symbol C
- added D1: ES2F, Diodes_SMD:DO-214BA, symbol D
- added L1: 100uH, Inductors:self_cms_we-pd3, symbol INDUCTOR
- added LED1: +5V, LEDs:LED_0805, symbol LED
- added P4: VOUT, footprints:JACK_SMA, symbol BNC
- added P5: LIGHT, Pin_Headers:Pin_Header_Straight_1x02, symbol CONN_01X02
- added P6: MAGNET, Pin_Headers:Pin_Header_Straight_1x03, symbol CONN_01X03
- added Q1: IRF644PBF, TO_SOT_Packages_THT:TO-220_Neutral123_Vertical_LargePads, symbol IRF644PBF
- added Q2: P16NF06, TO_SOT_Packages_THT:TO-220_Neutral123_Vertical_LargePads, symbol Q_NMOS_GDS
- added R1: 1k, Resistors_SMD:R_1206, symbol R
- added R10: 4.75k, Resistors_SMD:R_1206, symbol R
- added R11, R12: 375, Resistors_SMD:R_1206, symbol R
- added R13: 5k, Resistors_SMD:R_1206, symbol R
- added R14: 5, Resistors_SMD:R_1206, symbol R
- added R15, R17: 50k, Resistors_SMD:R_1206, symbol R
- added R16: 100k, Resistors_SMD:R_1206, symbol R
- added R18: 10k, Resistors_ThroughHole:Resistor_Horizontal_RM25mm, symbol R
- added R3, R4: 5.1k, Resistors_SMD:R_1206, symbol R
- added R5: 50m, Resistors_SMD:R_2512, symbol R
- added R6, R8: 2M, Resistors_SMD:R_1206, symbol R
- added R7: 10k, Resistors_SMD:R_1206, symbol R
- added R9: 40k, Resistors_SMD:R_1206, symbol R
- added U1: HV513, footprints:SOW-24, symbol HV513
- added U2: MAX1771, Housings_SOIC:SOIC-8_3.9x4.9mm_Pitch1.27mm, symbol MAX1771
- added U3: MCP41050, Housings_SOIC:SOIC-8_3.9x4.9mm_Pitch1.27mm, symbol MCP41050
- added U4: HV7802, footprints:MSOP-8, symbol HV7802
- added U5: AQW216, SMD_Packages:DIP-8_SMD, symbol AQW216
- C10, C11, C13, C3: footprint (none) -> Capacitors_SMD:C_1206
- IC1: footprint (none) -> Housings_DIP:DIP-28_W7.62mm_LongPads
- J2: value CONN_01X10 -> COMM_BUS; footprint (none) -> Connect:he10-10d
- JP1: value JUMPER -> USB_PWR; footprint (none) -> Pin_Headers:Pin_Header_Straight_1x02
- LED2: renamed from DS1; value +5V -> +12V; footprint (none) -> LEDs:LED_0805
- P1: value CONN_01X06 -> FTDI_USB; footprint (none) -> Pin_Headers:Pin_Header_Angled_1x06
- P2: value CONN_01X06 -> ISP; footprint (none) -> Pin_Headers:Pin_Header_Straight_2x03
- P3: renamed from P?; value CONN_01X03 -> POWER; footprint (none) -> Connect:bornier3
- R19: renamed from R99; footprint (none) -> Resistors_SMD:R_1206
- R2: renamed from R45; value 1k -> 2k; footprint (none) -> Resistors_SMD:R_1206
- R20: renamed from R43; footprint (none) -> Resistors_SMD:R_1206
- SW1: value Switch_DPST -> RESET; footprint (none) -> footprints:SW_PUSH_6mm
- X1: footprint (none) -> footprints:SparkFun-HC49U-V
Connections:
- net labels added: +12V, A0/SHORT_CHK, A1/HV_FB, A3/OUTPUT_SELECT, D10/MCP41050_CS, D2/SERVO, D3/A2/CURRENT_SENSE, D4/SHDN, D5/LED, D6/BL, D7/HV513_CS, D8/S_SCK, D9/S_MOSI, VOUT
- net labels removed: D10/SS, D3/S_SS, D4/S_SCK, D5/S_MOSI, D7, HVGND, VCC
- wire segments 37 -> 95
- no-connect marks 10 -> 9
Other:
- note added: "BOOST CONVERTER"
- note added: "I2C PULLUPS"
- note added: "LIGHT"
- note added: "MAGNET"
- note added: "OUTPUT SELECT"
- note added: "SQUARE WAVE"

Commit message: Move C1 and C2 closer to MAX1771 chip and ...
Add layout notes
Other:
- note added: "BOOST CONVERTER\nBased on circuit by Nick de Smith http://desmith.net/NMdS/Electronics/NixiePSU.html"
- note added: "Q1 should be selected for low Qg, Rdson & Coss\nR6, R8, C7 and C9 must be rated at >240V\nD1 should be an ultra-fast (<50ns) recovery, 1A 240V)\nC1 & C6 should be a low ESR type (e.g., AVX TPS series)\nC1 & C2 should be sited very close to pin 2 (VCC) of U2\nC7 should be low ESR (<3ohms and rated >240V)\nIf you have stability issues, a 100pF 250 V ceramic cap\n could be soldered on top of R8\nL1 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"
- note removed: "BOOST CONVERTER"
Changed lines of the file:
@@
 	1    0    0    -1
 $EndComp
-Text Notes 4150 4350 0    60   ~ 0
-BOOST CONVERTER
+Text Notes 3500 4350 0    60   ~ 0
+BOOST CONVERTER\nBased on circuit by Nick de Smith http://desmith.net/NMdS/Electronics/NixiePSU.html
 $Comp
 L R R3
@@
 Wire Wire Line
 	3550 2450 3550 2550
+Text Notes 4050 7400 0    60   ~ 0
+Q1 should be selected for low Qg, Rdson & Coss\nR6, R8, C7 and C9 must be rated at >240V\nD1 should be an ultra-fast (<50ns) recovery, 1A 240V)\nC1 & C6 should be a low ESR type (e.g., AVX TPS series)\nC1 & C2 should be sited very close to pin 2 (VCC) of U2\nC7 should be low ESR (<3ohms and rated >240V)\nIf you have stability issues, a 100pF 250 V ceramic cap\n  could be soldered on top of R8\nL1 should be 2A rated (e.g., EPCOS B82479 series\n  for 50mA output\nR5 must be capable of handling at least 2A
 $EndSCHEMATC

Commit message: Add part numbers to schematic`
Parts:
- C1: Mfg_Part_No (none) -> T494D106M025AT
- C10, C11: Mfg_Part_No (none) -> CL31C220JCCNNNC
- C12, C13, C3, C8: Mfg_Part_No (none) -> C1206C104K5RACTU
- C4: Mfg_Part_No (none) -> GRM43DR72J104KW01L
- C6: Mfg_Part_No (none) -> TAJE107K020RNJ
- C7: value 4u7,250V -> 10uF,250V; Mfg_Part_No (none) -> EEV-EB2E100Q
- C9: Mfg_Part_No (none) -> ECW-U2104V16
- D1: Mfg_Part_No (none) -> ES2F-E3/52T
- IC1: Mfg_Part_No (none) -> ATMEGA328P-PU
- J2: Mfg_Part_No (none) -> XG4A-1034
- JP1: Mfg_Part_No (none) -> M20-9990246
- L1: Mfg_Part_No (none) -> B82479-A1-104M
- LED1, LED2: Mfg_Part_No (none) -> APL3015SGC-F01
- P1: Mfg_Part_No (none) -> PRPC006SBAN-M71RC
- P2: Mfg_Part_No (none) -> M20-9980346
- P3: Mfg_Part_No (none) -> OSTTC032162
- P4: Mfg_Part_No (none) -> 5-1814400-1
- P5: Mfg_Part_No (none) -> 0705430036
- P6: Mfg_Part_No (none) -> 0705430037
- Q1: Mfg_Part_No (none) -> IRF644PBF
- Q2: Mfg_Part_No (none) -> STP16NF06
- R1: Mfg_Part_No (none) -> RMCF1206FT1K00
- R10: Mfg_Part_No (none) -> RC1206FR-074K75L
- R11, R12: value 375 -> 374; Mfg_Part_No (none) -> RC1206FR-07374RL
- R13: value 5k -> 5.1k; Mfg_Part_No (none) -> RMCF1206JT5K10
- R14: value 5 -> 5.1; Mfg_Part_No (none) -> RC1206FR-075R1L
- R15, R17: value 50k -> 51k; Mfg_Part_No (none) -> RC1206FR-0751KL
- R16: Mfg_Part_No (none) -> RMCF1206FT100K
- R18: Mfg_Part_No (none) -> 55J10KE
- R19: Mfg_Part_No (none) -> RMCF1206FT1M00
- R2: Mfg_Part_No (none) -> RMCF1206FT2K00
- R20, R7: Mfg_Part_No (none) -> RMCF1206FT10K0
- R3, R4: Mfg_Part_No (none) -> RMCF1206JT5K10
- R5: Mfg_Part_No (none) -> ERJ-L1WKF50MU
- R6, R8: Mfg_Part_No (none) -> HVCB1206KDL2M00
- R9: value 40k -> 39k; Mfg_Part_No (none) -> RC1206FR-0739KL
- SW1: Mfg_Part_No (none) -> PTS645SK43 LFS
- U1: Mfg_Part_No (none) -> HV513WG-G
- U2: Mfg_Part_No (none) -> MAX1771ESA+
- U3: Mfg_Part_No (none) -> MCP41050-I/SN
- U4: Mfg_Part_No (none) -> HV7802MG-G
- U5: Mfg_Part_No (none) -> AQW216EHA
- X1: Mfg_Part_No (none) -> HC49US-16.000MABJ-UB

Commit message: [WIP] Remove HV513, fix orientation of FTDI header
* fix footprint of L1
Parts:
- removed C12: 0.1uF, Capacitors_SMD:C_1206, symbol C
- removed C4: 0.1uF, Capacitors_SMD:C_1812, symbol C_Small
- removed R18: 10k, Resistors_ThroughHole:Resistor_Horizontal_RM25mm, symbol R
- removed U1: HV513, footprints:SOW-24, symbol HV513
- C7: footprint Capacitors_SMD:c_elec_8x10.5 -> Capacitors_SMD:c_elec_10x10
- L1: footprint Inductors:self_cms_we-pd3 -> footprints:DU1971
Connections:
- wire segments 95 -> 86
- no-connect marks 9 -> 5
Other:
- note removed: "SQUARE WAVE"
Changed lines of the file:
@@
 	1    0    0    -1
 $EndComp
-Text GLabel 3600 6800 2    60   Input ~ 0
-VOUT
 Text GLabel 5050 1600 0    60   Input ~ 0
 GND
@@
 F 4 "PRPC006SBAN-M71RC" H 1150 3900 60  0001 C CNN "Mfg_Part_No"
 	1    1150 3900
-	-1   0    0    -1
+	-1   0    0    1
 $EndComp
 $Comp
@@
 F 0 "L1" V 5650 4500 50  0000 C CNN
 F 1 "100uH" V 5800 4500 50  0000 C CNN
-F 2 "Inductors:self_cms_we-pd3" H 5700 4500 60  0001 C CNN
+F 2 "footprints:DU1971" H 5700 4500 60  0001 C CNN
 F 3 "" H 5700 4500 60  0000 C CNN
 F 4 "B82479-A1-104M" H 5700 4500 60  0001 C CNN "Mfg_Part_No"
@@
 F 0 "C7" H 6675 5500 50  0000 L CNN
 F 1 "10uF,250V" H 6675 5300 50  0000 C TNN
-F 2 "Capacitors_SMD:c_elec_8x10.5" H 6688 5250 30  0001 C CNN
+F 2 "Capacitors_SMD:c_elec_10x10" H 6688 5250 30  0001 C CNN
 F 3 "" H 6650 5400 60  0000 C CNN
 F 4 "EEV-EB2E100Q" H 6650 5400 60  0001 C CNN "Mfg_Part_No"
@@
 D4/SHDN
 $Comp
-L HV513 U1
-U 1 1 56C01A7B
-P 2150 6750
-F 0 "U1" H 2150 6900 60  0000 C CNN
-F 1 "HV513" H 2150 6700 60  0000 C CNN
-F 2 "footprints:SOW-24" H 2900 6600 60  0001 C CNN
-F 3 "" H 2900 6600 60  0000 C CNN
-F 4 "HV513WG-G" H 2150 6750 60  0001 C CNN "Mfg_Part_No"
-	1    2150 6750
-	1    0    0    -1
-$EndComp
-$Comp
 L BNC P4
 U 1 1 56C01A7F
@@
 	1    0    0    -1
 $EndComp
-Text GLabel 2850 6200 2    60   Input ~ 0
-HV
-Text GLabel 1500 6300 0    60   Input ~ 0
-+5V
-Text GLabel 1500 7200 0    60   Input ~ 0
-GND
-$Comp
-L R R18
-U 1 1 56C01A83
-P 3300 7050
-F 0 "R18" V 3380 7050 50  0000 C CNN
-F 1 "10k" V 3300 7050 50  0000 C CNN
-F 2 "Resistors_ThroughHole:Resistor_Horizontal_RM25mm" V 3230 7050 30  0001 C CNN
-F 3 "" H 3300 7050 30  0000 C CNN
-F 4 "55J10KE" H 3300 7050 60  0001 C CNN "Mfg_Part_No"
-	1    3300 7050
-	-1   0    0    1
-$EndComp
-$Comp
-L C_Small C4
-U 1 1 56C01A85
-P 3050 6800
-F 0 "C4" V 2950 6800 50  0000 L CNN
-F 1 "0.1uF" V 3150 6700 50  0000 L CNN
-F 2 "Capacitors_SMD:C_1812" H 3050 6800 60  0001 C CNN
-F 3 "" H 3050 6800 60  0000 C CNN
-F 4 "GRM43DR72J104KW01L" H 3050 6800 60  0001 C CNN "Mfg_Part_No"
-	1    3050 6800
-	0    1    1    0
-$EndComp
-Text GLabel 1500 7100 0    60   Input ~ 0
-D9/S_MOSI
 Text GLabel 6950 1400 2    60   Input ~ 0
 D10/MCP41050_CS
@@
 Text GLabel 4650 5300 0    60   Input ~ 0
 D4/SHDN
-Text GLabel 3600 7250 2    60   Input ~ 0
-GND
-NoConn ~ 1500 6400
-Text GLabel 1500 6700 0    60   Input ~ 0
-D8/S_SCK
 Text GLabel 6950 3300 2    60   Input ~ 0
-D7/HV513_CS
-Text GLabel 1500 6800 0    60   Input ~ 0
 D7/HV513_CS
 Text GLabel 6950 2900 2    60   Input ~ 0
@@
 Text GLabel 6950 2000 2    60   Input ~ 0
 A1/HV_FB
-NoConn ~ 1500 6600
-NoConn ~ 1500 7000
-Text GLabel 1500 6500 0    60   Input ~ 0
-D6/BL
 Text GLabel 8050 5800 2    60   Input ~ 0
 D10/MCP41050_CS
@@
 Text GLabel 10350 2650 2    60   Input ~ 0
 GND
-Text Notes 1700 6050 0    60   ~ 0
-SQUARE WAVE
 Text Notes 8550 1600 0    60   ~ 0
 OUTPUT SELECT
@@
 Text GLabel 4650 3850 2    60   Input ~ 0
 A5/SCL
-NoConn ~ 1500 6900
 $Comp
 L CONN_01X02 P5
@@
 Wire Wire Line
 	7050 5350 7050 5600
-Wire Wire Line
-	2850 6200 2850 6300
-Wire Wire Line
-	3150 6800 3600 6800
-Connection ~ 3300 6800
-Wire Wire Line
-	2850 6400 2850 7100
-Connection ~ 2850 6600
-Connection ~ 2850 6700
-Connection ~ 2850 6800
-Connection ~ 2850 6900
-Connection ~ 2850 7000
-Connection ~ 2850 7100
-Connection ~ 2850 6400
-Connection ~ 2850 6500
-Wire Wire Line
-	2950 6800 2850 6800
-Wire Wire Line
-	2850 7200 2850 7300
-Wire Wire Line
-	2850 7250 3600 7250
-Connection ~ 2850 7250
-Connection ~ 3300 7250
 Connection ~ 9050 6250
 Connection ~ 9050 4800
@@
 Wire Wire Line
 	8750 2300 8750 2400
-Wire Wire Line
-	3300 6900 3300 6800
-Wire Wire Line
-	3300 7200 3300 7250
 Wire Wire Line
 	3800 6250 10250 6250
@@
 Wire Wire Line
 	5200 4900 5200 4800
-$Comp
-L C C12
-U 1 1 56C4B14D
-P 1500 5950
-F 0 "C12" V 1450 6000 50  0000 L CNN
-F 1 "0.1uF" V 1350 5900 50  0000 L CNN
-F 2 "Capacitors_SMD:C_1206" H 1500 5950 60  0001 C CNN
-F 3 "" H 1500 5950 60  0001 C CNN
-F 4 "C1206C104K5RACTU" H 1500 5950 60  0001 C CNN "Mfg_Part_No"
-	1    1500 5950
-	-1   0    0    1
-$EndComp
-Wire Wire Line
-	1500 6300 1500 6100
-Text GLabel 1500 5800 0    60   Input ~ 0
-GND
 Connection ~ 4650 3500
 NoConn ~ 1350 4050

Commit message: [WIP] Add hv signal generator breakout headers
Parts:
- added P7: CONN_01X05, Pin_Headers:Pin_Header_Straight_1x05, symbol CONN_01X05
- added P8: CONN_01X03, Pin_Headers:Pin_Header_Straight_1x03, symbol CONN_01X03
Connections:
- net labels added: D6, D7
- net labels removed: D6/BL, D7/HV513_CS
Other:
- note added: "Breakout board switches HV\nto produce an AC signal (VOUT)"
- note added: "HV SIGNAL GENERATOR HEADERS"
Changed lines of the file:
@@
 D4/SHDN
 Text GLabel 6950 3300 2    60   Input ~ 0
-D7/HV513_CS
+D7
 Text GLabel 6950 2900 2    60   Input ~ 0
 D3/A2/CURRENT_SENSE
@@
 D10/MCP41050_CS
 Text GLabel 6950 3200 2    60   Input ~ 0
-D6/BL
+D6
 Text GLabel 6950 3100 2    60   Input ~ 0
 D5/LED
@@
 Text Notes 4050 7400 0    60   ~ 0
 Q1 should be selected for low Qg, Rdson & Coss\nR6, R8, C7 and C9 must be rated at >240V\nD1 should be an ultra-fast (<50ns) recovery, 1A 240V)\nC1 & C6 should be a low ESR type (e.g., AVX TPS series)\nC1 & C2 should be sited very close to pin 2 (VCC) of U2\nC7 should be low ESR (<3ohms and rated >240V)\nIf you have stability issues, a 100pF 250 V ceramic cap\n  could be soldered on top of R8\nL1 should be 2A rated (e.g., EPCOS B82479 series\n  for 50mA output\nR5 must be capable of handling at least 2A
+$Comp
+L CONN_01X05 P7
+U 1 1 5710F690
+P 1250 6250
+F 0 "P7" H 1250 6550 50  0000 C CNN
+F 1 "CONN_01X05" V 1350 6250 50  0000 C CNN
+F 2 "Pin_Headers:Pin_Header_Straight_1x05" H 1250 6250 60  0001 C CNN
+F 3 "" H 1250 6250 60  0000 C CNN
+	1    1250 6250
+	-1   0    0    -1
+$EndComp
+$Comp
+L CONN_01X03 P8
+U 1 1 5710F76D
+P 1250 6850
+F 0 "P8" H 1250 7050 50  0000 C CNN
+F 1 "CONN_01X03" V 1350 6850 50  0000 C CNN
+F 2 "Pin_Headers:Pin_Header_Straight_1x03" H 1250 6850 60  0001 C CNN
+F 3 "" H 1250 6850 60  0000 C CNN
+	1    1250 6850
+	-1   0    0    -1
+$EndComp
+Text GLabel 1450 6950 2    60   Input ~ 0
+HV
+Text GLabel 1450 6750 2    60   Input ~ 0
+GND
+Text GLabel 1450 6850 2    60   Input ~ 0
+VOUT
+Text GLabel 1450 6350 2    60   Input ~ 0
+D7
+Text GLabel 1450 6250 2    60   Input ~ 0
+D6
+Text GLabel 1450 6050 2    60   Input ~ 0
++12V
+Text GLabel 1450 6150 2    60   Input ~ 0
+GND
+Text GLabel 1450 6450 2    60   Input ~ 0
++5V
+Text Notes 1150 5850 0    60   ~ 0
+HV SIGNAL GENERATOR HEADERS
+Text Notes 1800 6350 0    60   ~ 0
+Breakout board switches HV\nto produce an AC signal (VOUT)
 $EndSCHEMATC

Commit message: Swap parts to support up to 400V and use BJT for LED
Parts:
- removed Q2: P16NF06, TO_SOT_Packages_THT:TO-220_Neutral123_Vertical_LargePads, symbol Q_NMOS_GDS
- added Q2: TIP120, TO_SOT_Packages_THT:TO-220_Neutral123_Vertical_LargePads, symbol Q_NPN_BCE
- added R18: 1k, Resistors_SMD:R_1206, symbol R
- C7: value 10uF,250V -> 3.3uF,400V
- C9: value 100nF,250V -> 100nF,400V; footprint Capacitors_SMD:C_1812 -> Capacitors_SMD:C_2225
- R6, R8: value 2M -> 1M
- R7: value 10k -> 4k
- R9: value 39k -> 20k
Changed lines of the file:
@@
 P 6650 5400
 F 0 "C7" H 6675 5500 50  0000 L CNN
-F 1 "10uF,250V" H 6675 5300 50  0000 C TNN
+F 1 "3.3uF,400V" H 6675 5300 50  0000 C TNN
 F 2 "Capacitors_SMD:c_elec_10x10" H 6688 5250 30  0001 C CNN
 F 3 "" H 6650 5400 60  0000 C CNN
@@
 P 7050 6050
 F 0 "R7" V 7130 6050 50  0000 C CNN
-F 1 "10k" V 7050 6050 50  0000 C CNN
+F 1 "4k" V 7050 6050 50  0000 C CNN
 F 2 "Resistors_SMD:R_1206" V 6980 6050 30  0001 C CNN
 F 3 "" H 7050 6050 30  0000 C CNN
@@
 P 7050 5200
 F 0 "R6" V 7130 5200 50  0000 C CNN
-F 1 "2M" V 7050 5200 50  0000 C CNN
+F 1 "1M" V 7050 5200 50  0000 C CNN
 F 2 "Resistors_SMD:R_1206" V 6980 5200 30  0001 C CNN
 F 3 "" H 7050 5200 30  0000 C CNN
@@
 P 9250 5500
 F 0 "C9" H 9275 5600 50  0000 L CNN
-F 1 "100nF,250V" H 9275 5400 50  0000 L CNN
-F 2 "Capacitors_SMD:C_1812" H 9288 5350 30  0001 C CNN
+F 1 "100nF,400V" H 9275 5400 50  0000 L CNN
+F 2 "Capacitors_SMD:C_2225" H 9288 5350 30  0001 C CNN
 F 3 "" H 9250 5500 60  0000 C CNN
 F 4 "ECW-U2104V16 " H 9250 5500 60  0001 C CNN "Mfg_Part_No"
@@
 P 9050 5100
 F 0 "R8" V 9130 5100 50  0000 C CNN
-F 1 "2M" V 9050 5100 50  0000 C CNN
+F 1 "1M" V 9050 5100 50  0000 C CNN
 F 2 "Resistors_SMD:R_1206" V 8980 5100 30  0001 C CNN
 F 3 "" H 9050 5100 30  0000 C CNN
@@
 P 9050 6100
 F 0 "R9" V 9130 6100 50  0000 C CNN
-F 1 "39k" V 9050 6100 50  0000 C CNN
+F 1 "20k" V 9050 6100 50  0000 C CNN
 F 2 "Resistors_SMD:R_1206" V 8980 6100 30  0001 C CNN
 F 3 "" H 9050 6100 30  0000 C CNN
@@
 Text GLabel 3350 2350 2    60   Input ~ 0
 +12V
-Text GLabel 3250 2750 0    60   Input ~ 0
+Text GLabel 2950 2750 0    60   Input ~ 0
 D5/LED
 Text GLabel 3550 2950 3    60   Input ~ 0
@@
 Wire Wire Line
 	1550 1700 2150 1700
-$Comp
-L Q_NMOS_GDS Q2
-U 1 1 56C3FB51
-P 3450 2750
-F 0 "Q2" H 3750 2800 50  0000 R CNN
-F 1 "P16NF06" H 3650 2700 50  0000 L CNN
-F 2 "TO_SOT_Packages_THT:TO-220_Neutral123_Vertical_LargePads" H 3650 2850 50  0001 C CNN
-F 3 "" H 3450 2750 50  0000 C CNN
-F 4 "STP16NF06" H 3450 2750 60  0001 C CNN "Mfg_Part_No"
-	1    3450 2750
-	1    0    0    -1
-$EndComp
 Wire Wire Line
 	3550 2450 3550 2550
@@
 Text Notes 1800 6350 0    60   ~ 0
 Breakout board switches HV\nto produce an AC signal (VOUT)
+$Comp
+L Q_NPN_BCE Q2
+U 1 1 57112CE3
+P 3450 2750
+F 0 "Q2" H 3750 2800 50  0000 R CNN
+F 1 "TIP120" H 3900 2700 50  0000 R CNN
+F 2 "TO_SOT_Packages_THT:TO-220_Neutral123_Vertical_LargePads" H 3650 2850 50  0001 C CNN
+F 3 "" H 3450 2750 50  0000 C CNN
+	1    3450 2750
+	1    0    0    -1
+$EndComp
+$Comp
+L R R18
+U 1 1 57113011
+P 3100 2750
+F 0 "R18" V 3180 2750 50  0000 C CNN
+F 1 "1k" V 3100 2750 50  0000 C CNN
+F 2 "Resistors_SMD:R_1206" V 3030 2750 50  0001 C CNN
+F 3 "" H 3100 2750 50  0000 C CNN
+	1    3100 2750
+	0    1    1    0
+$EndComp
 $EndSCHEMATC

Commit message: Swap ATMEGA328 for Teensy
Parts:
- removed C10, C11: 22pF, Capacitors_SMD:C_1206, symbol C
- removed C13, C3: 0.1uF, Capacitors_SMD:C_1206, symbol C
- removed IC1: ATMEG328PU, Housings_DIP:DIP-28_W7.62mm_LongPads, symbol ATMEGA8-P
- removed JP1: USB_PWR, Pin_Headers:Pin_Header_Straight_1x02, symbol JUMPER
- removed P1: FTDI_USB, Pin_Headers:Pin_Header_Angled_1x06, symbol CONN_01X06
- removed P2: ISP, Pin_Headers:Pin_Header_Straight_2x03, symbol CONN_01X06
- removed SW1: RESET, footprints:SW_PUSH_6mm, symbol Switch_DPST
- removed X1: 16MHz, footprints:SparkFun-HC49U-V, symbol Crystal
- added Q3, Q4: 2N7002, TO_SOT_Packages_THT:TO-92_Inline_Narrow_Oval, symbol 2N7002
- added U1: Teensy_3.1, footprints:Teensy-3.1, symbol Teensy_3.1
- R11, R12: value 374 -> 200
- R19: value 1Meg -> 5.1k; Mfg_Part_No RMCF1206FT1M00 -> RMCF1206JT5K10
- R20: value 10k -> 5.1k; Mfg_Part_No RMCF1206FT10K0 -> RMCF1206JT5K10
Connections:
- net labels added: +3.3V, A2/CURRENT_SENSE, D3/OUTPUT_SELECT, D6/DRIVER_HI, D7/DRIVER_LO, SCL_3.3V, SCL_5V, SDA_3.3V, SDA_5V
- net labels removed: +5V_USB, A4/SDA, A5/SCL, D3/A2/CURRENT_SENSE, D6, D7, D8/S_SCK, D9/S_MOSI, RST, RX, TX
- wire segments 86 -> 76
- no-connect marks 5 -> 21
Other:
- note added: "I2C LEVEL SHIFTING"
- note removed: "ARDUINO PROGRAMMING INTERFACE"
- note removed: "I2C PULLUPS"
- note removed: "ISP"
- note removed: "POWER JUMPERS"

Commit message: Replace footprint for transistors with SOT-23
Parts:
- Q3, Q4: footprint TO_SOT_Packages_THT:TO-92_Inline_Narrow_Oval -> TO_SOT_Packages_SMD:SOT-23
Changed lines of the file:
@@
 F 0 "Q3" H 3300 1001 40  0000 R CNN
 F 1 "2N7002" H 3300 1300 40  0000 R CNN
-F 2 "TO_SOT_Packages_THT:TO-92_Inline_Narrow_Oval" H 3170 1252 29  0000 C CNN
+F 2 "TO_SOT_Packages_SMD:SOT-23" H 3170 1252 29  0000 C CNN
 F 3 "" H 3300 1150 60  0000 C CNN
 	1    3300 1150
@@
 F 0 "Q4" H 3650 1401 40  0000 R CNN
 F 1 "2N7002" H 3650 1700 40  0000 R CNN
-F 2 "TO_SOT_Packages_THT:TO-92_Inline_Narrow_Oval" H 3520 1652 29  0000 C CNN
+F 2 "TO_SOT_Packages_SMD:SOT-23" H 3520 1652 29  0000 C CNN
 F 3 "" H 3650 1550 60  0000 C CNN
 	1    3650 1550
