File: dropbot_control_board.sch (KiCad schematic (older format))
At the start: 47 parts, among them J2 COMM_BUS, P3 POWER, P4 VOUT, P5 LIGHT, P6 MAGNET, P7 CONN_01X05, P8 CONN_01X03, Q1 IRF644PBF, Q2 TIP120, Q3 2N7002, Q4 2N7002, U1 Teensy_3.1, U2 MAX1771, U3 MCP41050, U4 HV7802, U5 AQW216

Commit message: Fix routing of D3/OUTPUT_SELECT and add MAX1771...
Fix routing of D3/OUTPUT_SELECT and add MAX1771 current sensing.
Connections:
- net labels added: A2/HV507_CS, A3/MAX1771_CS
- net labels removed: A2/CURRENT_SENSE, A3/OUTPUT_SELECT
- no-connect marks 21 -> 20
Changed lines of the file:
@@
 Text GLabel 10400 1250 2    60   Input ~ 0
 VOUT
-Text GLabel 5550 1400 0    60   Input ~ 0
+Text GLabel 5600 1400 0    60   Input ~ 0
 D3/OUTPUT_SELECT
 Text GLabel 9350 800  2    60   Input ~ 0
-A3/OUTPUT_SELECT
+D3/OUTPUT_SELECT
 $Comp
 L HV7802 U4
@@
 NoConn ~ 1350 3050
 Text GLabel 10900 6350 0    60   Input ~ 0
-A2/CURRENT_SENSE
-Text GLabel 7600 2300 2    60   Input ~ 0
-A2/CURRENT_SENSE
+A2/HV507_CS
 Text GLabel 10400 1850 2    60   Input ~ 0
 A0/SHORT_CHK
@@
 NoConn ~ 6800 3300
 NoConn ~ 6950 3300
-NoConn ~ 7600 2150
 NoConn ~ 7600 1700
 NoConn ~ 7600 1550
@@
 NoConn ~ 7600 950
 NoConn ~ 7600 800
+Text GLabel 6500 5750 2    60   Input ~ 0
+A3/MAX1771_CS
+Text GLabel 7600 2300 2    60   Input ~ 0
+A2/HV507_CS
+Text GLabel 7600 2150 2    60   Input ~ 0
+A3/MAX1771_CS
 $EndSCHEMATC

Commit message: Connect 5V pin on COMM_BUS
Connections:
- no-connect marks 20 -> 19
Changed lines of the file:
@@
 NoConn ~ 1350 2850
 NoConn ~ 1350 2950
-NoConn ~ 1350 2250
 $Comp
 L 2N7002 Q3
@@
 Text GLabel 7600 2150 2    60   Input ~ 0
 A3/MAX1771_CS
+Text GLabel 1350 2250 2    60   Input ~ 0
++5V
 $EndSCHEMATC

Commit message: [WIP] Integrate HV square-wave driver (not routed)
Parts:
- added C10: C, Capacitors_SMD:C_1210, symbol C
- added C3: 0.1uF, Capacitors_SMD:C_1206, symbol C_Small
- added C4: 0.1uF, Capacitors_SMD:C_1210, symbol C_Small
- added D2, D3: D, Diodes_SMD:SMA_Standard, symbol D
- added F1: FUSE, Resistors_ThroughHole:Resistor_Vertical_RM5mm, symbol FUSE
- added Q5, Q6: Q_NMOS_GDS, TO_SOT_Packages_THT:TO-220_Neutral123_Vertical, symbol Q_NMOS_GDS
- added R21: 10, Resistors_SMD:R_1206, symbol R
- added R22: R, Resistors_SMD:R_1206, symbol R
- added U6: NCP5304, SMD_Packages:SOIC-8-N, symbol NCP5304
Connections:
- wire segments 76 -> 99
Other:
- note added: "HV SQUARE WAVE DRIVER"
- note removed: "Breakout board switches HV\nto produce an AC signal (VOUT)"
- note removed: "HV SIGNAL GENERATOR HEADERS"

Commit message: [WIP] Add feedback circuit and on-board calibration
Parts:
- removed P7: CONN_01X05, Pin_Headers:Pin_Header_Straight_1x05, symbol CONN_01X05
- removed U1: Teensy_3.1, footprints:Teensy-3.1, symbol Teensy_3.1
- added C11: 1uF, Capacitors_SMD:C_1206, symbol C
- added C12: 1pF, Capacitors_SMD:C_1206, symbol C
- added C13, C15, C17: 0.1uF, Capacitors_SMD:C_1206, symbol C
- added C14: 10pF, Capacitors_SMD:C_1206, symbol C
- added C16: 100pF, Capacitors_SMD:C_1206, symbol C
- added C18, C20, C22: 1nF, Capacitors_SMD:C_1206, symbol C
- added C19: 4.7nF, Capacitors_SMD:C_1206, symbol C
- added C21: 0.15uF, Capacitors_SMD:C_1206, symbol C
- added IC1: MCP6024, SMD_Packages:SOIC-14_N, symbol MCP6024
- added P1: FEEDBACK, footprints:JACK_SMA, symbol BNC
- added P7: CONN_01X04, symbol CONN_01X04
- added R23, R27: 1Meg, Resistors_SMD:R_1206, symbol R
- added R24, R28, R29, R30: 200, Resistors_SMD:R_1206, symbol R
- added R25: 10k, Resistors_SMD:R_1206, symbol R
- added R26: 2.2k, Resistors_SMD:R_1206, symbol R
- added R31: 1.91k, Resistors_SMD:R_1206, symbol R
- added R32: 16.9k, Resistors_SMD:R_1206, symbol R
- added R33: 806, Resistors_SMD:R_1206, symbol R
- added R34: 13.3k, Resistors_SMD:R_1206, symbol R
- added U1: Teensy_3.2, footprints:Teensy_3.2, symbol Teensy_3.2
- added U7, U8: AQW216, SMD_Packages:DIP-8_SMD, symbol AQW216
Connections:
- net labels added: +0.6V, A1, A11, CUR_SENSE, D0, D1, D2, D3, D8/OUTPUT_SELECT, D9/SERVO
- net labels removed: D2/SERVO, D3/OUTPUT_SELECT
- wire segments 99 -> 149
- no-connect marks 19 -> 16
Other:
- note added: "4th-order Chebychev\nLow-pass filter\nfc=11kHz"
- note added: "BOOST CONVERTER\nBased on circuit by Nick de Smith\nhttp://desmith.net/NMdS/Electronics/NixiePSU.html"
- note added: "CURRENT-TO-VOLTAGE\nCONVERTER"
- note added: "FEEDBACK"
- note added: "HV DRIVER BREAKOUTS"
- note added: "ON-BOARD CALIBRATION"
- note removed: "BOOST CONVERTER\nBased on circuit by Nick de Smith http://desmith.net/NMdS/Electronics/NixiePSU.html"

Commit message: Re-do layout
Parts:
- C11, C12, C19, C2, C20, C21, C22, C3, C5, C8: footprint Capacitors_SMD:C_1206 -> Capacitors_SMD:C_0805
- C13: renamed from C14; footprint Capacitors_SMD:C_1206 -> Capacitors_SMD:C_0805
- C14: renamed from C16; footprint Capacitors_SMD:C_1206 -> Capacitors_SMD:C_0805
- C15: renamed from C18; footprint Capacitors_SMD:C_1206 -> Capacitors_SMD:C_0805
- C16: renamed from C13; footprint Capacitors_SMD:C_1206 -> Capacitors_SMD:C_0805
- C17: renamed from C15; footprint Capacitors_SMD:C_1206 -> Capacitors_SMD:C_0805
- C18: renamed from C17; footprint Capacitors_SMD:C_1206 -> Capacitors_SMD:C_0805
- P7: footprint (none) -> Pin_Headers:Pin_Header_Straight_1x04
- Q1, Q2: footprint TO_SOT_Packages_THT:TO-220_Neutral123_Vertical_LargePads -> TO_SOT_Packages_THT:TO-220_Neutral123_Horizontal_LargePads
- Q5, Q6: footprint TO_SOT_Packages_THT:TO-220_Neutral123_Vertical -> TO_SOT_Packages_THT:TO-220_Neutral123_Horizontal_LargePads
- R1, R10, R11, R12, R13, R14, R15, R16, R17, R18, R19, R2, R20, R21, R22, R23, R24, R25, R26, R27, R28, R29, R3, R30, R31, R32, R33, R34, R4, R7, R9: footprint Resistors_SMD:R_1206 -> Resistors_SMD:R_0805
- U1: footprint footprints:Teensy_3.2 -> footprints:Teensy-3.2
Connections:
- net labels added: HVAC
- net labels removed: A1
- wire segments 149 -> 150
Other:
- note added: "4th-order low-pass\nanti-aliasing filter"
- note added: "C12-15 should be\nrated for >100V"
- note removed: "4th-order Chebychev\nLow-pass filter\nfc=11kHz"

Commit message: Minor fixes
* fix inductor footprint
* footprints for various HV resistors
* labels for some resistors/caps
* remove shorted +12V trace
Parts:
- removed C10: C, Capacitors_SMD:C_1210, symbol C
- removed C9: 100nF,400V, Capacitors_SMD:C_2225, symbol C
- added C10: 100n,500V, Capacitors_SMD:C_1210, symbol C_Small
- C11: Mfg_Part_No (none) -> CC0805KKX7R9BB105
- C12: Mfg_Part_No (none) -> CBR08C109CAGAC
- C13: Mfg_Part_No (none) -> CL21C100JECNNWC
- C14: Mfg_Part_No (none) -> CL21C101JECNNWC
- C15: Mfg_Part_No (none) -> C2012C0G2E102J085AA
- C16, C17, C18, C3, C5: Mfg_Part_No (none) -> CL21B104KBCNNNC
- C19: value 4.7nF -> 0.015uF; Mfg_Part_No (none) -> CGA4F1C0G2A153J085AC
- C20, C22: value 1nF -> 100pF; Mfg_Part_No (none) -> CL21C101JECNNWC
- C21: value 0.15uF -> 470pF; Mfg_Part_No (none) -> CL21C471JBANNNC
- C4: value 0.1uF -> 100n,500V; Mfg_Part_No (none) -> C1210C104KCRACTU
- C8: Mfg_Part_No C1206C104K5RACTU -> CL21B104KBCNNNC
- D1: value ES2F -> ES3J; footprint Diodes_SMD:DO-214BA -> Diodes_SMD:SMC_Standard; Mfg_Part_No ES2F-E3/52T -> ES3J
- D2, D3: Mfg_Part_No (none) -> US1J-13-F
- F1: Mfg_Part_No (none) -> B59773B120A70
- IC1: Mfg_Part_No (none) -> MCP6024T-I/SL
- J2: footprint Connect:he10-10d -> Connect:HE10-10C
- L1: value 100uH -> 47uH,3.8A; footprint footprints:DU1971 -> footprints:SRR1210; Mfg_Part_No B82479-A1-104M -> SRR1210-470M
- LED1, LED2: Mfg_Part_No APL3015SGC-F01 -> 150080BS75000
- P1: Mfg_Part_No (none) -> 5-1814400-1
- P3: Mfg_Part_No OSTTC032162 -> OSTTA034163
- Q1: value IRF644PBF -> STP33N65M2; Mfg_Part_No IRF644PBF -> STP33N65M2
- Q2: Mfg_Part_No (none) -> TIP120G
- Q3, Q4: Mfg_Part_No (none) -> T2N7002AK,LM
- Q5, Q6: value Q_NMOS_GDS -> IRF740BPBF; Mfg_Part_No (none) -> IRF740BPBF
- R1: Mfg_Part_No RMCF1206FT1K00 -> RC0805FR-071KL
- R10: Mfg_Part_No RC1206FR-074K75L -> RC0805FR-074K75L
- R11, R12: Mfg_Part_No RC1206FR-07374RL -> RC0805FR-07200RL
- R13, R19, R20, R3, R4: Mfg_Part_No RMCF1206JT5K10 -> RC0805FR-075K1L
- R14: Mfg_Part_No RC1206FR-075R1L -> MCR10ERTFL5R10
- R15, R17: Mfg_Part_No RC1206FR-0751KL -> RC0805FR-0751KL
- R16: Mfg_Part_No RMCF1206FT100K -> RC0805FR-07100KL
- R18: Mfg_Part_No (none) -> RC0805FR-071KL
- R2: Mfg_Part_No RMCF1206FT2K00 -> RC0805FR-072KL
- R21: Mfg_Part_No (none) -> RC0805FR-0710RL
- R22: value R -> 2M; footprint Resistors_SMD:R_0805 -> Resistors_SMD:R_1206; Mfg_Part_No (none) -> HVCB1206KDL2M00
- R23: Mfg_Part_No RC1206FR-072K2L -> RC0805FR-071ML
- R24, R28, R29, R30: Mfg_Part_No (none) -> RC0805FR-07200RL
- R25: Mfg_Part_No (none) -> RC0805FR-0710KL
- R26: Mfg_Part_No RC1206FR-072K2L -> RC0805FR-072K2L
- R27: Mfg_Part_No RC1206FR-07200RL -> RC0805FR-071ML
- R31: value 1.91k -> 18.7k; Mfg_Part_No (none) -> RC0805FR-0718K7L
- R32: value 16.9k -> 2.1k; Mfg_Part_No (none) -> RC0805FR-072K1L
- R33: value 806 -> 14.7k; Mfg_Part_No (none) -> RC0805FR-0714K7L
- R34: value 13.3k -> 887; Mfg_Part_No (none) -> RC0805FR-07887RL
- R5: value 50m -> 30m; Mfg_Part_No ERJ-L1WKF50MU -> CSR2512C0R03F
- R6, R8: value 1M -> 2M
- R7: value 4k -> 2k; Mfg_Part_No RMCF1206FT10K0 -> RC0805FR-072KL
- R9: Mfg_Part_No RC1206FR-0739KL -> RC0805FR-0720KL
- U5: value AQW216 -> DPST (2 Form A), 350V; Mfg_Part_No AQW216EHA -> TLP227G-2(TP1,N,F)
- U6: Mfg_Part_No (none) -> NCP5304DR2G
- U7, U8: value AQW216 -> DPST (2 Form A), 350V; Mfg_Part_No (none) -> TLP227G-2(TP1,N,F)
Connections:
- wire segments 150 -> 148
Other:
- note added: "Q1 should be selected for low Qg, Rdson & Coss\nR6, R8, and C7 must be rated at >400V\nD1 should be an ultra-fast (<50ns) recovery, 3A, 400V\nC1 & C6 should be a low ESR type (e.g., AVX TPS series)\nC1 & C2 should be sited very close to pin 2 (VCC) of U2\nC7 should be low ESR (<3ohms and rated >400V)\nIf you have stability issues, a 100pF 400 V ceramic cap\n could be soldered on top of R8\nL1 sho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"
- note removed: "Q1 should be selected for low Qg, Rdson & Coss\nR6, R8, C7 and C9 must be rated at >240V\nD1 should be an ultra-fast (<50ns) recovery, 1A 240V)\nC1 & C6 should be a low ESR type (e.g., AVX TPS series)\nC1 & C2 should be sited very close to pin 2 (VCC) of U2\nC7 should be low ESR (<3ohms and rated >240V)\nIf you have stability issues, a 100pF 250 V ceramic cap\n could be soldered on top of R8\nL1 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"

Commit message: Use edge connectors and ...
* Add SPI flash memory
* Add HV output enable
* Make feedback circuit breakout and use DIP op-amp
* Pass Teensy's USB signals through edge connector
Parts:
- removed J2: COMM_BUS, Connect:HE10-10C, symbol CONN_01X10
- removed P1: FEEDBACK, footprints:JACK_SMA, symbol BNC
- removed P3: POWER, Connect:bornier3, symbol CONN_01X03
- removed P4: VOUT, footprints:JACK_SMA, symbol BNC
- removed P5: LIGHT, Pin_Headers:Pin_Header_Straight_1x02, symbol CONN_01X02
- removed P6: MAGNET, Pin_Headers:Pin_Header_Straight_1x03, symbol CONN_01X03
- removed Q2: TIP120, TO_SOT_Packages_THT:TO-220_Neutral123_Horizontal_LargePads, symbol Q_NPN_BCE
- removed Q3, Q4: 2N7002, TO_SOT_Packages_SMD:SOT-23, symbol 2N7002
- removed U3: MCP41050, Housings_SOIC:SOIC-8_3.9x4.9mm_Pitch1.27mm, symbol MCP41050
- added C9: 0.1uF, Capacitors_SMD:C_0805, symbol C
- added LED2: +5V, LEDs:LED_0805, symbol LED
- added P1: CONN_02X10, WheelerLab:HSEC8-110-XX-X-RA-MATE, symbol CONN_02X10
- added P2, P3, P4: CONN_01X04, Pin_Headers:Pin_Header_Straight_1x04, symbol CONN_01X04
- added R35: 5.1k, Resistors_SMD:R_0805, symbol R
- added R36: 4.75k, Resistors_SMD:R_0805, symbol R
- added U10: W25Q64FV, SMD_Packages:SOIC-8-N, symbol W25Q64FV
- added U3: CAT5171, WheelerLab:SOT-23-8, symbol CAT5171
- added U9: 74AHC1G32, TO_SOT_Packages_SMD:SOT-353, symbol 74AHC1G32
- IC1: footprint SMD_Packages:SOIC-14_N -> Housings_DIP:DIP-14_W7.62mm
- LED1: value +5V -> +3.3V
- R18: Mfg_Part_No RC0805FR-071KL -> RC0805FR-072KL
- R19, R20, R3, R4: Mfg_Part_No RC0805FR-075K1L -> RC0805FR-071KL
- renumbered LED2 to LED3
Connections:
- net labels added: A6, A7, D+, D-, D10/SHDN, D11/DI, D12/DO, D13/CLK, D4/SSDA, D5/SSCL, D6/DRIVER_LO, D7/DRIVER_HI, D9/CS, HV_OE, SCL, SDA
- net labels removed: D10/MCP41050_CS, D11/MOSI, D12/MISO, D13/SCK, D4/SHDN, D5/LED, D6/DRIVER_HI, D7/DRIVER_LO, D9/SERVO, SCL_3.3V, SCL_5V, SDA_3.3V, SDA_5V
- wire segments 148 -> 149
- no-connect marks 16 -> 8
Other:
- note added: "4th-order low-pass\nanti-aliasing filter\nfc=100kHz"
- note added: "Both inputs must be low to select HV output"
- note added: "EDGE CONNECTOR"
- note added: "FEEDBACK BREAKOUTS"
- note added: "I2C PULLUPS"
- note added: "USB PASSTHROUGH"
- note removed: "4th-order low-pass\nanti-aliasing filter"
- note removed: "COMMUNICATION\nBUS"
- note removed: "FEEDBACK"
- note removed: "I2C LEVEL SHIFTING"
- note removed: "LIGHT"
- note removed: "MAGNET"

Commit message: Update BOM
Parts:
- U10: Mfg_Part_No (none) -> W25Q64FVSSIG TR
- U3: Mfg_Part_No (none) -> CAT5171TBI-50GT3
- U4: Mfg_Part_No HV7802MG-G -> HV7802MG-G
- U9: Mfg_Part_No (none) -> 74AHC1G32GW,125
Changed lines of the file:
@@
 EESchema Schematic File Version 2
-LIBS:dropbot_control_board-rescue
 LIBS:power
 LIBS:device
@@
 F 2 "footprints:MSOP-8" H 10050 5600 60  0001 C CNN
 F 3 "" H 10050 5600 60  0000 C CNN
-F 4 " HV7802MG-G" H 10050 5600 60  0001 C CNN "Mfg_Part_No"
+F 4 "HV7802MG-G" H 10050 5600 60  0001 C CNN "Mfg_Part_No"
 	1    10050 5600
 	1    0    0    -1
@@
 F 1 "CAT5171" H 8100 6100 50  0000 L CNN
 F 2 "WheelerLab:SOT-23-8" H 8050 5750 50  0001 C CNN
-F 3 "" H 8050 5750 50  0000 C CNN
+F 3 "http://www.onsemi.com/pub_link/Collateral/CAT5171-D.PDF" H 8050 5750 50  0001 C CNN
+F 4 "CAT5171TBI-50GT3" H 8050 5750 60  0001 C CNN "Mfg_Part_No"
 	1    8050 5750
 	-1   0    0    -1
@@
 F 1 "74AHC1G32" H 9790 975 50  0000 C CNN
 F 2 "TO_SOT_Packages_SMD:SOT-353" H 9750 1000 50  0001 C CNN
-F 3 "" H 9750 1000 50  0000 C CNN
+F 3 "http://www.nxp.com/documents/data_sheet/74AHC_AHCT1G32.pdf" H 9750 1000 50  0001 C CNN
+F 4 "74AHC1G32GW,125" H 9750 1000 60  0001 C CNN "Mfg_Part_No"
 	1    9750 1000
 	1    0    0    -1
@@
 F 1 "W25Q64FV" H 5200 3595 60  0000 C CNN
 F 2 "SMD_Packages:SOIC-8-N" H 5190 3845 60  0001 C CNN
-F 3 "" H 5190 3845 60  0000 C CNN
+F 3 "https://www.winbond.com/resource-files/w25q64fv%20revq%2006142016.pdf" H 5190 3845 60  0001 C CNN
+F 4 "W25Q64FVSSIG TR" H 5200 3850 60  0001 C CNN "Mfg_Part_No"
 	1    5200 3850
 	1    0    0    -1
