File: dropbot_control_board.sch (KiCad schematic (older format))
At the start: 86 parts, among them IC1 MCP6024, P1 CONN_02X10, P2 CONN_01X04, P3 CONN_01X04, P4 CONN_01X04, P7 CONN_01X04, P8 CONN_01X03, Q1 STP33N65M2, Q5 IRF740BPBF, Q6 IRF740BPBF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

Commit message: Fix BOM
Parts:
- R18: Mfg_Part_No RC0805FR-072KL -> RC0805FR-071KL
- R19, R20, R3, R35, R4: value 5.1k -> 4.75k; Mfg_Part_No RC0805FR-071KL -> RC0805FR-074K75L
- R36: Mfg_Part_No RC0805FR-07200RL -> RC0805FR-074K75L
Changed lines of the file:
@@
 P 2450 2550
 F 0 "R3" V 2530 2550 50  0000 C CNN
-F 1 "5.1k" V 2450 2550 50  0000 C CNN
+F 1 "4.75k" V 2450 2550 50  0000 C CNN
 F 2 "Resistors_SMD:R_0805" H 2450 2550 60  0001 C CNN
 F 3 "" H 2450 2550 60  0001 C CNN
-F 4 "RC0805FR-071KL" H 2450 2550 60  0001 C CNN "Mfg_Part_No"
+F 4 "RC0805FR-074K75L" H 2450 2550 60  0001 C CNN "Mfg_Part_No"
 	1    2450 2550
 	1    0    0    -1
@@
 P 2650 2550
 F 0 "R4" V 2730 2550 50  0000 C CNN
-F 1 "5.1k" V 2650 2550 50  0000 C CNN
+F 1 "4.75k" V 2650 2550 50  0000 C CNN
 F 2 "Resistors_SMD:R_0805" H 2650 2550 60  0001 C CNN
 F 3 "" H 2650 2550 60  0001 C CNN
-F 4 "RC0805FR-071KL" H 2650 2550 60  0001 C CNN "Mfg_Part_No"
+F 4 "RC0805FR-074K75L" H 2650 2550 60  0001 C CNN "Mfg_Part_No"
 	1    2650 2550
 	1    0    0    -1
@@
 F 2 "Resistors_SMD:R_0805" H 1150 1000 60  0001 C CNN
 F 3 "" H 1150 1000 60  0001 C CNN
-F 4 "RC0805FR-072KL" H 1150 1000 60  0001 C CNN "Mfg_Part_No"
+F 4 "RC0805FR-071KL" H 1150 1000 60  0001 C CNN "Mfg_Part_No"
 	1    1150 1000
 	1    0    0    -1
@@
 P 2850 2550
 F 0 "R19" V 2750 2550 50  0000 C CNN
-F 1 "5.1k" V 2850 2550 50  0000 C CNN
+F 1 "4.75k" V 2850 2550 50  0000 C CNN
 F 2 "Resistors_SMD:R_0805" H 2850 2550 60  0001 C CNN
 F 3 "" H 2850 2550 60  0001 C CNN
-F 4 "RC0805FR-071KL" H 2850 2550 60  0001 C CNN "Mfg_Part_No"
+F 4 "RC0805FR-074K75L" H 2850 2550 60  0001 C CNN "Mfg_Part_No"
 	1    2850 2550
 	-1   0    0    1
@@
 P 3050 2550
 F 0 "R20" V 2950 2550 50  0000 C CNN
-F 1 "5.1k" V 3050 2550 50  0000 C CNN
+F 1 "4.75k" V 3050 2550 50  0000 C CNN
 F 2 "Resistors_SMD:R_0805" H 3050 2550 60  0001 C CNN
 F 3 "" H 3050 2550 60  0001 C CNN
-F 4 "RC0805FR-071KL" H 3050 2550 60  0001 C CNN "Mfg_Part_No"
+F 4 "RC0805FR-074K75L" H 3050 2550 60  0001 C CNN "Mfg_Part_No"
 	1    3050 2550
 	-1   0    0    1
@@
 P 4800 3550
 F 0 "R35" V 4880 3550 50  0000 C CNN
-F 1 "5.1k" V 4800 3550 50  0000 C CNN
+F 1 "4.75k" V 4800 3550 50  0000 C CNN
 F 2 "Resistors_SMD:R_0805" H 4800 3550 60  0001 C CNN
 F 3 "" H 4800 3550 60  0001 C CNN
-F 4 "RC0805FR-071KL" H 4800 3550 60  0001 C CNN "Mfg_Part_No"
+F 4 "RC0805FR-074K75L" H 4800 3550 60  0001 C CNN "Mfg_Part_No"
 	1    4800 3550
 	-1   0    0    1
@@
 F 2 "Resistors_SMD:R_0805" V 8930 750 30  0001 C CNN
 F 3 "" H 9000 750 30  0000 C CNN
-F 4 "RC0805FR-07200RL" H 9000 750 60  0001 C CNN "Mfg_Part_No"
+F 4 "RC0805FR-074K75L" H 9000 750 60  0001 C CNN "Mfg_Part_No"
 	1    9000 750
 	-1   0    0    1

Commit message: Fix op-amp package in BOM
Parts:
- IC1: Mfg_Part_No MCP6024T-I/SL -> MCP6024-I/P
Changed lines of the file:
@@
 LIBS:valves
 LIBS:wheelerlab
-LIBS:dropbot_control_board-cache
 EELAYER 25 0
 EELAYER END
@@
 F 2 "Housings_DIP:DIP-14_W7.62mm" H 2200 4600 60  0001 C CNN
 F 3 "" H 2200 4600 60  0000 C CNN
-F 4 "MCP6024T-I/SL" H 2200 4600 60  0001 C CNN "Mfg_Part_No"
+F 4 "MCP6024-I/P" H 2200 4600 60  0001 C CNN "Mfg_Part_No"
 	1    2200 4600
 	1    0    0    -1

Commit message: EMC related improvements
* convert to 4-layer board
* add jumper to connect 3.3V of Teensy
* put filters on i2c
* add guard traces around i2c and current-sense lines
* add ferrites to SPI lines
* add snubber on SPMS diode
* add pads for gate driver current limiting resistors
* add LPF to HV driver
* add PTC fuse and voltage clamp to feedback (current-sense) signal
Parts:
- removed C11: 1uF, Capacitors_SMD:C_0805, symbol C
- removed F1: FUSE, Resistors_ThroughHole:Resistor_Vertical_RM5mm, symbol FUSE
- removed LED2: +5V, LEDs:LED_0805, symbol LED
- removed P1: CONN_02X10, WheelerLab:HSEC8-110-XX-X-RA-MATE, symbol CONN_02X10
- removed P2: CONN_01X04, Pin_Headers:Pin_Header_Straight_1x04, symbol CONN_01X04
- added C11: 1uF, Capacitors_SMD:C_0805, symbol C_Small
- added C23, C25, C30, C31: C_Small, Capacitors_SMD:C_0805, symbol C_Small
- added C24: 1000pF, Capacitors_SMD:C_0805, symbol C
- added C26, C36: 0.1uF, Capacitors_SMD:C_0805, symbol C_Small
- added C27: 0.01uF, Capacitors_SMD:C_0805, symbol C_Small
- added C28, C29: C, Capacitors_SMD:C_0805, symbol C_Small
- added C32: 33uF, WheelerLab:SM2917, symbol CP1
- added C33, C37, C38: 0.1uF, Capacitors_SMD:C_0805, symbol C
- added C34: 0.01uF, Capacitors_SMD:C_0805, symbol C
- added C35: C, Capacitors_SMD:C_1206, symbol C_Small
- added D4: BAV99, TO_SOT_Packages_SMD:SOT-23, symbol BAV99
- added F1: PTC, Resistors_ThroughHole:Resistor_Vertical_RM5mm, symbol F_Small
- added F2: PTC 30mA, Resistors_SMD:R_0805, symbol F_Small
- added FB1, FB2, FB3, FB4, FB5, FB6: FERRITE, Resistors_SMD:R_0805, symbol FERRITE
- added J1: TFM-105-02-X-DH, WheelerLab:TFM-105-02-X-DH, symbol TFM-105-02-X-DH
- added P1, P2, P5: CONN_01X01, Connect:1pin, symbol CONN_01X01
- added R37, R38, R39: 10, Resistors_SMD:R_0805, symbol R
- added R40, R41, R42, R43, R44, R45, R46, R47, R48, R49, R50, R51: R, Resistors_SMD:R_0805, symbol R
- added R52: 0R, Resistors_SMD:R_0805, symbol R
- R18: value 1k -> 10; Mfg_Part_No RC0805FR-071KL -> RC0805FR-0710RL
- renumbered LED3 to LED2
Connections:
- net labels added: CHASIS_GND, D11/M0SI, D12/MISO
- net labels removed: +5V, D+, D-, D11/DI, D12/DO
- wire segments 149 -> 195
- no-connect marks 8 -> 11
Other:
- note added: "Both inputs must be\nlow to select HV output"
- note added: "MOUNTING\nHOLES"
- note removed: "Both inputs must be low to select HV output"
- note removed: "I2C PULLUPS"
- note removed: "USB PASSTHROUGH"

Commit message: Lower the resistance of i2c pullups (4.75k --> 2k)
Parts:
- removed C2: 0.1uF, Capacitors_SMD:C_0805, symbol CP
- added C2: 0.1uF, Capacitors_SMD:C_0805, symbol C
- C23, C25, C30, C31: value C_Small -> C
- C24: Mfg_Part_No CL21B104KBCNNNC -> 501R15W102KV4E
- C27: Mfg_Part_No (none) -> CC0805KRX7R9BB103
- C34: Mfg_Part_No CL21B103KCANNNC -> CC0805KRX7R9BB103
- FB1, FB2, FB3, FB4, FB5, R52: Mfg_Part_No (none) -> RC0805JR-070RL
- FB6: Mfg_Part_No (none) -> 742792040
- J1: Mfg_Part_No (none) -> TFM-105-02-L-DH
- R19, R20, R3, R4: value 4.75k -> 2k; Mfg_Part_No RC0805FR-074K75L -> RC0805FR-072KL
- R40, R41, R42, R43, R44, R45, R46, R47, R48, R49, R50, R51: value R -> 0R; Mfg_Part_No (none) -> RC0805JR-070RL
Changed lines of the file:
@@
 Text GLabel 10350 4850 2    60   Input ~ 0
 HV
-$Comp
-L CP C2
-U 1 1 56BEF332
-P 4700 5000
-F 0 "C2" H 4725 5100 50  0000 L CNN
-F 1 "0.1uF" H 4725 4900 50  0000 L CNN
-F 2 "Capacitors_SMD:C_0805" H 4738 4850 30  0001 C CNN
-F 3 "" H 4700 5000 60  0000 C CNN
-	1    4700 5000
-	1    0    0    -1
-$EndComp
 Text GLabel 1350 750  2    60   Input ~ 0
 +3.3V
@@
 P 9000 2950
 F 0 "R3" V 9000 3200 50  0000 C CNN
-F 1 "4.75k" V 9000 2950 50  0000 C CNN
+F 1 "2k" V 9000 2950 50  0000 C CNN
 F 2 "Resistors_SMD:R_0805" H 9000 2950 60  0001 C CNN
 F 3 "" H 9000 2950 60  0001 C CNN
-F 4 "RC0805FR-074K75L" H 9000 2950 60  0001 C CNN "Mfg_Part_No"
+F 4 "RC0805FR-072KL" H 9000 2950 60  0001 C CNN "Mfg_Part_No"
 	1    9000 2950
 	-1   0    0    1
@@
 P 9250 2950
 F 0 "R4" V 9250 3200 50  0000 C CNN
-F 1 "4.75k" V 9250 2950 50  0000 C CNN
+F 1 "2k" V 9250 2950 50  0000 C CNN
 F 2 "Resistors_SMD:R_0805" H 9250 2950 60  0001 C CNN
 F 3 "" H 9250 2950 60  0001 C CNN
-F 4 "RC0805FR-074K75L" H 9250 2950 60  0001 C CNN "Mfg_Part_No"
+F 4 "RC0805FR-072KL" H 9250 2950 60  0001 C CNN "Mfg_Part_No"
 	1    9250 2950
 	-1   0    0    1
@@
 P 4150 1050
 F 0 "R19" V 4200 1250 50  0000 C CNN
-F 1 "4.75k" V 4150 1050 50  0000 C CNN
+F 1 "2k" V 4150 1050 50  0000 C CNN
 F 2 "Resistors_SMD:R_0805" H 4150 1050 60  0001 C CNN
 F 3 "" H 4150 1050 60  0001 C CNN
-F 4 "RC0805FR-074K75L" H 4150 1050 60  0001 C CNN "Mfg_Part_No"
+F 4 "RC0805FR-072KL" H 4150 1050 60  0001 C CNN "Mfg_Part_No"
 	1    4150 1050
 	-1   0    0    1
@@
 P 4300 1050
 F 0 "R20" V 4350 1250 50  0000 C CNN
-F 1 "4.75k" V 4300 1050 50  0000 C CNN
+F 1 "2k" V 4300 1050 50  0000 C CNN
 F 2 "Resistors_SMD:R_0805" H 4300 1050 60  0001 C CNN
 F 3 "" H 4300 1050 60  0001 C CNN
-F 4 "RC0805FR-074K75L" H 4300 1050 60  0001 C CNN "Mfg_Part_No"
+F 4 "RC0805FR-072KL" H 4300 1050 60  0001 C CNN "Mfg_Part_No"
 	1    4300 1050
 	-1   0    0    1
@@
 F 2 "WheelerLab:TFM-105-02-X-DH" H 2780 1100 20  0001 C CNN
 F 3 "" H 2750 950 60  0000 C CNN
+F 4 "TFM-105-02-L-DH" H 2750 950 60  0001 C CNN "Mfg_Part_No"
 	1    2750 950
 	1    0    0    -1
@@
 F 2 "Capacitors_SMD:C_0805" H 7038 4400 30  0001 C CNN
 F 3 "" H 7000 4550 60  0000 C CNN
-F 4 "CL21B104KBCNNNC" H 7000 4550 60  0001 C CNN "Mfg_Part_No"
+F 4 "501R15W102KV4E" H 7000 4550 60  0001 C CNN "Mfg_Part_No"
 	1    7000 4550
 	0    1    1    0
@@
 P 7850 2550
 F 0 "R45" V 7800 2750 50  0000 C CNN
-F 1 "R" V 7850 2550 50  0000 C CNN
+F 1 "0R" V 7850 2550 50  0000 C CNN
 F 2 "Resistors_SMD:R_0805" V 7780 2550 50  0001 C CNN
 F 3 "" H 7850 2550 50  0000 C CNN
+F 4 "RC0805JR-070RL" H 7850 2550 60  0001 C CNN "Mfg_Part_No"
 	1    7850 2550
 	0    1    1    0
@@
 P 7850 2400
 F 0 "R44" V 7800 2600 50  0000 C CNN
-F 1 "R" V 7850 2400 50  0000 C CNN
+F 1 "0R" V 7850 2400 50  0000 C CNN
 F 2 "Resistors_SMD:R_0805" V 7780 2400 50  0001 C CNN
 F 3 "" H 7850 2400 50  0000 C CNN
+F 4 "RC0805JR-070RL" H 7850 2400 60  0001 C CNN "Mfg_Part_No"
 	1    7850 2400
 	0    1    1    0
@@
 P 8850 2550
 F 0 "R51" V 8950 2550 50  0000 C CNN
-F 1 "R" V 8850 2550 50  0000 C CNN
+F 1 "0R" V 8850 2550 50  0000 C CNN
 F 2 "Resistors_SMD:R_0805" V 8780 2550 50  0001 C CNN
 F 3 "" H 8850 2550 50  0000 C CNN
+F 4 "RC0805JR-070RL" H 8850 2550 60  0001 C CNN "Mfg_Part_No"
 	1    8850 2550
 	0    1    1    0
@@
 P 9100 2400
 F 0 "R50" V 9000 2400 50  0000 C CNN
-F 1 "R" V 9100 2400 50  0000 C CNN
+F 1 "0R" V 9100 2400 50  0000 C CNN
 F 2 "Resistors_SMD:R_0805" V 9030 2400 50  0001 C CNN
 F 3 "" H 9100 2400 50  0000 C CNN
+F 4 "RC0805JR-070RL" H 9100 2400 60  0001 C CNN "Mfg_Part_No"
 	1    9100 2400
 	0    1    1    0
@@
 P 8900 5550
 F 0 "C30" H 8700 5550 50  0000 L CNN
-F 1 "C_Small" H 9000 5500 50  0000 L CNN
+F 1 "C" H 9000 5500 50  0000 L CNN
 F 2 "Capacitors_SMD:C_0805" H 8900 5550 50  0001 C CNN
 F 3 "" H 8900 5550 50  0000 C CNN
@@
 P 8750 5650
 F 0 "R46" V 8700 5450 50  0000 C CNN
-F 1 "R" V 8750 5650 50  0000 C CNN
+F 1 "0R" V 8750 5650 50  0000 C CNN
 F 2 "Resistors_SMD:R_0805" V 8680 5650 50  0001 C CNN
 F 3 "" H 8750 5650 50  0000 C CNN
+F 4 "RC0805JR-070RL" H 8750 5650 60  0001 C CNN "Mfg_Part_No"
 	1    8750 5650
 	0    1    1    0
@@
 P 8750 5750
 F 0 "R47" V 8700 5550 50  0000 C CNN
-F 1 "R" V 8750 5750 50  0000 C CNN
+F 1 "0R" V 8750 5750 50  0000 C CNN
 F 2 "Resistors_SMD:R_0805" V 8680 5750 50  0001 C CNN
 F 3 "" H 8750 5750 50  0000 C CNN
+F 4 "RC0805JR-070RL" H 8750 5750 60  0001 C CNN "Mfg_Part_No"
 	1    8750 5750
 	0    1    1    0
@@
 P 8900 5850
 F 0 "C31" H 8700 5850 50  0000 L CNN
-F 1 "C_Small" H 9000 5850 50  0000 L CNN
+F 1 "C" H 9000 5850 50  0000 L CNN
 F 2 "Capacitors_SMD:C_0805" H 8900 5850 50  0001 C CNN
 F 3 "" H 8900 5850 50  0000 C CNN
@@
 P 9050 5650
 F 0 "R48" V 8950 5800 50  0000 C CNN
-F 1 "R" V 9050 5650 50  0000 C CNN
+F 1 "0R" V 9050 5650 50  0000 C CNN
 F 2 "Resistors_SMD:R_0805" V 8980 5650 50  0001 C CNN
 F 3 "" H 9050 5650 50  0000 C CNN
+F 4 "RC0805JR-070RL" H 9050 5650 60  0001 C CNN "Mfg_Part_No"
 	1    9050 5650
 	0    1    1    0
@@
 P 9050 5750
 F 0 "R49" V 9150 5900 50  0000 C CNN
-F 1 "R" V 9050 5750 50  0000 C CNN
+F 1 "0R" V 9050 5750 50  0000 C CNN
 F 2 "Resistors_SMD:R_0805" V 8980 5750 50  0001 C CNN
 F 3 "" H 9050 5750 50  0000 C CNN
+F 4 "RC0805JR-070RL" H 9050 5750 60  0001 C CNN "Mfg_Part_No"
 	1    9050 5750
 	0    1    1    0
@@
 F 2 "Resistors_SMD:R_0805" H 9750 3000 60  0001 C CNN
 F 3 "" H 9750 3000 60  0000 C CNN
+F 4 "RC0805JR-070RL" H 9750 3100 60  0001 C CNN "Mfg_Part_No"
 	1    9750 3100
 	1    0    0    -1
@@
 F 2 "Capacitors_SMD:C_0805" H 9550 3200 50  0001 C CNN
 F 3 "" H 9550 3200 50  0000 C CNN
+F 4 "CC0805KRX7R9BB103" H 9550 3200 60  0001 C CNN "Mfg_Part_No"
 	1    9550 3200
 	-1   0    0    1
@@
 P 5400 2250
 F 0 "R43" V 5350 2450 50  0000 C CNN
-F 1 "R" V 5400 2250 50  0000 C CNN
+F 1 "0R" V 5400 2250 50  0000 C CNN
 F 2 "Resistors_SMD:R_0805" V 5330 2250 50  0001 C CNN
 F 3 "" H 5400 2250 50  0000 C CNN
+F 4 "RC0805JR-070RL" H 5400 2250 60  0001 C CNN "Mfg_Part_No"
 	1    5400 2250
 	0    1    1    0
@@
 P 5400 2100
 F 0 "R42" V 5350 2300 50  0000 C CNN
-F 1 "R" V 5400 2100 50  0000 C CNN
+F 1 "0R" V 5400 2100 50  0000 C CNN
 F 2 "Resistors_SMD:R_0805" V 5330 2100 50  0001 C CNN
 F 3 "" H 5400 2100 50  0000 C CNN
+F 4 "RC0805JR-070RL" H 5400 2100 60  0001 C CNN "Mfg_Part_No"
 	1    5400 2100
 	0    1    1    0
@@
 P 4750 2350
 F 0 "C25" H 4600 2450 50  0000 L CNN
-F 1 "C_Small" H 4400 2300 50  0000 L CNN
+F 1 "C" H 4600 2300 50  0000 L CNN
 F 2 "Capacitors_SMD:C_0805" H 4750 2350 50  0001 C CNN
 F 3 "" H 4750 2350 50  0000 C CNN
@@
 P 4600 2250
 F 0 "R41" V 4550 2450 50  0000 C CNN
-F 1 "R" V 4600 2250 50  0000 C CNN
+F 1 "0R" V 4600 2250 50  0000 C CNN
 F 2 "Resistors_SMD:R_0805" V 4530 2250 50  0001 C CNN
 F 3 "" H 4600 2250 50  0000 C CNN
+F 4 "RC0805JR-070RL" H 4600 2250 60  0001 C CNN "Mfg_Part_No"
 	1    4600 2250
 	0    1    1    0
@@
 P 4600 2100
 F 0 "R40" V 4500 2100 50  0000 C CNN
-F 1 "R" V 4600 2100 50  0000 C CNN
+F 1 "0R" V 4600 2100 50  0000 C CNN
 F 2 "Resistors_SMD:R_0805" V 4530 2100 50  0001 C CNN
 F 3 "" H 4600 2100 50  0000 C CNN
+F 4 "RC0805JR-070RL" H 4600 2100 60  0001 C CNN "Mfg_Part_No"
 	1    4600 2100
 	0    1    1    0
@@
 P 4750 2000
 F 0 "C23" H 4600 1900 50  0000 L CNN
-F 1 "C_Small" H 4400 2050 50  0000 L CNN
+F 1 "C" H 4600 2050 50  0000 L CNN
 F 2 "Capacitors_SMD:C_0805" H 4750 2000 50  0001 C CNN
 F 3 "" H 4750 2000 50  0000 C CNN
@@
 F 2 "Capacitors_SMD:C_0805" H 1100 1100 60  0001 C CNN
 F 3 "" H 1100 1100 60  0001 C CNN
-F 4 "CL21B103KCANNNC" H 1100 1100 60  0001 C CNN "Mfg_Part_No"
+F 4 "CC0805KRX7R9BB103" H 1100 1100 60  0001 C CNN "Mfg_Part_No"
 	1    1100 1100
 	-1   0    0    1
@@
 F 2 "Resistors_SMD:R_0805" H 5950 7300 60  0001 C CNN
 F 3 "" H 5950 7300 60  0000 C CNN
+F 4 "RC0805JR-070RL" H 5950 7400 60  0001 C CNN "Mfg_Part_No"
 	1    5950 7400
 	1    0    0    -1
@@
 F 2 "Resistors_SMD:R_0805" H 5550 3050 60  0001 C CNN
 F 3 "" H 5550 3050 60  0000 C CNN
+F 4 "RC0805JR-070RL" H 5550 3150 60  0001 C CNN "Mfg_Part_No"
 	1    5550 3150
 	1    0    0    -1
@@
 F 2 "Resistors_SMD:R_0805" H 4250 3700 60  0001 C CNN
 F 3 "" H 4250 3700 60  0000 C CNN
+F 4 "RC0805JR-070RL" H 4250 3800 60  0001 C CNN "Mfg_Part_No"
 	1    4250 3800
 	1    0    0    -1
@@
 F 2 "Resistors_SMD:R_0805" H 7850 3200 60  0001 C CNN
 F 3 "" H 7850 3200 60  0000 C CNN
+F 4 "RC0805JR-070RL" H 7850 3300 60  0001 C CNN "Mfg_Part_No"
 	1    7850 3300
 	1    0    0    -1
@@
 F 2 "Resistors_SMD:R_0805" H 1700 1650 60  0001 C CNN
 F 3 "" H 1700 1650 60  0000 C CNN
+F 4 "742792040" H 1700 1750 60  0001 C CNN "Mfg_Part_No"
 	1    1700 1750
 	0    1    1    0
@@
 F 2 "Resistors_SMD:R_0805" V 7780 1650 50  0001 C CNN
 F 3 "" H 7850 1650 50  0000 C CNN
+F 4 "RC0805JR-070RL" H 7850 1650 60  0001 C CNN "Mfg_Part_No"
 	1    7850 1650
 	0    1    1    0
@@
 NoConn ~ 6600 3850
 NoConn ~ 6750 3850
+$Comp
+L C C2
+U 1 1 58CA2C47
+P 4700 5000
+F 0 "C2" H 4550 4900 50  0000 L CNN
+F 1 "0.1uF" H 4450 5100 50  0000 L CNN
+F 2 "Capacitors_SMD:C_0805" H 4700 5000 60  0001 C CNN
+F 3 "" H 4700 5000 60  0001 C CNN
+F 4 "CL21B104KBCNNNC" H 4700 5000 60  0001 C CNN "Mfg_Part_No"
+	1    4700 5000
+	-1   0    0    1
+$EndComp
 $EndSCHEMATC

Commit message: Add usb passthrough, reset button, ...
* add usb passthrough
* add reset button
* fix bad trace on U5
* fix part number for C7 (3.3uF instead of 10uF)
Parts:
- removed C10, C4: 100n,500V, Capacitors_SMD:C_1210, symbol C_Small
- removed C12: 1pF, Capacitors_SMD:C_0805, symbol C
- removed C13: 10pF, Capacitors_SMD:C_0805, symbol C
- removed C14: 100pF, Capacitors_SMD:C_0805, symbol C
- removed C15: 1nF, Capacitors_SMD:C_0805, symbol C
- removed C3: 0.1uF, Capacitors_SMD:C_0805, symbol C_Small
- removed C35: C, Capacitors_SMD:C_1206, symbol C_Small
- removed D2, D3: D, Diodes_SMD:SMA_Standard, symbol D
- removed F1: PTC, Resistors_ThroughHole:Resistor_Vertical_RM5mm, symbol F_Small
- removed FB2: FERRITE, Resistors_SMD:R_0805, symbol FERRITE
- removed Q5, Q6: IRF740BPBF, TO_SOT_Packages_THT:TO-220_Neutral123_Horizontal_LargePads, symbol Q_NMOS_GDS
- removed R18, R21, R37: 10, Resistors_SMD:R_0805, symbol R
- removed R22: 2M, Resistors_SMD:R_1206, symbol R
- removed R24, R28, R29, R30: 200, Resistors_SMD:R_0805, symbol R
- removed U6: NCP5304, SMD_Packages:SOIC-8-N, symbol NCP5304
- removed U7, U8: DPST (2 Form A), 350V, SMD_Packages:DIP-8_SMD, symbol AQW216
- added P10: CONN_01X01, Pin_Headers:Pin_Header_Straight_1x01_Pitch2.54mm, symbol CONN_01X01
- added SW1: PROG, WheelerLab:PTS840_GK_SMTR_LFS, symbol SPST
- C7: Mfg_Part_No EEV-EB2E100Q -> EEV-EB2G3R3Q
Connections:
- wire segments 195 -> 156
Other:
- note added: "PROGRAM BUTTON"
- note removed: "C12-15 should be\nrated for >100V"
- note removed: "HV SQUARE WAVE DRIVER"
- note removed: "ON-BOARD CALIBRATION"

Commit message: Swap F2 for higher voltage rating, monitor HV_OE
* swap F2 for 1210 footprint: B59807A90A62 (higher voltage rating)
* monitor HV_OE with A8
Parts:
- F2: footprint Resistors_SMD:R_0805 -> Resistors_SMD:R_1210; Mfg_Part_No PRG21BB220MB1RK -> B59807A90A62
Connections:
- no-connect marks 11 -> 10
Changed lines of the file:
@@
 Sheet 1 4
 Title "DropBot control board"
-Date "2017-03-21"
-Rev "3.2"
+Date "2017-04-04"
+Rev "3.3"
 Comp "Sci-Bots Inc."
 Comment1 ""
@@
 NoConn ~ 6900 3850
 NoConn ~ 7050 3850
-NoConn ~ 7700 1950
 NoConn ~ 7700 1800
 NoConn ~ 7700 1500
@@
 F 0 "F2" H 810 4160 50  0000 L CNN
 F 1 "PTC 30mA" H 700 4000 50  0000 L CNN
-F 2 "Resistors_SMD:R_0805" H 850 4100 50  0001 C CNN
+F 2 "Resistors_SMD:R_1210" H 850 4100 50  0001 C CNN
 F 3 "" H 850 4100 50  0000 C CNN
-F 4 "PRG21BB220MB1RK" H 850 4100 60  0001 C CNN "Mfg_Part_No"
+F 4 "B59807A90A62" H 850 4100 60  0001 C CNN "Mfg_Part_No"
 	1    850  4100
 	0    1    1    0
@@
 Wire Wire Line
 	4300 2750 4300 2950
+Text GLabel 7700 1950 2    60   Input ~ 0
+HV_OE
 $EndSCHEMATC
