File: dropbot_control_board.sch (KiCad schematic (older format))
At the start: 104 parts, among them IC1 MCP6024, J1 TFM-105-02-X-DH, P1 CONN_01X01, P10 CONN_01X01, P2 CONN_01X01, P3 CONN_01X04, P4 CONN_01X04, P5 CONN_01X01, P7 CONN_01X04, P8 CONN_01X03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

Commit message: Change part numbers for i2c filters
Parts:
- C23, C25, C28, C29, C30, C31: value C -> 150pF; Mfg_Part_No (none) -> CL21C151JBANNNC
- R40, R41, R48, R49, R50, R51: value 0R -> 150; Mfg_Part_No RC0805JR-070RL -> RC0805FR-07150RL
- R42, R43, R44, R45, R46, R47: value 0R -> 51; Mfg_Part_No RC0805JR-070RL -> RC0805FR-0751RL
Changed lines of the file:
@@
 Sheet 1 4
 Title "DropBot control board"
-Date "2017-04-04"
+Date "2017-04-05"
 Rev "3.3"
 Comp "Sci-Bots Inc."
@@
 P 7850 2550
 F 0 "R45" V 7800 2750 50  0000 C CNN
-F 1 "0R" V 7850 2550 50  0000 C CNN
+F 1 "51" V 7850 2550 50  0000 C CNN
 F 2 "Resistors_SMD:R_0805" V 7780 2550 50  0001 C CNN
 F 3 "" H 7850 2550 50  0000 C CNN
-F 4 "RC0805JR-070RL" H 7850 2550 60  0001 C CNN "Mfg_Part_No"
+F 4 "RC0805FR-0751RL" H 7850 2550 60  0001 C CNN "Mfg_Part_No"
 	1    7850 2550
 	0    1    1    0
@@
 P 7850 2400
 F 0 "R44" V 7800 2600 50  0000 C CNN
-F 1 "0R" V 7850 2400 50  0000 C CNN
+F 1 "51" V 7850 2400 50  0000 C CNN
 F 2 "Resistors_SMD:R_0805" V 7780 2400 50  0001 C CNN
 F 3 "" H 7850 2400 50  0000 C CNN
-F 4 "RC0805JR-070RL" H 7850 2400 60  0001 C CNN "Mfg_Part_No"
+F 4 "RC0805FR-0751RL" H 7850 2400 60  0001 C CNN "Mfg_Part_No"
 	1    7850 2400
 	0    1    1    0
@@
 P 8200 2300
 F 0 "C28" H 8050 2200 50  0000 L CNN
-F 1 "C" H 8150 2350 50  0000 L CNN
+F 1 "150pF" H 7900 2300 50  0000 L CNN
 F 2 "Capacitors_SMD:C_0805" H 8200 2300 50  0001 C CNN
 F 3 "" H 8200 2300 50  0000 C CNN
+F 4 "CL21C151JBANNNC" H 8200 2300 60  0001 C CNN "Mfg_Part_No"
 	1    8200 2300
 	-1   0    0    1
@@
 P 8850 2550
 F 0 "R51" V 8950 2550 50  0000 C CNN
-F 1 "0R" V 8850 2550 50  0000 C CNN
+F 1 "150" V 8850 2550 50  0000 C CNN
 F 2 "Resistors_SMD:R_0805" V 8780 2550 50  0001 C CNN
 F 3 "" H 8850 2550 50  0000 C CNN
-F 4 "RC0805JR-070RL" H 8850 2550 60  0001 C CNN "Mfg_Part_No"
+F 4 "RC0805FR-07150RL" H 8850 2550 60  0001 C CNN "Mfg_Part_No"
 	1    8850 2550
 	0    1    1    0
@@
 P 9100 2400
 F 0 "R50" V 9000 2400 50  0000 C CNN
-F 1 "0R" V 9100 2400 50  0000 C CNN
+F 1 "150" V 9100 2400 50  0000 C CNN
 F 2 "Resistors_SMD:R_0805" V 9030 2400 50  0001 C CNN
 F 3 "" H 9100 2400 50  0000 C CNN
-F 4 "RC0805JR-070RL" H 9100 2400 60  0001 C CNN "Mfg_Part_No"
+F 4 "RC0805FR-07150RL" H 9100 2400 60  0001 C CNN "Mfg_Part_No"
 	1    9100 2400
 	0    1    1    0
@@
 P 8600 2650
 F 0 "C29" H 8450 2750 50  0000 L CNN
-F 1 "C" H 8550 2600 50  0000 L CNN
+F 1 "150pF" H 8650 2600 50  0000 L CNN
 F 2 "Capacitors_SMD:C_0805" H 8600 2650 50  0001 C CNN
 F 3 "" H 8600 2650 50  0000 C CNN
+F 4 "CL21C151JBANNNC" H 8600 2650 60  0001 C CNN "Mfg_Part_No"
 	1    8600 2650
 	-1   0    0    1
@@
 P 8900 5550
 F 0 "C30" H 8700 5550 50  0000 L CNN
-F 1 "C" H 9000 5500 50  0000 L CNN
+F 1 "150pF" H 9000 5500 50  0000 L CNN
 F 2 "Capacitors_SMD:C_0805" H 8900 5550 50  0001 C CNN
 F 3 "" H 8900 5550 50  0000 C CNN
+F 4 "CL21C151JBANNNC" H 8900 5550 60  0001 C CNN "Mfg_Part_No"
 	1    8900 5550
 	-1   0    0    1
@@
 P 8750 5650
 F 0 "R46" V 8700 5450 50  0000 C CNN
-F 1 "0R" V 8750 5650 50  0000 C CNN
+F 1 "51" V 8750 5650 50  0000 C CNN
 F 2 "Resistors_SMD:R_0805" V 8680 5650 50  0001 C CNN
 F 3 "" H 8750 5650 50  0000 C CNN
-F 4 "RC0805JR-070RL" H 8750 5650 60  0001 C CNN "Mfg_Part_No"
+F 4 "RC0805FR-0751RL" H 8750 5650 60  0001 C CNN "Mfg_Part_No"
 	1    8750 5650
 	0    1    1    0
@@
 P 8750 5750
 F 0 "R47" V 8700 5550 50  0000 C CNN
-F 1 "0R" V 8750 5750 50  0000 C CNN
+F 1 "51" V 8750 5750 50  0000 C CNN
 F 2 "Resistors_SMD:R_0805" V 8680 5750 50  0001 C CNN
 F 3 "" H 8750 5750 50  0000 C CNN
-F 4 "RC0805JR-070RL" H 8750 5750 60  0001 C CNN "Mfg_Part_No"
+F 4 "RC0805FR-0751RL" H 8750 5750 60  0001 C CNN "Mfg_Part_No"
 	1    8750 5750
 	0    1    1    0
@@
 P 8900 5850
 F 0 "C31" H 8700 5850 50  0000 L CNN
-F 1 "C" H 9000 5850 50  0000 L CNN
+F 1 "150pF" H 9000 5850 50  0000 L CNN
 F 2 "Capacitors_SMD:C_0805" H 8900 5850 50  0001 C CNN
 F 3 "" H 8900 5850 50  0000 C CNN
+F 4 "CL21C151JBANNNC" H 8900 5850 60  0001 C CNN "Mfg_Part_No"
 	1    8900 5850
 	-1   0    0    1
@@
 P 9050 5650
 F 0 "R48" V 8950 5800 50  0000 C CNN
-F 1 "0R" V 9050 5650 50  0000 C CNN
+F 1 "150" V 9050 5650 50  0000 C CNN
 F 2 "Resistors_SMD:R_0805" V 8980 5650 50  0001 C CNN
 F 3 "" H 9050 5650 50  0000 C CNN
-F 4 "RC0805JR-070RL" H 9050 5650 60  0001 C CNN "Mfg_Part_No"
+F 4 "RC0805FR-07150RL" H 9050 5650 60  0001 C CNN "Mfg_Part_No"
 	1    9050 5650
 	0    1    1    0
@@
 P 9050 5750
 F 0 "R49" V 9150 5900 50  0000 C CNN
-F 1 "0R" V 9050 5750 50  0000 C CNN
+F 1 "150" V 9050 5750 50  0000 C CNN
 F 2 "Resistors_SMD:R_0805" V 8980 5750 50  0001 C CNN
 F 3 "" H 9050 5750 50  0000 C CNN
-F 4 "RC0805JR-070RL" H 9050 5750 60  0001 C CNN "Mfg_Part_No"
+F 4 "RC0805FR-07150RL" H 9050 5750 60  0001 C CNN "Mfg_Part_No"
 	1    9050 5750
 	0    1    1    0
@@
 P 5400 2250
 F 0 "R43" V 5350 2450 50  0000 C CNN
-F 1 "0R" V 5400 2250 50  0000 C CNN
+F 1 "51" V 5400 2250 50  0000 C CNN
 F 2 "Resistors_SMD:R_0805" V 5330 2250 50  0001 C CNN
 F 3 "" H 5400 2250 50  0000 C CNN
-F 4 "RC0805JR-070RL" H 5400 2250 60  0001 C CNN "Mfg_Part_No"
+F 4 "RC0805FR-0751RL" H 5400 2250 60  0001 C CNN "Mfg_Part_No"
 	1    5400 2250
 	0    1    1    0
@@
 P 5400 2100
 F 0 "R42" V 5350 2300 50  0000 C CNN
-F 1 "0R" V 5400 2100 50  0000 C CNN
+F 1 "51" V 5400 2100 50  0000 C CNN
 F 2 "Resistors_SMD:R_0805" V 5330 2100 50  0001 C CNN
 F 3 "" H 5400 2100 50  0000 C CNN
-F 4 "RC0805JR-070RL" H 5400 2100 60  0001 C CNN "Mfg_Part_No"
+F 4 "RC0805FR-0751RL" H 5400 2100 60  0001 C CNN "Mfg_Part_No"
 	1    5400 2100
 	0    1    1    0
@@
 P 4750 2350
 F 0 "C25" H 4600 2450 50  0000 L CNN
-F 1 "C" H 4600 2300 50  0000 L CNN
+F 1 "150pF" H 4450 2300 50  0000 L CNN
 F 2 "Capacitors_SMD:C_0805" H 4750 2350 50  0001 C CNN
 F 3 "" H 4750 2350 50  0000 C CNN
+F 4 "CL21C151JBANNNC" H 4750 2350 60  0001 C CNN "Mfg_Part_No"
 	1    4750 2350
 	-1   0    0    1
@@
 P 4600 2250
 F 0 "R41" V 4550 2450 50  0000 C CNN
-F 1 "0R" V 4600 2250 50  0000 C CNN
+F 1 "150" V 4600 2250 50  0000 C CNN
 F 2 "Resistors_SMD:R_0805" V 4530 2250 50  0001 C CNN
 F 3 "" H 4600 2250 50  0000 C CNN
-F 4 "RC0805JR-070RL" H 4600 2250 60  0001 C CNN "Mfg_Part_No"
+F 4 "RC0805FR-07150RL" H 4600 2250 60  0001 C CNN "Mfg_Part_No"
 	1    4600 2250
 	0    1    1    0
@@
 P 4600 2100
 F 0 "R40" V 4500 2100 50  0000 C CNN
-F 1 "0R" V 4600 2100 50  0000 C CNN
+F 1 "150" V 4600 2100 50  0000 C CNN
 F 2 "Resistors_SMD:R_0805" V 4530 2100 50  0001 C CNN
 F 3 "" H 4600 2100 50  0000 C CNN
-F 4 "RC0805JR-070RL" H 4600 2100 60  0001 C CNN "Mfg_Part_No"
+F 4 "RC0805FR-07150RL" H 4600 2100 60  0001 C CNN "Mfg_Part_No"
 	1    4600 2100
 	0    1    1    0
@@
 P 4750 2000
 F 0 "C23" H 4600 1900 50  0000 L CNN
-F 1 "C" H 4600 2050 50  0000 L CNN
+F 1 "150pF" H 4450 2000 50  0000 L CNN
 F 2 "Capacitors_SMD:C_0805" H 4750 2000 50  0001 C CNN
 F 3 "" H 4750 2000 50  0000 C CNN
+F 4 "CL21C151JBANNNC" H 4750 2000 60  0001 C CNN "Mfg_Part_No"
 	1    4750 2000
 	-1   0    0    1

Commit message: Update BOM with alternate parts for C6 and D4
These parts were out of stock at Digi-key as of 2017-04-18.
Parts:
- C6: value 100uF,35V -> 100uF; Mfg_Part_No TAJE107K020RNJ -> T491X107K025AT
- D4: Mfg_Part_No BAV99LT1G -> BAV99-7-F
Changed lines of the file:
@@
 P 5450 4700
 F 0 "C6" H 5475 4800 50  0000 L CNN
-F 1 "100uF,35V" H 5475 4600 50  0000 L CNN
+F 1 "100uF" H 5475 4600 50  0000 L CNN
 F 2 "Capacitors_Tantalum_SMD:TantalC_SizeE_EIA-7360_Reflow" H 5488 4550 30  0001 C CNN
 F 3 "" H 5450 4700 60  0000 C CNN
-F 4 "TAJE107K020RNJ" H 5450 4700 60  0001 C CNN "Mfg_Part_No"
+F 4 "T491X107K025AT" H 5450 4700 60  0001 C CNN "Mfg_Part_No"
 	1    5450 4700
 	1    0    0    -1
@@
 F 2 "TO_SOT_Packages_SMD:SOT-23" H 650 4900 50  0001 C CNN
 F 3 "" H 650 4900 50  0000 C CNN
-F 4 "BAV99LT1G" H 650 4900 60  0001 C CNN "Mfg_Part_No"
+F 4 "BAV99-7-F" H 650 4900 60  0001 C CNN "Mfg_Part_No"
 	1    650  4900
 	0    -1   -1   0
