File: dropbot_control_board.sch (KiCad schematic (older format))
At the start: 48 parts, among them P1 CONN_01X01, P10 CONN_01X01, P11 TFM-105-02-X-DH, P2 CONN_01X01, P3 CONN_01X03, P4 CONN_01X02, P5 CONN_01X01, P7 CONN_01X04, P8 CONN_01X03, SW1 PROG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

Commit message: Improve layout/stability of boost converter, etc.
* improve layout/stability of boost converter
* enable on board calibration without HVOE
* add decoupling cap to 0.6V reference
* fix footprint for U10
* add programming wire
Parts:
- added C22: 0.1uF, Capacitors_SMD:C_0805, symbol C_Small
- U1: footprint footprints:Teensy-3.2 -> WheelerLab:Teensy-3.2
- U10: footprint SMD_Packages:SOIC-8-N -> WheelerLab:SSO-8_5.2x5.2mm_Pitch1.27mm
Connections:
- net labels added: PROG
- wire segments 52 -> 54
- no-connect marks 10 -> 9
Changed lines of the file:
@@
 LIBS:valves
 LIBS:wheelerlab
+LIBS:dropbot_control_board-cache
 EELAYER 25 0
 EELAYER END
@@
 Sheet 1 7
 Title "DropBot control board"
-Date "2017-05-17"
-Rev "3.5"
+Date "2017-06-19"
+Rev "3.6"
 Comp "Sci-Bots Inc."
 Comment1 ""
@@
 +3.3V
 NoConn ~ 6600 5200
-NoConn ~ 7050 5200
 NoConn ~ 7200 5200
 NoConn ~ 7850 3150
@@
 Text GLabel 1050 2700 2    60   Input ~ 0
 D6/DRIVER_LO
-Text GLabel 7850 2250 2    60   Input ~ 0
+Text GLabel 8300 2250 2    60   Input ~ 0
 +0.6V
 NoConn ~ 7850 2100
@@
 F 0 "U10" H 4855 5445 60  0000 C CNN
 F 1 "W25Q64FV" H 4850 4945 60  0000 C CNN
-F 2 "SMD_Packages:SOIC-8-N" H 4840 5195 60  0001 C CNN
+F 2 "WheelerLab:SSO-8_5.2x5.2mm_Pitch1.27mm" H 4840 5195 60  0001 C CNN
 F 3 "https://www.winbond.com/resource-files/w25q64fv%20revq%2006142016.pdf" H 4840 5195 60  0001 C CNN
 F 4 "W25Q64FVSSIG TR" H 4850 5200 60  0001 C CNN "Mfg_Part_No"
@@
 F 0 "U1" H 6850 3450 60  0000 C CNN
 F 1 "Teensy_3.2" H 6850 4900 60  0000 C CNN
-F 2 "footprints:Teensy-3.2" H 6950 2900 60  0001 C CNN
+F 2 "WheelerLab:Teensy-3.2" H 6950 2900 60  0001 C CNN
 F 3 "" H 6950 2900 60  0000 C CNN
 	1    6850 3450
@@
 Wire Wire Line
 	1950 1500 1950 1400
+$Comp
+L C_Small C22
+U 1 1 5947932E
+P 8300 2350
+F 0 "C22" H 8050 2350 50  0000 L CNN
+F 1 "0.1uF" H 8050 2450 50  0000 L CNN
+F 2 "Capacitors_SMD:C_0805" H 8300 2350 50  0001 C CNN
+F 3 "" H 8300 2350 50  0000 C CNN
+F 4 "CL21B104KBCNNNC" H 8300 2350 60  0001 C CNN "Mfg_Part_No"
+	1    8300 2350
+	-1   0    0    1
+$EndComp
+Wire Wire Line
+	7850 2250 8300 2250
+Text GLabel 8300 2550 2    60   Input ~ 0
+GND
+Wire Wire Line
+	8300 2550 8300 2450
+Text GLabel 1050 3900 3    60   Input ~ 0
+PROG
+Text GLabel 7050 5200 3    60   Input ~ 0
+PROG
 $EndSCHEMATC

Commit message: Change EEPROM and swap 150 Ohm resisotors for 100...
Change EEPROM and swap 150 Ohm resisotors for 100 resistors
driving the PhotoMOS switches.
Parts:
- U10: value W25Q64FV -> IS25LP064A-JBLE; Mfg_Part_No W25Q64FVSSIG TR -> IS25LP064A-JBLE
Changed lines of the file:
@@
 P 4850 5200
 F 0 "U10" H 4855 5445 60  0000 C CNN
-F 1 "W25Q64FV" H 4850 4945 60  0000 C CNN
+F 1 "IS25LP064A-JBLE" H 4850 4945 60  0000 C CNN
 F 2 "WheelerLab:SSO-8_5.2x5.2mm_Pitch1.27mm" H 4840 5195 60  0001 C CNN
 F 3 "https://www.winbond.com/resource-files/w25q64fv%20revq%2006142016.pdf" H 4840 5195 60  0001 C CNN
-F 4 "W25Q64FVSSIG TR" H 4850 5200 60  0001 C CNN "Mfg_Part_No"
+F 4 "IS25LP064A-JBLE" H 4850 5200 60  0001 C CNN "Mfg_Part_No"
 	1    4850 5200
 	1    0    0    -1

Commit message: Fix label of A2, update netlist
Connections:
- net labels added: A2/HV7802_CS
- net labels removed: A2/HV507_CS
Changed lines of the file:
@@
 NoConn ~ 7850 2700
 Text GLabel 7850 4200 2    60   Input ~ 0
-A2/HV507_CS
+A2/HV7802_CS
 Text GLabel 7850 4050 2    60   Input ~ 0
 A3/MAX1771_CS

Commit message: Update schematic to use power ports
Connections:
- wire segments 54 -> 63

Commit message: Update to use Sci-Bots library
Parts:
- C32: footprint WheelerLab:SM2917 -> Sci-Bots:SM2917
- P11: footprint WheelerLab:TFM-105-02-X-DH -> Sci-Bots:TFM-105-02-X-DH
- SW1: footprint WheelerLab:PTS840_GK_SMTR_LFS -> Sci-Bots:PTS840_GK_SMTR_LFS
- U1: footprint WheelerLab:Teensy-3.2 -> Sci-Bots:Teensy-3.2
- U10: footprint WheelerLab:SSO-8_5.2x5.2mm_Pitch1.27mm -> Sci-Bots:SSO-8_5.2x5.2mm_Pitch1.27mm
Changed lines of the file:
@@
 LIBS:contrib
 LIBS:valves
-LIBS:wheelerlab
+LIBS:sci-bots
 LIBS:dropbot_control_board-cache
 EELAYER 25 0
@@
 F 0 "U10" H 4855 5445 60  0000 C CNN
 F 1 "IS25LP064A-JBLE" H 4850 4945 60  0000 C CNN
-F 2 "WheelerLab:SSO-8_5.2x5.2mm_Pitch1.27mm" H 4840 5195 60  0001 C CNN
+F 2 "Sci-Bots:SSO-8_5.2x5.2mm_Pitch1.27mm" H 4840 5195 60  0001 C CNN
 F 3 "https://www.winbond.com/resource-files/w25q64fv%20revq%2006142016.pdf" H 4840 5195 60  0001 C CNN
 F 4 "IS25LP064A-JBLE" H 4850 5200 60  0001 C CNN "Mfg_Part_No"
@@
 F 0 "P11" H 3250 1030 45  0000 L BNN
 F 1 "TFM-105-02-X-DH" V 3500 250 45  0000 L BNN
-F 2 "WheelerLab:TFM-105-02-X-DH" H 3080 1050 20  0001 C CNN
+F 2 "Sci-Bots:TFM-105-02-X-DH" H 3080 1050 20  0001 C CNN
 F 3 "" H 3050 900 60  0000 C CNN
 F 4 "TFM-105-02-L-DH" H 3050 900 60  0001 C CNN "Mfg_Part_No"
@@
 F 0 "C32" H 700 1050 50  0000 L CNN
 F 1 "33uF" V 700 1200 50  0000 L CNN
-F 2 "WheelerLab:SM2917" H 650 1150 50  0001 C CNN
+F 2 "Sci-Bots:SM2917" H 650 1150 50  0001 C CNN
 F 3 "" H 650 1150 50  0000 C CNN
 F 4 "T491D336K020AT" H 650 1150 60  0001 C CNN "Mfg_Part_No"
@@
 F 0 "U1" H 6850 3450 60  0000 C CNN
 F 1 "Teensy_3.2" H 6850 4900 60  0000 C CNN
-F 2 "WheelerLab:Teensy-3.2" H 6950 2900 60  0001 C CNN
+F 2 "Sci-Bots:Teensy-3.2" H 6950 2900 60  0001 C CNN
 F 3 "" H 6950 2900 60  0000 C CNN
 	1    6850 3450
@@
 F 0 "SW1" H 1300 4000 50  0000 C CNN
 F 1 "PROG" H 1300 3800 50  0000 C CNN
-F 2 "WheelerLab:PTS840_GK_SMTR_LFS" H 1300 3900 50  0001 C CNN
+F 2 "Sci-Bots:PTS840_GK_SMTR_LFS" H 1300 3900 50  0001 C CNN
 F 3 "" H 1300 3900 50  0000 C CNN
 F 4 "PTS840 GK SMTR LFS" H 1300 3900 60  0001 C CNN "Mfg_Part_No"

Commit message: Update with kicad-helpers files
Parts:
- C22, C23, C25, C26, C27, C28, C29, C36: symbol C_Small -> Device:C_Small
- C32: symbol CP1 -> Device:CP1
- C33, C34, C37, C38, C9: symbol C -> Device:C
- LED1, LED2: symbol LED -> Device:LED
- R1, R19, R2, R20, R3, R35, R4, R40, R41, R42, R43, R44, R45, R50, R51, R52: symbol R -> Device:R
Connections:
- wire segments 63 -> 83

Commit message: Fix broken symbols and DRC tests
Parts:
- FB1, FB3, FB4, FB5, FB6: symbol FERRITE -> sci-bots:FERRITE
- P1, P10, P2, P5: symbol CONN_01X01 -> Connector_Generic:Conn_01x01
- P11: symbol TFM-105-02-X-DH -> sci-bots:TFM-105-02-X-DH
- P3, P8: symbol CONN_01X03 -> Connector_Generic:Conn_01x03
- P4: symbol CONN_01X02 -> Connector_Generic:Conn_01x02
- P7: symbol CONN_01X04 -> Connector_Generic:Conn_01x04
- SW1: symbol SPST -> sci-bots:SPST
- U1: symbol Teensy_3.2 -> sci-bots:Teensy_3.2
- U10: symbol W25Q64FV -> sci-bots:W25Q64FV
Connections:
- net labels removed: A6, A7
- no-connect marks 9 -> 12

Commit message: Update BOM
Parts:
- C22, C26, C33, C36, C37, C38, C9: MPN (none) -> CL21B104KBCNNNC; Manufacturer (none) -> Samsung
- C23, C25, C28, C29: MPN (none) -> CL21C151JBANNNC; Manufacturer (none) -> Samsung
- C27, C34: MPN (none) -> CC0805KRX7R9BB103; Manufacturer (none) -> Yageo
- C32: MPN (none) -> T491D336K020AT; Manufacturer (none) -> KEMET
- FB1, FB3, FB4, FB5, FB6: MPN (none) -> 742792040; Manufacturer (none) -> Würth Elektronik
- LED1, LED2: MPN (none) -> 150080BS75000; Manufacturer (none) -> Würth Elektronik
- P1, P10, P2, P3, P4, P5, P7, P8, U1: MPN (none) -> DNP; Manufacturer (none) -> DNP
- P11: MPN (none) -> TFM-105-02-L-DH; Manufacturer (none) -> Samtec
- R1: MPN (none) -> RC0805FR-071KL; Manufacturer (none) -> Yageo
- R19, R2, R20, R3, R4: MPN (none) -> RC0805FR-072KL; Manufacturer (none) -> Yageo
- R35: MPN (none) -> RC0805FR-075K1L; Manufacturer (none) -> Yageo
- R40, R41, R50, R51: MPN (none) -> RC0805FR-07150RL; Manufacturer (none) -> Yageo
- R42, R43, R44, R45: MPN (none) -> RC0805FR-0751RL; Manufacturer (none) -> Yageo
- R52: MPN (none) -> RC0805JR-070RL; Manufacturer (none) -> Yageo
- SW1: MPN (none) -> PTS840 GK SMTR LFS; Manufacturer (none) -> C&K Components
- U10: MPN (none) -> IS25LP064A-JBLE; Manufacturer (none) -> ISSI
