File: hv-square-wave-driver.sch (KiCad schematic (older format))
At the start: 15 parts, among them Q5 IRF740BPBF, Q6 IRF740BPBF, U6 NCP5304

Commit message: Add missing schematic diagrams and change some part numbers
Parts:
- removed F1: PTC, Resistors_ThroughHole:Resistor_Vertical_RM5mm, symbol F_Small
- added F1: PTC, Resistors_ThroughHole:Resistor_Vertical_RM5mm, symbol Fuse_Small
Changed lines of the file:
@@
-$EndComp
-$Comp
-L F_Small F1
-U 1 1 58D0BDAD
-P 6400 3950
-F 0 "F1" H 6350 4000 50  0000 L CNN
-F 1 "PTC" H 6350 3850 50  0000 L CNN
-F 2 "Resistors_ThroughHole:Resistor_Vertical_RM5mm" H 6400 3950 50  0001 C CNN
-F 3 "" H 6400 3950 50  0000 C CNN
-F 4 "B59773B120A70" H 6400 3950 60  0001 C CNN "Mfg_Part_No"
-	1    6400 3950
-	1    0    0    -1
 $EndComp
 $Comp
@@
 Wire Wire Line
 	6300 4450 6300 4400
+$Comp
+L Fuse_Small F1
+U 1 1 5931BF6A
+P 6400 3950
+F 0 "F1" H 6400 3890 50  0000 C CNN
+F 1 "PTC" H 6400 4010 50  0000 C CNN
+F 2 "Resistors_ThroughHole:Resistor_Vertical_RM5mm" H 6400 3950 50  0001 C CNN
+F 3 "" H 6400 3950 50  0001 C CNN
+F 4 "B59773B120A70" H 6400 3950 60  0001 C CNN "Mfg_Part_No"
+	1    6400 3950
+	1    0    0    -1
+$EndComp
 $EndSCHEMATC

Commit message: Change part number for ferrites, add *.pos files
Parts:
- FB2: Mfg_Part_No RC0805JR-070RL -> 742792040
Changed lines of the file:
@@
 LIBS:valves
 LIBS:wheelerlab
-LIBS:dropbot_control_board-cache
 EELAYER 25 0
 EELAYER END
@@
 F 2 "Resistors_SMD:R_0805" H 6650 3850 60  0001 C CNN
 F 3 "" H 6650 3850 60  0000 C CNN
-F 4 "RC0805JR-070RL" H 6650 3950 60  0001 C CNN "Mfg_Part_No"
+F 4 "742792040" H 6650 3950 60  0001 C CNN "Mfg_Part_No"
 	1    6650 3950
 	1    0    0    -1

Commit message: Update BOM
2 part numbers (F1 and F2) had typos and updated D4 to a part that
is more commonly available.
Parts:
- F1: Mfg_Part_No B59773B120A70 -> B59773B0120A070
Changed lines of the file:
@@
 F 2 "Resistors_ThroughHole:Resistor_Vertical_RM5mm" H 6400 3950 50  0001 C CNN
 F 3 "" H 6400 3950 50  0001 C CNN
-F 4 "B59773B120A70" H 6400 3950 60  0001 C CNN "Mfg_Part_No"
+F 4 "B59773B0120A070" H 6400 3950 60  0001 C CNN "Mfg_Part_No"
 	1    6400 3950
 	1    0    0    -1

Commit message: Update schematic to use power ports
Changed lines of the file:
@@
 Text Notes 4300 3050 0    60   ~ 0
 HV SQUARE WAVE DRIVER
-Text GLabel 6100 4450 0    60   Input ~ 0
-GND
 $Comp
 L NCP5304 U6
@@
 	-1   0    0    1
 $EndComp
-Text GLabel 4600 3400 0    60   Input ~ 0
-GND
-Text GLabel 4350 4050 0    60   Input ~ 0
-GND
 Text GLabel 6100 3550 1    60   Input ~ 0
 HV
@@
 Text GLabel 4250 3850 0    60   Input ~ 0
 D7/DRIVER_HI
-Text GLabel 4300 3200 0    60   Input ~ 0
-+12V
 $Comp
 L C_Small C4
@@
 	5900 3950 6100 3950
 Wire Wire Line
-	4300 3200 4750 3200
+	4050 3200 4750 3200
 Wire Wire Line
 	6100 4450 6850 4450
@@
 	1    0    0    -1
 $EndComp
+$Comp
+L +12V #PWR031
+U 1 1 5B3C009D
+P 4050 3200
+F 0 "#PWR031" H 4050 3050 50  0001 C CNN
+F 1 "+12V" H 4050 3340 50  0000 C CNN
+F 2 "" H 4050 3200 50  0001 C CNN
+F 3 "" H 4050 3200 50  0001 C CNN
+	1    4050 3200
+	1    0    0    -1
+$EndComp
+Connection ~ 4300 3200
+$Comp
+L GND #PWR032
+U 1 1 5B3C9B2A
+P 4600 3400
+F 0 "#PWR032" H 4600 3150 50  0001 C CNN
+F 1 "GND" H 4600 3250 50  0000 C CNN
+F 2 "" H 4600 3400 50  0001 C CNN
+F 3 "" H 4600 3400 50  0001 C CNN
+	1    4600 3400
+	1    0    0    -1
+$EndComp
+$Comp
+L GND #PWR033
+U 1 1 5B3C9BB4
+P 4350 4400
+F 0 "#PWR033" H 4350 4150 50  0001 C CNN
+F 1 "GND" H 4350 4250 50  0000 C CNN
+F 2 "" H 4350 4400 50  0001 C CNN
+F 3 "" H 4350 4400 50  0001 C CNN
+	1    4350 4400
+	1    0    0    -1
+$EndComp
+$Comp
+L GND #PWR034
+U 1 1 5B3C9C0A
+P 6100 4450
+F 0 "#PWR034" H 6100 4200 50  0001 C CNN
+F 1 "GND" H 6100 4300 50  0000 C CNN
+F 2 "" H 6100 4450 50  0001 C CNN
+F 3 "" H 6100 4450 50  0001 C CNN
+	1    6100 4450
+	1    0    0    -1
+$EndComp
