File: hv-square-wave-driver.sch (KiCad schematic (older format))
At the start: 15 parts, among them Q5 IRF740BPBF, Q6 IRF740BPBF, U6 NCP5304

Commit message: Update with kicad-helpers files
Parts:
- C10, C3, C35, C4: symbol C_Small -> Device:C_Small
- D2, D3: symbol D -> Device:D
- F1: symbol Fuse_Small -> Device:Fuse_Small
- Q5, Q6: symbol Q_NMOS_GDS -> Device:Q_NMOS_GDS
- R18, R21, R22, R37: symbol R -> Device:R
Changed lines of the file:
@@
-EESchema Schematic File Version 2
-LIBS:power
-LIBS:device
-LIBS:transistors
-LIBS:conn
-LIBS:linear
-LIBS:regul
-LIBS:74xx
-LIBS:cmos4000
-LIBS:adc-dac
-LIBS:memory
-LIBS:xilinx
-LIBS:microcontrollers
-LIBS:dsp
-LIBS:microchip
-LIBS:analog_switches
-LIBS:motorola
-LIBS:texas
-LIBS:intel
-LIBS:audio
-LIBS:interface
-LIBS:digital-audio
-LIBS:philips
-LIBS:display
-LIBS:cypress
-LIBS:siliconi
-LIBS:opto
-LIBS:atmel
-LIBS:contrib
-LIBS:valves
-LIBS:sci-bots
-LIBS:dropbot_control_board-cache
-EELAYER 25 0
+EESchema Schematic File Version 4
+EELAYER 30 0
 EELAYER END
 $Descr USLetter 11000 8500
@@
 $EndComp
 $Comp
-L D D2
+L Device:D D2
 U 1 1 58D0BD5A
 P 4900 3200
@@
 $EndComp
 $Comp
-L C_Small C3
+L Device:C_Small C3
 U 1 1 58D0BD61
 P 4600 3300
@@
 HV
 $Comp
-L D D3
+L Device:D D3
 U 1 1 58D0BD6B
 P 4900 4400
@@
 $EndComp
 $Comp
-L R R21
+L Device:R R21
 U 1 1 58D0BD72
 P 5750 3950
@@
 HVAC
 $Comp
-L R R22
+L Device:R R22
 U 1 1 58D0BD7A
 P 6300 4250
@@
 $EndComp
 $Comp
-L Q_NMOS_GDS Q5
+L Device:Q_NMOS_GDS Q5
 U 1 1 58D0BD81
 P 6000 3750
@@
 $EndComp
 $Comp
-L Q_NMOS_GDS Q6
+L Device:Q_NMOS_GDS Q6
 U 1 1 58D0BD88
 P 6000 4150
@@
 D7/DRIVER_HI
 $Comp
-L C_Small C4
+L Device:C_Small C4
 U 1 1 58D0BD91
 P 5550 3500
@@
 $EndComp
 $Comp
-L C_Small C10
+L Device:C_Small C10
 U 1 1 58D0BD98
 P 6200 3950
@@
 $EndComp
 $Comp
-L R R37
+L Device:R R37
 U 1 1 58D0BD9F
 P 5650 3750
@@
 $EndComp
 $Comp
-L R R18
+L Device:R R18
 U 1 1 58D0BDA6
 P 5600 4150
@@
 $EndComp
 $Comp
-L C_Small C35
+L Device:C_Small C35
 U 1 1 58D0BDBA
 P 6850 4350
@@
 	6300 4450 6300 4400
 $Comp
-L Fuse_Small F1
+L Device:Fuse_Small F1
 U 1 1 5931BF6A
 P 6400 3950
@@
 $EndComp
 $Comp
-L +12V #PWR031
+L power:+12V #PWR031
 U 1 1 5B3C009D
 P 4050 3200
@@
 Connection ~ 4300 3200
 $Comp
-L GND #PWR032
+L power:GND #PWR032
 U 1 1 5B3C9B2A
 P 4600 3400
@@
 $EndComp
 $Comp
-L GND #PWR033
+L power:GND #PWR033
 U 1 1 5B3C9BB4
 P 4350 4400
@@
 $EndComp
 $Comp
-L GND #PWR034
+L power:GND #PWR034
 U 1 1 5B3C9C0A
 P 6100 4450

Commit message: Fix broken symbols and DRC tests
Parts:
- FB2: symbol FERRITE -> sci-bots:FERRITE
- U6: symbol NCP5304 -> sci-bots:NCP5304
Connections:
- wire segments 25 -> 30
Changed lines of the file:
@@
 HV SQUARE WAVE DRIVER
 $Comp
-L NCP5304 U6
+L sci-bots:NCP5304 U6
 U 1 1 58D0BD53
 P 4900 3900
@@
 $EndComp
 $Comp
-L FERRITE FB2
+L sci-bots:FERRITE FB2
 U 1 1 58D0BDB4
 P 6650 3950
@@
 	5450 4050 5450 4150
 Wire Wire Line
-	5050 3200 5550 3200
+	5050 3200 5450 3200
 Wire Wire Line
 	4350 3950 4300 3950
@@
 	4350 4400 4350 4050
 Wire Wire Line
-	5550 3600 5550 4400
+	5550 3600 5550 3950
 Connection ~ 5550 3950
 Wire Wire Line
 	5550 3200 5550 3400
-Wire Wire Line
-	5450 3750 5450 3750
 Wire Wire Line
 	5450 3750 5450 3200
 Connection ~ 5450 3200
 Wire Wire Line
-	5450 3950 5600 3950
+	5450 3950 5550 3950
 Wire Wire Line
 	5450 3850 5500 3850
@@
 	5900 3950 6100 3950
 Wire Wire Line
-	4050 3200 4750 3200
-Wire Wire Line
-	6100 4450 6850 4450
+	4050 3200 4300 3200
+Wire Wire Line
+	6100 4450 6300 4450
 Wire Wire Line
 	5750 4150 5800 4150
@@
 	1    0    0    -1
 $EndComp
+Wire Wire Line
+	4600 3200 4750 3200
+Wire Wire Line
+	5550 3950 5550 4400
+Wire Wire Line
+	5550 3950 5600 3950
+Wire Wire Line
+	5450 3200 5550 3200
+Wire Wire Line
+	6300 4450 6850 4450
+Wire Wire Line
+	4300 3200 4600 3200
 $EndSCHEMATC

Commit message: Update BOM
Parts:
- C10, C4: MPN (none) -> C1210C104KCRACTU; Manufacturer (none) -> KEMET
- C3: MPN (none) -> CL21B104KBCNNNC; Manufacturer (none) -> Samsung
- C35: MPN (none) -> DNP; Manufacturer (none) -> DNP
- D2, D3: MPN (none) -> US1J-13-F; Manufacturer (none) -> Diodes Inc.
- F1: MPN (none) -> B59773B0120A070; Manufacturer (none) -> EPCOS
- FB2: MPN (none) -> 742792040; Manufacturer (none) -> Würth Elektronik
- Q5, Q6: MPN (none) -> IRF740BPBF; Manufacturer (none) -> Vishay
- R18, R21, R37: MPN (none) -> RC0805FR-0710RL; Manufacturer (none) -> Yageo
- R22: MPN (none) -> HVCB1206KDL2M00; Manufacturer (none) -> Stackpole Electronics
- U6: MPN (none) -> NCP5304DR2G; Manufacturer (none) -> onsemi

Commit message: Remove "Mfg_Part_No" field (replaced by  "MPN")
Parts:
- C10, C4: Mfg_Part_No C1210C104KCRACTU -> (none)
- C3: Mfg_Part_No CL21B104KBCNNNC -> (none)
- D2, D3: Mfg_Part_No US1J-13-F -> (none)
- F1: Mfg_Part_No B59773B0120A070 -> (none)
- FB2: Mfg_Part_No 742792040 -> (none)
- Q5, Q6: Mfg_Part_No IRF740BPBF -> (none)
- R18, R21, R37: Mfg_Part_No RC0805FR-0710RL -> (none)
- R22: Mfg_Part_No HVCB1206KDL2M00 -> (none)
- U6: Mfg_Part_No NCP5304DR2G -> (none)
Changed lines of the file:
@@
 F 4 "NCP5304DR2G" H 4900 4300 50 0001 C CNN "MPN"
 F 5 "onsemi" H 4900 4300 50 0001 C CNN "Manufacturer"
-F 6 "NCP5304DR2G" H 4900 3900 60 0001 C CNN "Mfg_Part_No"
 	1    4900 3900
 	1    0    0    -1
@@
 F 4 "US1J-13-F" H 4900 3400 50 0001 C CNN "MPN"
 F 5 "Diodes Inc." H 4900 3400 50 0001 C CNN "Manufacturer"
-F 6 "US1J-13-F" H 4900 3200 60 0001 C CNN "Mfg_Part_No"
 	1    4900 3200
 	-1   0    0    1
@@
 F 4 "CL21B104KBCNNNC" H 4750 3350 50 0001 C CNN "MPN"
 F 5 "Samsung" H 4750 3350 50 0001 C CNN "Manufacturer"
-F 6 "CL21B104KBCNNNC" H 4600 3300 60 0001 C CNN "Mfg_Part_No"
 	1    4600 3300
 	-1   0    0    1
@@
 F 4 "US1J-13-F" H 4900 4600 50 0001 C CNN "MPN"
 F 5 "Diodes Inc." H 4900 4600 50 0001 C CNN "Manufacturer"
-F 6 "US1J-13-F" H 4900 4400 60 0001 C CNN "Mfg_Part_No"
 	1    4900 4400
 	-1   0    0    1
@@
 F 4 "RC0805FR-0710RL" H 5830 4050 50 0001 C CNN "MPN"
 F 5 "Yageo" H 5830 4050 50 0001 C CNN "Manufacturer"
-F 6 "RC0805FR-0710RL" H 5750 3950 60 0001 C CNN "Mfg_Part_No"
 	1    5750 3950
 	0    1    1    0
@@
 F 4 "HVCB1206KDL2M00" H 6400 4300 50 0001 C CNN "MPN"
 F 5 "Stackpole Electronics" H 6400 4300 50 0001 C CNN "Manufacturer"
-F 6 "HVCB1206KDL2M00" H 6300 4250 60 0001 C CNN "Mfg_Part_No"
 	1    6300 4250
 	1    0    0    -1
@@
 F 4 "IRF740BPBF" H 6000 4000 50 0001 C CNN "MPN"
 F 5 "Vishay" H 6000 4000 50 0001 C CNN "Manufacturer"
-F 6 "IRF740BPBF" H 6000 3750 60 0001 C CNN "Mfg_Part_No"
 	1    6000 3750
 	1    0    0    -1
@@
 F 4 "IRF740BPBF" H 5900 4300 50 0001 C CNN "MPN"
 F 5 "Vishay" H 5900 4300 50 0001 C CNN "Manufacturer"
-F 6 "IRF740BPBF" H 6000 4150 60 0001 C CNN "Mfg_Part_No"
 	1    6000 4150
 	1    0    0    -1
@@
 F 4 "C1210C104KCRACTU" H 5400 3700 50 0001 C CNN "MPN"
 F 5 "KEMET" H 5400 3700 50 0001 C CNN "Manufacturer"
-F 6 "C1210C104KCRACTU" H 5550 3500 60 0001 C CNN "Mfg_Part_No"
 	1    5550 3500
 	-1   0    0    1
@@
 F 4 "C1210C104KCRACTU" H 6100 4000 50 0001 C CNN "MPN"
 F 5 "KEMET" H 6100 4000 50 0001 C CNN "Manufacturer"
-F 6 "C1210C104KCRACTU" H 6200 3950 60 0001 C CNN "Mfg_Part_No"
 	1    6200 3950
 	0    -1   -1   0
@@
 F 4 "RC0805FR-0710RL" H 5730 3850 50 0001 C CNN "MPN"
 F 5 "Yageo" H 5730 3850 50 0001 C CNN "Manufacturer"
-F 6 "RC0805FR-0710RL" H 5650 3750 60 0001 C CNN "Mfg_Part_No"
 	1    5650 3750
 	0    1    1    0
@@
 F 4 "RC0805FR-0710RL" H 5680 4250 50 0001 C CNN "MPN"
 F 5 "Yageo" H 5680 4250 50 0001 C CNN "Manufacturer"
-F 6 "RC0805FR-0710RL" H 5600 4150 60 0001 C CNN "Mfg_Part_No"
 	1    5600 4150
 	0    1    1    0
@@
 F 4 "742792040" H 6600 4150 50 0001 C CNN "MPN"
 F 5 "Würth Elektronik" H 6600 4150 50 0001 C CNN "Manufacturer"
-F 6 "742792040" H 6650 3950 60 0001 C CNN "Mfg_Part_No"
 	1    6650 3950
 	1    0    0    -1
@@
 F 4 "B59773B0120A070" H 6400 3990 50 0001 C CNN "MPN"
 F 5 "EPCOS" H 6400 3990 50 0001 C CNN "Manufacturer"
-F 6 "B59773B0120A070" H 6400 3950 60 0001 C CNN "Mfg_Part_No"
 	1    6400 3950
 	1    0    0    -1
