File: on-board-calibration.sch (KiCad schematic (older format))
At the start: 10 parts, among them U7 DPST (2 Form A), 350V, U8 DPST (2 Form A), 350V

Commit message: Fix feedback and on-board calibration and move USB
Parts:
- removed C14: 100pF, Capacitors_SMD:C_0805, symbol C
- added R31, R32, R55: 5.1k, Resistors_SMD:R_0805, symbol R
- added R54, R56: 200, Resistors_SMD:R_0805, symbol R
- added U12: DPST (2 Form A), 350V, SMD_Packages:DIP-8_SMD, symbol AQW216
- C15: value 1nF -> 100pF; Mfg_Part_No C2012C0G2E102J085AA -> CL21C100JECNNWC
Connections:
- net labels added: +3.3V
- net labels removed: D3
- wire segments 15 -> 20
Other:
- note added: "C12-14 should be\nrated for >100V"
- note removed: "C12-15 should be\nrated for >100V"

Commit message: Add missing schematic diagrams and change some part numbers
Parts:
- C12: value 1pF -> 10pF; Mfg_Part_No CBR08C109CAGAC -> CL21C100JECNNWC
- C13: value 10pF -> 100pF
- C14: renamed from C15; value 100pF -> 470pF; Mfg_Part_No CL21C100JECNNWC -> CL21C471JDFNNWG
Changed lines of the file:
@@
 P 4800 4650
 F 0 "C12" H 4825 4750 50  0000 L CNN
-F 1 "1pF" H 4825 4550 50  0000 L CNN
+F 1 "10pF" H 4825 4550 50  0000 L CNN
 F 2 "Capacitors_SMD:C_0805" H 4838 4500 50  0001 C CNN
 F 3 "" H 4800 4650 50  0000 C CNN
-F 4 "CBR08C109CAGAC" H 4800 4650 60  0001 C CNN "Mfg_Part_No"
+F 4 "CL21C100JECNNWC" H 4800 4650 60  0001 C CNN "Mfg_Part_No"
 	1    4800 4650
 	1    0    0    -1
@@
 P 5550 4650
 F 0 "C13" H 5575 4750 50  0000 L CNN
-F 1 "10pF" H 5575 4550 50  0000 L CNN
+F 1 "100pF" H 5575 4550 50  0000 L CNN
 F 2 "Capacitors_SMD:C_0805" H 5588 4500 50  0001 C CNN
 F 3 "" H 5550 4650 50  0000 C CNN
@@
 VOUT
 $Comp
-L C C15
+L C C14
 U 1 1 591E7390
 P 6300 4650
-F 0 "C15" H 6325 4750 50  0000 L CNN
-F 1 "100pF" H 6325 4550 50  0000 L CNN
+F 0 "C14" H 6325 4750 50  0000 L CNN
+F 1 "470pF" H 6325 4550 50  0000 L CNN
 F 2 "Capacitors_SMD:C_0805" H 6338 4500 50  0001 C CNN
 F 3 "" H 6300 4650 50  0000 C CNN
-F 4 "CL21C100JECNNWC" H 6300 4650 60  0001 C CNN "Mfg_Part_No"
+F 4 "CL21C471JDFNNWG" H 6300 4650 60  0001 C CNN "Mfg_Part_No"
 	1    6300 4650
 	1    0    0    -1

Commit message: Improve layout/stability of boost converter, etc.
* improve layout/stability of boost converter
* enable on board calibration without HVOE
* add decoupling cap to 0.6V reference
* fix footprint for U10
* add programming wire
Parts:
- C13: Mfg_Part_No CL21C100JECNNWC -> CL21C101JECNNWC
- R24, R28, R29, R30, R54, R56: value 200 -> 150; Mfg_Part_No RC0805FR-07200RL -> RC0805FR-07150RL
Connections:
- net labels added: HVAC
- net labels removed: VOUT
Changed lines of the file:
@@
 LIBS:valves
 LIBS:wheelerlab
+LIBS:dropbot_control_board-cache
 EELAYER 25 0
 EELAYER END
@@
 Sheet 3 7
 Title "DropBot control board"
-Date "2017-05-17"
-Rev "3.5"
+Date "2017-06-19"
+Rev "3.6"
 Comp "Sci-Bots Inc."
 Comment1 ""
@@
 $EndComp
 Text GLabel 5050 4300 3    60   Input ~ 0
-VOUT
+HVAC
 Text GLabel 4850 3050 2    60   Input ~ 0
 D0
@@
 P 4550 3350
 F 0 "R24" V 4630 3350 50  0000 C CNN
-F 1 "200" V 4550 3350 50  0000 C CNN
+F 1 "150" V 4550 3350 50  0000 C CNN
 F 2 "Resistors_SMD:R_0805" V 4480 3350 50  0001 C CNN
 F 3 "" H 4550 3350 50  0000 C CNN
-F 4 "RC0805FR-07200RL" H 4550 3350 60  0001 C CNN "Mfg_Part_No"
+F 4 "RC0805FR-07150RL" H 4550 3350 60  0001 C CNN "Mfg_Part_No"
 	1    4550 3350
 	1    0    0    -1
@@
 P 5050 3350
 F 0 "R28" V 5130 3350 50  0000 C CNN
-F 1 "200" V 5050 3350 50  0000 C CNN
+F 1 "150" V 5050 3350 50  0000 C CNN
 F 2 "Resistors_SMD:R_0805" V 4980 3350 50  0001 C CNN
 F 3 "" H 5050 3350 50  0000 C CNN
-F 4 "RC0805FR-07200RL" H 5050 3350 60  0001 C CNN "Mfg_Part_No"
+F 4 "RC0805FR-07150RL" H 5050 3350 60  0001 C CNN "Mfg_Part_No"
 	1    5050 3350
 	1    0    0    -1
@@
 P 5300 3350
 F 0 "R29" V 5380 3350 50  0000 C CNN
-F 1 "200" V 5300 3350 50  0000 C CNN
+F 1 "150" V 5300 3350 50  0000 C CNN
 F 2 "Resistors_SMD:R_0805" V 5230 3350 50  0001 C CNN
 F 3 "" H 5300 3350 50  0000 C CNN
-F 4 "RC0805FR-07200RL" H 5300 3350 60  0001 C CNN "Mfg_Part_No"
+F 4 "RC0805FR-07150RL" H 5300 3350 60  0001 C CNN "Mfg_Part_No"
 	1    5300 3350
 	1    0    0    -1
@@
 P 5800 3350
 F 0 "R30" V 5880 3350 50  0000 C CNN
-F 1 "200" V 5800 3350 50  0000 C CNN
+F 1 "150" V 5800 3350 50  0000 C CNN
 F 2 "Resistors_SMD:R_0805" V 5730 3350 50  0001 C CNN
 F 3 "" H 5800 3350 50  0000 C CNN
-F 4 "RC0805FR-07200RL" H 5800 3350 60  0001 C CNN "Mfg_Part_No"
+F 4 "RC0805FR-07150RL" H 5800 3350 60  0001 C CNN "Mfg_Part_No"
 	1    5800 3350
 	1    0    0    -1
@@
 F 2 "Capacitors_SMD:C_0805" H 5588 4500 50  0001 C CNN
 F 3 "" H 5550 4650 50  0000 C CNN
-F 4 "CL21C100JECNNWC" H 5550 4650 60  0001 C CNN "Mfg_Part_No"
+F 4 "CL21C101JECNNWC" H 5550 4650 60  0001 C CNN "Mfg_Part_No"
 	1    5550 4650
 	1    0    0    -1
@@
 GND
 Text GLabel 5800 4300 3    60   Input ~ 0
-VOUT
+HVAC
 Wire Wire Line
 	5050 3150 6850 3150
@@
 P 6050 3350
 F 0 "R54" V 6130 3350 50  0000 C CNN
-F 1 "200" V 6050 3350 50  0000 C CNN
+F 1 "150" V 6050 3350 50  0000 C CNN
 F 2 "Resistors_SMD:R_0805" V 5980 3350 50  0001 C CNN
 F 3 "" H 6050 3350 50  0000 C CNN
-F 4 "RC0805FR-07200RL" H 6050 3350 60  0001 C CNN "Mfg_Part_No"
+F 4 "RC0805FR-07150RL" H 6050 3350 60  0001 C CNN "Mfg_Part_No"
 	1    6050 3350
 	1    0    0    -1
@@
 P 6550 3350
 F 0 "R56" V 6630 3350 50  0000 C CNN
-F 1 "200" V 6550 3350 50  0000 C CNN
+F 1 "150" V 6550 3350 50  0000 C CNN
 F 2 "Resistors_SMD:R_0805" V 6480 3350 50  0001 C CNN
 F 3 "" H 6550 3350 50  0000 C CNN
-F 4 "RC0805FR-07200RL" H 6550 3350 60  0001 C CNN "Mfg_Part_No"
+F 4 "RC0805FR-07150RL" H 6550 3350 60  0001 C CNN "Mfg_Part_No"
 	1    6550 3350
 	1    0    0    -1
@@
 GND
 Text GLabel 6550 4300 3    60   Input ~ 0
-VOUT
+HVAC
 $Comp
 L C C14

Commit message: Change EEPROM and swap 150 Ohm resisotors for 100...
Change EEPROM and swap 150 Ohm resisotors for 100 resistors
driving the PhotoMOS switches.
Parts:
- R24, R28, R29, R30, R54, R56: value 150 -> 100; Mfg_Part_No RC0805FR-07150RL -> RC0805FR-07100RL
Changed lines of the file:
@@
 P 4550 3350
 F 0 "R24" V 4630 3350 50  0000 C CNN
-F 1 "150" V 4550 3350 50  0000 C CNN
+F 1 "100" V 4550 3350 50  0000 C CNN
 F 2 "Resistors_SMD:R_0805" V 4480 3350 50  0001 C CNN
 F 3 "" H 4550 3350 50  0000 C CNN
-F 4 "RC0805FR-07150RL" H 4550 3350 60  0001 C CNN "Mfg_Part_No"
+F 4 "RC0805FR-07100RL" H 4550 3350 60  0001 C CNN "Mfg_Part_No"
 	1    4550 3350
 	1    0    0    -1
@@
 P 5050 3350
 F 0 "R28" V 5130 3350 50  0000 C CNN
-F 1 "150" V 5050 3350 50  0000 C CNN
+F 1 "100" V 5050 3350 50  0000 C CNN
 F 2 "Resistors_SMD:R_0805" V 4980 3350 50  0001 C CNN
 F 3 "" H 5050 3350 50  0000 C CNN
-F 4 "RC0805FR-07150RL" H 5050 3350 60  0001 C CNN "Mfg_Part_No"
+F 4 "RC0805FR-07100RL" H 5050 3350 60  0001 C CNN "Mfg_Part_No"
 	1    5050 3350
 	1    0    0    -1
@@
 P 5300 3350
 F 0 "R29" V 5380 3350 50  0000 C CNN
-F 1 "150" V 5300 3350 50  0000 C CNN
+F 1 "100" V 5300 3350 50  0000 C CNN
 F 2 "Resistors_SMD:R_0805" V 5230 3350 50  0001 C CNN
 F 3 "" H 5300 3350 50  0000 C CNN
-F 4 "RC0805FR-07150RL" H 5300 3350 60  0001 C CNN "Mfg_Part_No"
+F 4 "RC0805FR-07100RL" H 5300 3350 60  0001 C CNN "Mfg_Part_No"
 	1    5300 3350
 	1    0    0    -1
@@
 P 5800 3350
 F 0 "R30" V 5880 3350 50  0000 C CNN
-F 1 "150" V 5800 3350 50  0000 C CNN
+F 1 "100" V 5800 3350 50  0000 C CNN
 F 2 "Resistors_SMD:R_0805" V 5730 3350 50  0001 C CNN
 F 3 "" H 5800 3350 50  0000 C CNN
-F 4 "RC0805FR-07150RL" H 5800 3350 60  0001 C CNN "Mfg_Part_No"
+F 4 "RC0805FR-07100RL" H 5800 3350 60  0001 C CNN "Mfg_Part_No"
 	1    5800 3350
 	1    0    0    -1
@@
 P 6050 3350
 F 0 "R54" V 6130 3350 50  0000 C CNN
-F 1 "150" V 6050 3350 50  0000 C CNN
+F 1 "100" V 6050 3350 50  0000 C CNN
 F 2 "Resistors_SMD:R_0805" V 5980 3350 50  0001 C CNN
 F 3 "" H 6050 3350 50  0000 C CNN
-F 4 "RC0805FR-07150RL" H 6050 3350 60  0001 C CNN "Mfg_Part_No"
+F 4 "RC0805FR-07100RL" H 6050 3350 60  0001 C CNN "Mfg_Part_No"
 	1    6050 3350
 	1    0    0    -1
@@
 P 6550 3350
 F 0 "R56" V 6630 3350 50  0000 C CNN
-F 1 "150" V 6550 3350 50  0000 C CNN
+F 1 "100" V 6550 3350 50  0000 C CNN
 F 2 "Resistors_SMD:R_0805" V 6480 3350 50  0001 C CNN
 F 3 "" H 6550 3350 50  0000 C CNN
-F 4 "RC0805FR-07150RL" H 6550 3350 60  0001 C CNN "Mfg_Part_No"
+F 4 "RC0805FR-07100RL" H 6550 3350 60  0001 C CNN "Mfg_Part_No"
 	1    6550 3350
 	1    0    0    -1

Commit message: Update schematic to use power ports
Connections:
- wire segments 20 -> 21
Changed lines of the file:
@@
 	0    1    1    0
 $EndComp
-Text GLabel 4550 3050 0    60   Input ~ 0
-GND
 $Comp
 L C C12
@@
 Wire Wire Line
 	4750 4300 4850 4300
-Text GLabel 4550 4300 3    60   Input ~ 0
-GND
 Wire Wire Line
 	4800 4300 4800 4500
@@
 	0    1    1    0
 $EndComp
-Text GLabel 6850 3150 2    60   Input ~ 0
-+3.3V
 Wire Wire Line
 	4550 3050 4550 3200
@@
 Wire Wire Line
 	5600 3500 5500 3500
-Text GLabel 5300 4300 3    60   Input ~ 0
-GND
 Text GLabel 5800 4300 3    60   Input ~ 0
 HVAC
@@
 	6550 3200 6550 3150
 Connection ~ 6550 3150
-Text GLabel 6050 4300 3    60   Input ~ 0
-GND
 Text GLabel 6550 4300 3    60   Input ~ 0
 HVAC
@@
 Wire Wire Line
 	6350 3500 6250 3500
+$Comp
+L +3.3V #PWR026
+U 1 1 5B3BEE57
+P 6850 3150
+F 0 "#PWR026" H 6850 3000 50  0001 C CNN
+F 1 "+3.3V" H 6850 3290 50  0000 C CNN
+F 2 "" H 6850 3150 50  0001 C CNN
+F 3 "" H 6850 3150 50  0001 C CNN
+	1    6850 3150
+	1    0    0    -1
+$EndComp
+$Comp
+L GND #PWR027
+U 1 1 5B3C828A
+P 4400 3050
+F 0 "#PWR027" H 4400 2800 50  0001 C CNN
+F 1 "GND" H 4400 2900 50  0000 C CNN
+F 2 "" H 4400 3050 50  0001 C CNN
+F 3 "" H 4400 3050 50  0001 C CNN
+	1    4400 3050
+	1    0    0    -1
+$EndComp
+Wire Wire Line
+	4400 3050 4550 3050
+$Comp
+L GND #PWR028
+U 1 1 5B3C84B2
+P 4550 4300
+F 0 "#PWR028" H 4550 4050 50  0001 C CNN
+F 1 "GND" H 4550 4150 50  0000 C CNN
+F 2 "" H 4550 4300 50  0001 C CNN
+F 3 "" H 4550 4300 50  0001 C CNN
+	1    4550 4300
+	1    0    0    -1
+$EndComp
+$Comp
+L GND #PWR029
+U 1 1 5B3C8624
+P 5300 4300
+F 0 "#PWR029" H 5300 4050 50  0001 C CNN
+F 1 "GND" H 5300 4150 50  0000 C CNN
+F 2 "" H 5300 4300 50  0001 C CNN
+F 3 "" H 5300 4300 50  0001 C CNN
+	1    5300 4300
+	1    0    0    -1
+$EndComp
+$Comp
+L GND #PWR030
+U 1 1 5B3C8721
+P 6050 4300
+F 0 "#PWR030" H 6050 4050 50  0001 C CNN
+F 1 "GND" H 6050 4150 50  0000 C CNN
+F 2 "" H 6050 4300 50  0001 C CNN
+F 3 "" H 6050 4300 50  0001 C CNN
+	1    6050 4300
+	1    0    0    -1
+$EndComp
 $EndSCHEMATC
