File: on-board-calibration.sch (KiCad schematic (older format))
At the start: 15 parts, among them U12 DPST (2 Form A), 350V, U7 DPST (2 Form A), 350V, U8 DPST (2 Form A), 350V

Commit message: Update with kicad-helpers files
Parts:
- C12, C13, C14: symbol C -> Device:C
- R24, R28, R29, R30, R31, R32, R54, R55, R56: symbol R -> Device:R
Changed lines of the file:
@@
-EESchema Schematic File Version 2
-LIBS:power
-LIBS:device
-LIBS:transistors
-LIBS:conn
-LIBS:linear
-LIBS:regul
-LIBS:74xx
-LIBS:cmos4000
-LIBS:adc-dac
-LIBS:memory
-LIBS:xilinx
-LIBS:microcontrollers
-LIBS:dsp
-LIBS:microchip
-LIBS:analog_switches
-LIBS:motorola
-LIBS:texas
-LIBS:intel
-LIBS:audio
-LIBS:interface
-LIBS:digital-audio
-LIBS:philips
-LIBS:display
-LIBS:cypress
-LIBS:siliconi
-LIBS:opto
-LIBS:atmel
-LIBS:contrib
-LIBS:valves
-LIBS:sci-bots
-LIBS:dropbot_control_board-cache
-EELAYER 25 0
+EESchema Schematic File Version 4
+EELAYER 30 0
 EELAYER END
 $Descr USLetter 11000 8500
@@
 $EndComp
 $Comp
-L C C12
+L Device:C C12
 U 1 1 57E388D0
 P 4800 4650
@@
 D1
 $Comp
-L R R24
+L Device:R R24
 U 1 1 57E388D5
 P 4550 3350
@@
 $EndComp
 $Comp
-L R R28
+L Device:R R28
 U 1 1 57E388D6
 P 5050 3350
@@
 $EndComp
 $Comp
-L R R29
+L Device:R R29
 U 1 1 57E388D7
 P 5300 3350
@@
 $EndComp
 $Comp
-L R R30
+L Device:R R30
 U 1 1 57E388D8
 P 5800 3350
@@
 	4750 3500 4850 3500
 $Comp
-L C C13
+L Device:C C13
 U 1 1 57E388D1
 P 5550 4650
@@
 Connection ~ 4800 4800
 $Comp
-L R R31
+L Device:R R31
 U 1 1 591C6194
 P 4700 3050
@@
 	5050 3200 5050 3150
 $Comp
-L R R32
+L Device:R R32
 U 1 1 591C662A
 P 5450 3050
@@
 $EndComp
 $Comp
-L R R54
+L Device:R R54
 U 1 1 591E724C
 P 6050 3350
@@
 $EndComp
 $Comp
-L R R56
+L Device:R R56
 U 1 1 591E72A2
 P 6550 3350
@@
 HVAC
 $Comp
-L C C14
+L Device:C C14
 U 1 1 591E7390
 P 6300 4650
@@
 D2
 $Comp
-L R R55
+L Device:R R55
 U 1 1 591E74B6
 P 6200 3050
@@
 	6350 3500 6250 3500
 $Comp
-L +3.3V #PWR026
+L power:+3.3V #PWR026
 U 1 1 5B3BEE57
 P 6850 3150
@@
 $EndComp
 $Comp
-L GND #PWR027
+L power:GND #PWR027
 U 1 1 5B3C828A
 P 4400 3050
@@
 	4400 3050 4550 3050
 $Comp
-L GND #PWR028
+L power:GND #PWR028
 U 1 1 5B3C84B2
 P 4550 4300
@@
 $EndComp
 $Comp
-L GND #PWR029
+L power:GND #PWR029
 U 1 1 5B3C8624
 P 5300 4300
@@
 $EndComp
 $Comp
-L GND #PWR030
+L power:GND #PWR030
 U 1 1 5B3C8721
 P 6050 4300

Commit message: Fix broken symbols and DRC tests
Parts:
- U12, U7, U8: symbol AQW216 -> sci-bots:AQW214
Connections:
- wire segments 21 -> 28
Changed lines of the file:
@@
 $EndDescr
 $Comp
-L AQW216 U7
+L sci-bots:AQW214 U7
 U 1 1 57E388CE
 P 4800 3900
@@
 $EndComp
 $Comp
-L AQW216 U8
+L sci-bots:AQW214 U8
 U 1 1 57E388CF
 P 5550 3900
@@
 $EndComp
 Wire Wire Line
-	4750 4300 4850 4300
+	4750 4300 4800 4300
 Wire Wire Line
 	4800 4300 4800 4500
 Connection ~ 4800 4300
 Wire Wire Line
-	4550 4800 6300 4800
-Wire Wire Line
-	5500 4300 5600 4300
+	4550 4800 4800 4800
+Wire Wire Line
+	5500 4300 5550 4300
 Wire Wire Line
 	5550 4500 5550 4300
@@
 HVAC
 Wire Wire Line
-	5050 3150 6850 3150
+	5050 3150 5800 3150
 Text GLabel 5300 3050 0    60   Input ~ 0
 GND
 $Comp
-L AQW216 U12
+L sci-bots:AQW214 U12
 U 1 1 591E71DB
 P 6300 3900
@@
 $EndComp
 Wire Wire Line
-	6250 4300 6350 4300
+	6250 4300 6300 4300
 Wire Wire Line
 	6300 4500 6300 4300
@@
 	1    0    0    -1
 $EndComp
+Wire Wire Line
+	4800 4300 4850 4300
+Wire Wire Line
+	5550 4300 5600 4300
+Wire Wire Line
+	4800 4800 5550 4800
+Wire Wire Line
+	5800 3150 6550 3150
+Wire Wire Line
+	6550 3150 6850 3150
+Wire Wire Line
+	6300 4300 6350 4300
+Wire Wire Line
+	5550 4800 6300 4800
 $EndSCHEMATC

Commit message: Update BOM
Parts:
- C12: MPN (none) -> CL21C100JECNNWC; Manufacturer (none) -> Samsung
- C13: MPN (none) -> CL21C101JECNNWC; Manufacturer (none) -> Samsung
- C14: MPN (none) -> CL21C471JDFNNWG; Manufacturer (none) -> Samsung
- R24, R28, R29, R30, R54, R56: MPN (none) -> RC0805FR-07100RL; Manufacturer (none) -> Yageo
- R31, R32, R55: MPN (none) -> RC0805FR-075K1L; Manufacturer (none) -> Yageo
- U12, U7, U8: MPN (none) -> TLP227G-2(TP1,N,F); Manufacturer (none) -> Toshiba

Commit message: Remove "Mfg_Part_No" field (replaced by  "MPN")
Parts:
- C12: Mfg_Part_No CL21C100JECNNWC -> (none)
- C13: Mfg_Part_No CL21C101JECNNWC -> (none)
- C14: Mfg_Part_No CL21C471JDFNNWG -> (none)
- R24, R28, R29, R30, R54, R56: Mfg_Part_No RC0805FR-07100RL -> (none)
- R31, R32, R55: Mfg_Part_No RC0805FR-075K1L -> (none)
- U12, U7, U8: Mfg_Part_No TLP227G-2(TP1,N,F) -> (none)
Changed lines of the file:
@@
 F 4 "TLP227G-2(TP1,N,F)" H 4800 3550 50 0001 C CNN "MPN"
 F 5 "Toshiba" H 4800 3550 50 0001 C CNN "Manufacturer"
-F 6 "TLP227G-2(TP1,N,F)" H 4800 3900 60 0001 C CNN "Mfg_Part_No"
 	1    4800 3900
 	0    1    1    0
@@
 F 4 "TLP227G-2(TP1,N,F)" H 5550 4350 50 0001 C CNN "MPN"
 F 5 "Toshiba" H 5550 4350 50 0001 C CNN "Manufacturer"
-F 6 "TLP227G-2(TP1,N,F)" H 5550 3900 60 0001 C CNN "Mfg_Part_No"
 	1    5550 3900
 	0    1    1    0
@@
 F 4 "CL21C100JECNNWC" H 4825 4850 50 0001 C CNN "MPN"
 F 5 "Samsung" H 4825 4850 50 0001 C CNN "Manufacturer"
-F 6 "CL21C100JECNNWC" H 4800 4650 60 0001 C CNN "Mfg_Part_No"
 	1    4800 4650
 	1    0    0    -1
@@
 F 4 "RC0805FR-07100RL" H 4630 3450 50 0001 C CNN "MPN"
 F 5 "Yageo" H 4630 3450 50 0001 C CNN "Manufacturer"
-F 6 "RC0805FR-07100RL" H 4550 3350 60 0001 C CNN "Mfg_Part_No"
 	1    4550 3350
 	1    0    0    -1
@@
 F 4 "RC0805FR-07100RL" H 5130 3450 50 0001 C CNN "MPN"
 F 5 "Yageo" H 5130 3450 50 0001 C CNN "Manufacturer"
-F 6 "RC0805FR-07100RL" H 5050 3350 60 0001 C CNN "Mfg_Part_No"
 	1    5050 3350
 	1    0    0    -1
@@
 F 4 "RC0805FR-07100RL" H 5380 3450 50 0001 C CNN "MPN"
 F 5 "Yageo" H 5380 3450 50 0001 C CNN "Manufacturer"
-F 6 "RC0805FR-07100RL" H 5300 3350 60 0001 C CNN "Mfg_Part_No"
 	1    5300 3350
 	1    0    0    -1
@@
 F 4 "RC0805FR-07100RL" H 5880 3450 50 0001 C CNN "MPN"
 F 5 "Yageo" H 5880 3450 50 0001 C CNN "Manufacturer"
-F 6 "RC0805FR-07100RL" H 5800 3350 60 0001 C CNN "Mfg_Part_No"
 	1    5800 3350
 	1    0    0    -1
@@
 F 4 "CL21C101JECNNWC" H 5575 4850 50 0001 C CNN "MPN"
 F 5 "Samsung" H 5575 4850 50 0001 C CNN "Manufacturer"
-F 6 "CL21C101JECNNWC" H 5550 4650 60 0001 C CNN "Mfg_Part_No"
 	1    5550 4650
 	1    0    0    -1
@@
 F 4 "RC0805FR-075K1L" H 4600 3150 50 0001 C CNN "MPN"
 F 5 "Yageo" H 4600 3150 50 0001 C CNN "Manufacturer"
-F 6 "RC0805FR-075K1L" H 4700 3050 60 0001 C CNN "Mfg_Part_No"
 	1    4700 3050
 	0    1    1    0
@@
 F 4 "RC0805FR-075K1L" H 5350 3150 50 0001 C CNN "MPN"
 F 5 "Yageo" H 5350 3150 50 0001 C CNN "Manufacturer"
-F 6 "RC0805FR-075K1L" H 5450 3050 60 0001 C CNN "Mfg_Part_No"
 	1    5450 3050
 	0    1    1    0
@@
 F 4 "TLP227G-2(TP1,N,F)" H 6300 4350 50 0001 C CNN "MPN"
 F 5 "Toshiba" H 6300 4350 50 0001 C CNN "Manufacturer"
-F 6 "TLP227G-2(TP1,N,F)" H 6300 3900 60 0001 C CNN "Mfg_Part_No"
 	1    6300 3900
 	0    1    1    0
@@
 F 4 "RC0805FR-07100RL" H 6130 3450 50 0001 C CNN "MPN"
 F 5 "Yageo" H 6130 3450 50 0001 C CNN "Manufacturer"
-F 6 "RC0805FR-07100RL" H 6050 3350 60 0001 C CNN "Mfg_Part_No"
 	1    6050 3350
 	1    0    0    -1
@@
 F 4 "RC0805FR-07100RL" H 6630 3450 50 0001 C CNN "MPN"
 F 5 "Yageo" H 6630 3450 50 0001 C CNN "Manufacturer"
-F 6 "RC0805FR-07100RL" H 6550 3350 60 0001 C CNN "Mfg_Part_No"
 	1    6550 3350
 	1    0    0    -1
@@
 F 4 "CL21C471JDFNNWG" H 6325 4850 50 0001 C CNN "MPN"
 F 5 "Samsung" H 6325 4850 50 0001 C CNN "Manufacturer"
-F 6 "CL21C471JDFNNWG" H 6300 4650 60 0001 C CNN "Mfg_Part_No"
 	1    6300 4650
 	1    0    0    -1
@@
 F 4 "RC0805FR-075K1L" H 6100 3150 50 0001 C CNN "MPN"
 F 5 "Yageo" H 6100 3150 50 0001 C CNN "Manufacturer"
-F 6 "RC0805FR-075K1L" H 6200 3050 60 0001 C CNN "Mfg_Part_No"
 	1    6200 3050
 	0    1    1    0
