File: usb-pass-through.sch (KiCad schematic (older format))
At the start: 7 parts, among them P6 USB_B, P9 USB_A

Commit message: Add missing schematic diagrams and change some part numbers
Changed lines of the file:
@@
 Comment4 ""
 $EndDescr
-$Comp
-L USB_A P9
-U 1 1 58AEE5D3
-P 5200 4700
-F 0 "P9" H 5400 4500 50  0000 C CNN
-F 1 "USB_A" H 5150 4900 50  0000 C CNN
-F 2 "WheelerLab:AU-Y1006" V 5150 4600 50  0001 C CNN
-F 3 "" V 5150 4600 50  0000 C CNN
-F 4 "AU-Y1006" H 5200 4700 60  0001 C CNN "Mfg_Part_No"
-	1    5200 4700
-	1    0    0    -1
-$EndComp
-$Comp
-L USB_B P6
-U 1 1 58AEE77B
-P 5200 2900
-F 0 "P6" H 5400 2700 50  0000 C CNN
-F 1 "USB_B" H 5150 3100 50  0000 C CNN
-F 2 "WheelerLab:1734346-1" V 5150 2800 50  0001 C CNN
-F 3 "" V 5150 2800 50  0000 C CNN
-F 4 "1734346-1" H 5200 2900 60  0001 C CNN "Mfg_Part_No"
-	1    5200 2900
-	1    0    0    -1
-$EndComp
-Text GLabel 5500 5000 2    60   Input ~ 0
+Text GLabel 4800 5100 0    60   Input ~ 0
 GND
-Text Notes 4450 2600 0    60   ~ 0
+Text Notes 4450 2450 0    60   ~ 0
 USB PASSTHROUGH\nIncludes ESD protection and\nEMI suppression (See Wurth\nElectronics App Note ANP002C).
-Text GLabel 5700 2800 2    60   Input ~ 0
+Text GLabel 5700 3650 2    60   Input ~ 0
 CHASIS_GND
 $Comp
@@
 $EndComp
 Wire Wire Line
-	5100 3250 5100 3200
+	5100 3100 5100 3250
 Wire Wire Line
-	4750 3250 5100 3250
+	5100 3250 4750 3250
 Wire Wire Line
-	5200 3200 5200 3250
+	5200 3100 5200 3250
 Wire Wire Line
 	5200 3250 5550 3250
@@
 	5550 4150 5200 4150
 Wire Wire Line
-	5100 4400 5100 5000
-Wire Wire Line
-	5200 5000 5200 4400
-Wire Wire Line
 	5100 4150 5100 4200
 Wire Wire Line
 	5200 4150 5200 4200
-Wire Wire Line
-	5500 2800 5700 2800
 $Comp
 L FERRITE FB7
@@
 Wire Wire Line
 	4550 3200 4550 3900
-Wire Wire Line
-	4550 3200 5000 3200
-Wire Wire Line
-	4550 5000 5000 5000
 $Comp
 L FERRITE FB8
@@
 	0    -1   -1   0
 $EndComp
-Wire Wire Line
-	4550 4700 4550 5000
 Connection ~ 4550 4300
 Connection ~ 4550 3650
 Wire Wire Line
 	4850 3650 4550 3650
-Wire Wire Line
-	5500 5000 5300 5000
-Text GLabel 5200 5000 3    60   Input ~ 0
+Text GLabel 5200 4550 2    60   Input ~ 0
 D+
-Text GLabel 5100 5000 3    60   Input ~ 0
+Text GLabel 5100 4550 0    60   Input ~ 0
 D-
 Wire Wire Line
@@
 Wire Wire Line
 	3950 4300 4150 4300
-Connection ~ 5700 3200
+$Comp
+L USB_B P6
+U 1 1 59320548
+P 5200 2800
+F 0 "P6" H 5000 3250 50  0000 L CNN
+F 1 "USB_B" H 5000 3150 50  0000 L CNN
+F 2 "WheelerLab:1734346-1" H 5350 2750 50  0001 C CNN
+F 3 "" H 5350 2750 50  0001 C CNN
+F 4 "1734346-1" H 5200 2800 60  0001 C CNN "Mfg_Part_No"
+	1    5200 2800
+	0    1    1    0
+$EndComp
 Wire Wire Line
-	5300 3200 5700 3200
+	4550 3200 5400 3200
+Wire Wire Line
+	5400 3200 5400 3100
 Wire Wire Line
 	5700 3650 5450 3650
+$Comp
+L USB_A P9
+U 1 1 59320AF4
+P 5200 5000
+F 0 "P9" H 5000 5450 50  0000 L CNN
+F 1 "USB_A" H 5000 5350 50  0000 L CNN
+F 2 "WheelerLab:AU-Y1006" H 5350 4950 50  0001 C CNN
+F 3 "" H 5350 4950 50  0001 C CNN
+F 4 "AU-Y1006" H 5200 5000 60  0001 C CNN "Mfg_Part_No"
+	1    5200 5000
+	0    1    -1   0
+$EndComp
+Text GLabel 4800 2700 0    60   Input ~ 0
+CHASIS_GND
 Wire Wire Line
-	5700 2800 5700 3650
+	4800 2800 4800 2700
 Wire Wire Line
-	5500 4600 5500 5000
+	5100 4700 5100 4400
+Wire Wire Line
+	5200 4400 5200 4700
+Wire Wire Line
+	4800 5000 4800 5100
+Wire Wire Line
+	4550 4700 4550 5300
+Wire Wire Line
+	4550 5300 5700 5300
+Wire Wire Line
+	5700 5300 5700 4700
+Wire Wire Line
+	5700 4700 5400 4700
 $EndSCHEMATC

Commit message: Update schematic to use power ports
Changed lines of the file:
@@
 Comment4 ""
 $EndDescr
-Text GLabel 4800 5100 0    60   Input ~ 0
-GND
 Text Notes 4450 2450 0    60   ~ 0
 USB PASSTHROUGH\nIncludes ESD protection and\nEMI suppression (See Wurth\nElectronics App Note ANP002C).
@@
 Wire Wire Line
 	5700 4700 5400 4700
+$Comp
+L GND #PWR025
+U 1 1 5B3C7E87
+P 4800 5100
+F 0 "#PWR025" H 4800 4850 50  0001 C CNN
+F 1 "GND" H 4800 4950 50  0000 C CNN
+F 2 "" H 4800 5100 50  0001 C CNN
+F 3 "" H 4800 5100 50  0001 C CNN
+	1    4800 5100
+	1    0    0    -1
+$EndComp
 $EndSCHEMATC

Commit message: Update to use Sci-Bots library
Parts:
- D5: footprint WheelerLab:wurth-WE-TVS_SOT23-6L -> Sci-Bots:wurth-WE-TVS_SOT23-6L
- L2: footprint WheelerLab:wurth-WE-CNSW_0805 -> Sci-Bots:wurth-WE-CNSW_0805
- P6: footprint WheelerLab:1734346-1 -> Sci-Bots:1734346-1
- P9: footprint WheelerLab:AU-Y1006 -> Sci-Bots:AU-Y1006
Changed lines of the file:
@@
 LIBS:contrib
 LIBS:valves
-LIBS:wheelerlab
+LIBS:sci-bots
 LIBS:dropbot_control_board-cache
 EELAYER 25 0
@@
 F 0 "D5" V 4800 3600 45  0000 L BNN
 F 1 "WE-TVS_824015" V 5615 3450 45  0000 L BNN
-F 2 "WheelerLab:wurth-WE-TVS_SOT23-6L" H 5180 3800 20  0001 C CNN
+F 2 "Sci-Bots:wurth-WE-TVS_SOT23-6L" H 5180 3800 20  0001 C CNN
 F 3 "" H 5150 3650 60  0000 C CNN
 F 4 "824015" H 5150 3650 60  0001 C CNN "Mfg_Part_No"
@@
 F 0 "L2" H 5250 4350 50  0000 L CNN
 F 1 "90 Ohm@100MHz" H 5250 4250 50  0000 L CNN
-F 2 "WheelerLab:wurth-WE-CNSW_0805" H 5200 4300 50  0001 C CNN
+F 2 "Sci-Bots:wurth-WE-CNSW_0805" H 5200 4300 50  0001 C CNN
 F 3 "" H 5200 4300 50  0000 C CNN
 F 4 "744231091" H 5150 4300 60  0001 C CNN "Mfg_Part_No"
@@
 F 0 "P6" H 5000 3250 50  0000 L CNN
 F 1 "USB_B" H 5000 3150 50  0000 L CNN
-F 2 "WheelerLab:1734346-1" H 5350 2750 50  0001 C CNN
+F 2 "Sci-Bots:1734346-1" H 5350 2750 50  0001 C CNN
 F 3 "" H 5350 2750 50  0001 C CNN
 F 4 "1734346-1" H 5200 2800 60  0001 C CNN "Mfg_Part_No"
@@
 F 0 "P9" H 5000 5450 50  0000 L CNN
 F 1 "USB_A" H 5000 5350 50  0000 L CNN
-F 2 "WheelerLab:AU-Y1006" H 5350 4950 50  0001 C CNN
+F 2 "Sci-Bots:AU-Y1006" H 5350 4950 50  0001 C CNN
 F 3 "" H 5350 4950 50  0001 C CNN
 F 4 "AU-Y1006" H 5200 5000 60  0001 C CNN "Mfg_Part_No"
