File: boost-converter.sch (KiCad schematic (older format))
At the start: 30 parts, among them Q1 STP33N65M2, U2 MAX1771, U3 CAT5171, U4 HV7802

Commit message: Add missing schematic diagrams and change some part numbers
Parts:
- R14: value 5.1 -> 1; Mfg_Part_No MCR10ERTFL5R10 -> ERJ-6DQJ1R0V
Changed lines of the file:
@@
 P 8350 3700
 F 0 "R14" V 8250 3700 50  0000 C CNN
-F 1 "5.1" V 8350 3700 50  0000 C CNN
+F 1 "1" V 8350 3700 50  0000 C CNN
 F 2 "Resistors_SMD:R_0805" V 8280 3700 30  0001 C CNN
 F 3 "" H 8350 3700 30  0000 C CNN
-F 4 "MCR10ERTFL5R10" H 8350 3700 60  0001 C CNN "Mfg_Part_No"
+F 4 "ERJ-6DQJ1R0V" H 8350 3700 60  0001 C CNN "Mfg_Part_No"
 	1    8350 3700
 	0    1    1    0

Commit message: Improve layout/stability of boost converter, etc.
* improve layout/stability of boost converter
* enable on board calibration without HVOE
* add decoupling cap to 0.6V reference
* fix footprint for U10
* add programming wire
Parts:
- added C19, C21: 100pF, Capacitors_SMD:C_0805, symbol C
- L1: symbol INDUCTOR -> L
Other:
- note added: "Q1 should be selected for low Qg, Rdson & Coss\nR6, R8, C7, and C19 must be rated at >400V\nD1 should be an ultra-fast (<50ns) recovery, 4A, >400V\nC1 & C6 should be a low ESR type (e.g., AVX TPS series)\nC1 & C2 should be sited very close to pin 2 (VCC) of U2\nC7 should be low ESR (<3ohms and rated >400V)\nIf you have stability issues, a 100pF 400 V ceramic cap\n could be soldered on top of R8\n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"
- note removed: "Q1 should be selected for low Qg, Rdson & Coss\nR6, R8, and C7 must be rated at >400V\nD1 should be an ultra-fast (<50ns) recovery, 4A, >400V\nC1 & C6 should be a low ESR type (e.g., AVX TPS series)\nC1 & C2 should be sited very close to pin 2 (VCC) of U2\nC7 should be low ESR (<3ohms and rated >400V)\nIf you have stability issues, a 100pF 400 V ceramic cap\n could be soldered on top of R8\nL1 sh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"

Commit message: Change value of R7 to 10k
Fixes #6
Parts:
- R7: value 2k -> 10k; Mfg_Part_No RC0805FR-072KL -> RC0805FR-0710KL
Changed lines of the file:
@@
 P 5950 4950
 F 0 "R7" V 6030 4950 50  0000 C CNN
-F 1 "2k" V 5950 4950 50  0000 C CNN
+F 1 "10k" V 5950 4950 50  0000 C CNN
 F 2 "Resistors_SMD:R_0805" V 5880 4950 30  0001 C CNN
 F 3 "" H 5950 4950 30  0000 C CNN
-F 4 "RC0805FR-072KL" H 5950 4950 60  0001 C CNN "Mfg_Part_No"
+F 4 "RC0805FR-0710KL" H 5950 4950 60  0001 C CNN "Mfg_Part_No"
 	1    5950 4950
 	1    0    0    -1

Commit message: Fix label of A2, update netlist
Connections:
- net labels added: A2/HV7802_CS
- net labels removed: A2/HV507_CS
Changed lines of the file:
@@
 $EndComp
 Text GLabel 8700 5250 0    60   Input ~ 0
-A2/HV507_CS
+A2/HV7802_CS
 Text GLabel 7550 4600 2    60   Input ~ 0
 D5/SSCL

Commit message: Update schematic to use power ports
Connections:
- wire segments 54 -> 55
Changed lines of the file:
@@
 	1    0    0    -1
 $EndComp
-Text GLabel 2200 3400 0    60   Input ~ 0
-+12V
-Text GLabel 2200 5150 0    60   Input ~ 0
-GND
 Text GLabel 8700 3700 2    60   Input ~ 0
 HV
-Text GLabel 6400 4100 0    60   Input ~ 0
-+3.3V
 $Comp
 L R R5
@@
 	0    1    1    0
 $EndComp
-Text GLabel 6800 4100 2    60   Input ~ 0
-GND
 $Comp
 L CP C1
@@
 	6400 4200 6400 4100
 Wire Wire Line
-	6700 4100 6800 4100
+	6700 4100 6900 4100
 Wire Wire Line
 	2200 5150 8550 5150
@@
 Wire Wire Line
 	3100 4500 3100 5150
+$Comp
+L +12V #PWR040
+U 1 1 5B3BF4CF
+P 2200 3400
+F 0 "#PWR040" H 2200 3250 50  0001 C CNN
+F 1 "+12V" H 2200 3540 50  0000 C CNN
+F 2 "" H 2200 3400 50  0001 C CNN
+F 3 "" H 2200 3400 50  0001 C CNN
+	1    2200 3400
+	1    0    0    -1
+$EndComp
+$Comp
+L +3.3V #PWR041
+U 1 1 5B3BFA2D
+P 6300 4100
+F 0 "#PWR041" H 6300 3950 50  0001 C CNN
+F 1 "+3.3V" H 6300 4240 50  0000 C CNN
+F 2 "" H 6300 4100 50  0001 C CNN
+F 3 "" H 6300 4100 50  0001 C CNN
+	1    6300 4100
+	1    0    0    -1
+$EndComp
+Wire Wire Line
+	6400 4100 6300 4100
+$Comp
+L GND #PWR042
+U 1 1 5B3C8BB3
+P 2200 5150
+F 0 "#PWR042" H 2200 4900 50  0001 C CNN
+F 1 "GND" H 2200 5000 50  0000 C CNN
+F 2 "" H 2200 5150 50  0001 C CNN
+F 3 "" H 2200 5150 50  0001 C CNN
+	1    2200 5150
+	1    0    0    -1
+$EndComp
+$Comp
+L GND #PWR043
+U 1 1 5B3C90C5
+P 6900 4100
+F 0 "#PWR043" H 6900 3850 50  0001 C CNN
+F 1 "GND" H 6900 3950 50  0000 C CNN
+F 2 "" H 6900 4100 50  0001 C CNN
+F 3 "" H 6900 4100 50  0001 C CNN
+	1    6900 4100
+	1    0    0    -1
+$EndComp
 $EndSCHEMATC

Commit message: Update to use Sci-Bots library
Parts:
- U3: footprint WheelerLab:SOT-23-8 -> Sci-Bots:SOT-23-8
Changed lines of the file:
@@
 LIBS:contrib
 LIBS:valves
-LIBS:wheelerlab
+LIBS:sci-bots
 LIBS:dropbot_control_board-cache
 EELAYER 25 0
@@
 F 0 "U3" H 6150 4950 50  0000 L CNN
 F 1 "CAT5171" H 6450 4950 50  0000 L CNN
-F 2 "WheelerLab:SOT-23-8" H 6400 4600 50  0001 C CNN
+F 2 "Sci-Bots:SOT-23-8" H 6400 4600 50  0001 C CNN
 F 3 "http://www.onsemi.com/pub_link/Collateral/CAT5171-D.PDF" H 6400 4600 50  0001 C CNN
 F 4 "CAT5171TBI-50GT3" H 6400 4600 60  0001 C CNN "Mfg_Part_No"

Commit message: Update with kicad-helpers files
Parts:
- C1, C6, C7: symbol CP -> Device:CP
- C19, C2, C21, C24, C5, C8: symbol C -> Device:C
- C30, C31: symbol C_Small -> Device:C_Small
- D1: symbol D -> Device:D
- L1: symbol L -> Device:L
- R13, R14, R15, R16, R38, R39, R46, R47, R48, R49, R5, R6, R7, R8, R9: symbol R -> Device:R
Changed lines of the file:
@@
-EESchema Schematic File Version 2
-LIBS:power
-LIBS:device
-LIBS:transistors
-LIBS:conn
-LIBS:linear
-LIBS:regul
-LIBS:74xx
-LIBS:cmos4000
-LIBS:adc-dac
-LIBS:memory
-LIBS:xilinx
-LIBS:microcontrollers
-LIBS:dsp
-LIBS:microchip
-LIBS:analog_switches
-LIBS:motorola
-LIBS:texas
-LIBS:intel
-LIBS:audio
-LIBS:interface
-LIBS:digital-audio
-LIBS:philips
-LIBS:display
-LIBS:cypress
-LIBS:siliconi
-LIBS:opto
-LIBS:atmel
-LIBS:contrib
-LIBS:valves
-LIBS:sci-bots
-LIBS:dropbot_control_board-cache
-EELAYER 25 0
+EESchema Schematic File Version 4
+EELAYER 30 0
 EELAYER END
 $Descr USLetter 11000 8500
@@
 $EndDescr
 $Comp
-L C C5
+L Device:C C5
 U 1 1 56BE95FE
 P 2900 4750
@@
 $EndComp
 $Comp
-L CP C6
+L Device:CP C6
 U 1 1 56BE9601
 P 2200 3850
@@
 $EndComp
 $Comp
-L L L1
+L Device:L L1
 U 1 1 56BE9603
 P 4250 3400
@@
 $EndComp
 $Comp
-L D D1
+L Device:D D1
 U 1 1 56BE9605
 P 5050 3700
@@
 $EndComp
 $Comp
-L CP C7
+L Device:CP C7
 U 1 1 56BE9606
 P 5350 4300
@@
 $EndComp
 $Comp
-L R R7
+L Device:R R7
 U 1 1 56BE9607
 P 5950 4950
@@
 $EndComp
 $Comp
-L R R6
+L Device:R R6
 U 1 1 56BE9608
 P 5950 4100
@@
 HV
 $Comp
-L R R5
+L Device:R R5
 U 1 1 56BF5E85
 P 4700 5000
@@
 D10/SHDN
 $Comp
-L R R8
+L Device:R R8
 U 1 1 56C13B29
 P 7650 4000
@@
 $EndComp
 $Comp
-L R R9
+L Device:R R9
 U 1 1 56C13BEC
 P 7650 5000
@@
 $EndComp
 $Comp
-L R R13
+L Device:R R13
 U 1 1 56BEB254
 P 8400 3900
@@
 $EndComp
 $Comp
-L R R14
+L Device:R R14
 U 1 1 56BEC206
 P 8550 3700
@@
 $EndComp
 $Comp
-L R R16
+L Device:R R16
 U 1 1 56BEC2BD
 P 8700 3900
@@
 $EndComp
 $Comp
-L R R15
+L Device:R R15
 U 1 1 56BECCAC
 P 8550 5000
@@
 $EndComp
 $Comp
-L C C8
+L Device:C C8
 U 1 1 56C02E02
 P 6550 4100
@@
 $EndComp
 $Comp
-L CP C1
+L Device:CP C1
 U 1 1 56BE9600
 P 2500 3850
@@
 $EndComp
 $Comp
-L R R38
+L Device:R R38
 U 1 1 58BB654C
 P 4250 4200
@@
 $EndComp
 $Comp
-L R R39
+L Device:R R39
 U 1 1 58BB914D
 P 4850 3400
@@
 $EndComp
 $Comp
-L C C24
+L Device:C C24
 U 1 1 58BB9423
 P 5150 3400
@@
 $EndComp
 $Comp
-L C_Small C30
+L Device:C_Small C30
 U 1 1 58BEFA2F
 P 7250 4400
@@
 $EndComp
 $Comp
-L R R46
+L Device:R R46
 U 1 1 58BEFA35
 P 7100 4500
@@
 $EndComp
 $Comp
-L R R47
+L Device:R R47
 U 1 1 58BEFA3B
 P 7100 4600
@@
 $EndComp
 $Comp
-L C_Small C31
+L Device:C_Small C31
 U 1 1 58BEFA41
 P 7250 4700
@@
 $EndComp
 $Comp
-L R R48
+L Device:R R48
 U 1 1 58BF0670
 P 7400 4500
@@
 $EndComp
 $Comp
-L R R49
+L Device:R R49
 U 1 1 58BF0676
 P 7400 4600
@@
 D4/SSDA
 $Comp
-L C C2
+L Device:C C2
 U 1 1 58CA2C47
 P 2750 3850
@@
 $EndComp
 $Comp
-L C C19
+L Device:C C19
 U 1 1 5947498F
 P 5650 4100
@@
 	5650 4250 5650 4700
 $Comp
-L C C21
+L Device:C C21
 U 1 1 5947519B
 P 5650 4850
@@
 	3100 4500 3100 5150
 $Comp
-L +12V #PWR040
+L power:+12V #PWR040
 U 1 1 5B3BF4CF
 P 2200 3400
@@
 $EndComp
 $Comp
-L +3.3V #PWR041
+L power:+3.3V #PWR041
 U 1 1 5B3BFA2D
 P 6300 4100
@@
 	6400 4100 6300 4100
 $Comp
-L GND #PWR042
+L power:GND #PWR042
 U 1 1 5B3C8BB3
 P 2200 5150
@@
 $EndComp
 $Comp
-L GND #PWR043
+L power:GND #PWR043
 U 1 1 5B3C90C5
 P 6900 4100
