File: feedback.sch (KiCad schematic (older format))
At the start: 16 parts, among them U11 MCP6022

Commit message: Add missing schematic diagrams and change some part numbers
Parts:
- U11: Mfg_Part_No (none) -> ED14DT
- renumbered C14 to C15
Changed lines of the file:
@@
 F 2 "Housings_DIP:DIP-8_W7.62mm" H 5900 4150 60  0001 C CNN
 F 3 "" H 5900 4150 60  0000 C CNN
+F 4 "ED14DT" H 5900 4150 60  0001 C CNN "Mfg_Part_No"
 	1    5900 4150
 	1    0    0    -1
@@
 GND
 $Comp
-L C_Small C14
+L C_Small C15
 U 1 1 591D89BB
 P 6200 3300
-F 0 "C14" V 6050 3250 50  0000 L CNN
+F 0 "C15" V 6050 3250 50  0000 L CNN
 F 1 "1uF" V 6350 3250 50  0000 L CNN
 F 2 "Capacitors_SMD:C_0805" H 6200 3300 50  0001 C CNN

Commit message: Improve layout/stability of boost converter, etc.
* improve layout/stability of boost converter
* enable on board calibration without HVOE
* add decoupling cap to 0.6V reference
* fix footprint for U10
* add programming wire
Parts:
- F2: symbol F_Small -> Fuse_Small
- U11: Mfg_Part_No ED14DT -> ED08DT
Changed lines of the file:
@@
 LIBS:valves
 LIBS:wheelerlab
+LIBS:dropbot_control_board-cache
 EELAYER 25 0
 EELAYER END
@@
 Sheet 5 7
 Title "DropBot control board"
-Date "2017-05-17"
-Rev "3.5"
+Date "2017-06-19"
+Rev "3.6"
 Comp "Sci-Bots Inc."
 Comment1 ""
@@
 $EndComp
 $Comp
-L F_Small F2
+L Fuse_Small F2
 U 1 1 58BC51B6
 P 3450 4100
@@
 F 2 "Housings_DIP:DIP-8_W7.62mm" H 5900 4150 60  0001 C CNN
 F 3 "" H 5900 4150 60  0000 C CNN
-F 4 "ED14DT" H 5900 4150 60  0001 C CNN "Mfg_Part_No"
+F 4 "ED08DT" H 5900 4150 60  0001 C CNN "Mfg_Part_No"
 	1    5900 4150
 	1    0    0    -1

Commit message: Update BOM
2 part numbers (F1 and F2) had typos and updated D4 to a part that
is more commonly available.
Parts:
- D4: Mfg_Part_No BAV99-7-F -> TBAV99,LM
- F2: Mfg_Part_No B59807A90A62 -> B59807A0090A062
Changed lines of the file:
@@
 F 2 "Resistors_SMD:R_1210" H 3450 4100 50  0001 C CNN
 F 3 "" H 3450 4100 50  0000 C CNN
-F 4 "B59807A90A62" H 3450 4100 60  0001 C CNN "Mfg_Part_No"
+F 4 "B59807A0090A062" H 3450 4100 60  0001 C CNN "Mfg_Part_No"
 	1    3450 4100
 	-1   0    0    1
@@
 F 2 "TO_SOT_Packages_SMD:SOT-23" H 4150 3700 50  0001 C CNN
 F 3 "" H 4150 3700 50  0000 C CNN
-F 4 "BAV99-7-F" H 4150 3700 60  0001 C CNN "Mfg_Part_No"
+F 4 "TBAV99,LM" H 4150 3700 60  0001 C CNN "Mfg_Part_No"
 	1    4150 3700
 	1    0    0    -1

Commit message: Update schematic to use power ports
Changed lines of the file:
@@
 L C C20
 U 1 1 57E388CA
-P 5850 3450
-F 0 "C20" H 5875 3550 50  0000 L CNN
-F 1 "100pF" H 5875 3350 50  0000 L CNN
-F 2 "Capacitors_SMD:C_0805" H 5888 3300 30  0001 C CNN
-F 3 "" H 5850 3450 60  0000 C CNN
-F 4 "CL21C101JECNNWC" H 5850 3450 60  0001 C CNN "Mfg_Part_No"
-	1    5850 3450
+P 5850 3400
+F 0 "C20" H 5875 3500 50  0000 L CNN
+F 1 "100pF" H 5875 3300 50  0000 L CNN
+F 2 "Capacitors_SMD:C_0805" H 5888 3250 30  0001 C CNN
+F 3 "" H 5850 3400 60  0000 C CNN
+F 4 "CL21C101JECNNWC" H 5850 3400 60  0001 C CNN "Mfg_Part_No"
+	1    5850 3400
 	-1   0    0    1
 $EndComp
@@
 	1    0    0    -1
 $EndComp
-Text GLabel 3850 3700 0    60   Input ~ 0
-GND
 Text Notes 3600 3400 0    60   ~ 0
 CURRENT-TO-VOLTAGE\nCONVERTER
@@
 $EndComp
 Connection ~ 7150 4300
-Text GLabel 7550 4000 2    60   Input ~ 0
-+3.3V
 $Comp
 L C_Small C11
@@
 Connection ~ 4700 4100
 Wire Wire Line
-	3800 4100 3550 4100
+	3550 4100 3800 4100
 Wire Wire Line
 	3200 4100 3350 4100
@@
 	4700 3800 5250 3800
 Wire Wire Line
-	5250 3300 5250 4000
+	5250 3250 5250 4000
 Connection ~ 4950 3800
-Text GLabel 4450 3700 2    60   Input ~ 0
-+3.3V
 Wire Wire Line
 	6550 4100 6550 4200
@@
 Connection ~ 6900 4600
 Wire Wire Line
-	7550 4300 7550 4000
-Wire Wire Line
-	7550 4000 6550 4000
+	7550 4000 7550 4300
+Wire Wire Line
+	6550 4000 7550 4000
 Connection ~ 7150 4000
 Connection ~ 7150 4600
@@
 L R R34
 U 1 1 591D8457
-P 5400 3300
-F 0 "R34" V 5480 3300 50  0000 C CNN
-F 1 "5.1k" V 5400 3300 50  0000 C CNN
-F 2 "Resistors_SMD:R_0805" V 5330 3300 30  0001 C CNN
-F 3 "" H 5400 3300 30  0000 C CNN
-F 4 "RC0805FR-075K1L" H 5400 3300 60  0001 C CNN "Mfg_Part_No"
-	1    5400 3300
+P 5400 3250
+F 0 "R34" V 5480 3250 50  0000 C CNN
+F 1 "5.1k" V 5400 3250 50  0000 C CNN
+F 2 "Resistors_SMD:R_0805" V 5330 3250 30  0001 C CNN
+F 3 "" H 5400 3250 30  0000 C CNN
+F 4 "RC0805FR-075K1L" H 5400 3250 60  0001 C CNN "Mfg_Part_No"
+	1    5400 3250
 	0    1    1    0
 $EndComp
 Connection ~ 5250 3800
-Text GLabel 5850 3600 2    60   Input ~ 0
-GND
 $Comp
 L C_Small C15
 U 1 1 591D89BB
-P 6200 3300
-F 0 "C15" V 6050 3250 50  0000 L CNN
-F 1 "1uF" V 6350 3250 50  0000 L CNN
-F 2 "Capacitors_SMD:C_0805" H 6200 3300 50  0001 C CNN
-F 3 "" H 6200 3300 50  0000 C CNN
-F 4 "CC0805KKX7R9BB105" H 6200 3300 60  0001 C CNN "Mfg_Part_No"
-	1    6200 3300
+P 6200 3250
+F 0 "C15" V 6050 3200 50  0000 L CNN
+F 1 "1uF" V 6350 3200 50  0000 L CNN
+F 2 "Capacitors_SMD:C_0805" H 6200 3250 50  0001 C CNN
+F 3 "" H 6200 3250 50  0000 C CNN
+F 4 "CC0805KKX7R9BB105" H 6200 3250 60  0001 C CNN "Mfg_Part_No"
+	1    6200 3250
 	0    -1   -1   0
 $EndComp
-Connection ~ 5850 3300
+Connection ~ 5850 3250
 $Comp
 L R R53
 U 1 1 591D8A9A
-P 6500 3450
-F 0 "R53" H 6650 3450 50  0000 C CNN
-F 1 "1Meg" V 6500 3450 50  0000 C CNN
-F 2 "Resistors_SMD:R_0805" V 6430 3450 50  0001 C CNN
-F 3 "" H 6500 3450 50  0000 C CNN
-F 4 "RC0805FR-071ML" H 6500 3450 60  0001 C CNN "Mfg_Part_No"
-	1    6500 3450
-	1    0    0    -1
-$EndComp
-Text GLabel 6750 3300 2    60   Input ~ 0
+P 6500 3400
+F 0 "R53" H 6650 3400 50  0000 C CNN
+F 1 "1Meg" V 6500 3400 50  0000 C CNN
+F 2 "Resistors_SMD:R_0805" V 6430 3400 50  0001 C CNN
+F 3 "" H 6500 3400 50  0000 C CNN
+F 4 "RC0805FR-071ML" H 6500 3400 60  0001 C CNN "Mfg_Part_No"
+	1    6500 3400
+	1    0    0    -1
+$EndComp
+Text GLabel 6750 3250 2    60   Input ~ 0
 A11
-Connection ~ 6500 3300
-Text GLabel 6500 3600 2    60   Input ~ 0
+Connection ~ 6500 3250
+Text GLabel 6500 3550 2    60   Input ~ 0
 +0.6V
 Wire Wire Line
-	5550 3300 6100 3300
-Wire Wire Line
-	6300 3300 6750 3300
-Text GLabel 7550 4600 2    60   Input ~ 0
-GND
+	5550 3250 6100 3250
+Wire Wire Line
+	6300 3250 6750 3250
+$Comp
+L +3.3V #PWR035
+U 1 1 5B3C0391
+P 4450 3700
+F 0 "#PWR035" H 4450 3550 50  0001 C CNN
+F 1 "+3.3V" H 4450 3840 50  0000 C CNN
+F 2 "" H 4450 3700 50  0001 C CNN
+F 3 "" H 4450 3700 50  0001 C CNN
+	1    4450 3700
+	1    0    0    -1
+$EndComp
+$Comp
+L +3.3V #PWR036
+U 1 1 5B3C07F1
+P 7550 4000
+F 0 "#PWR036" H 7550 3850 50  0001 C CNN
+F 1 "+3.3V" H 7550 4140 50  0000 C CNN
+F 2 "" H 7550 4000 50  0001 C CNN
+F 3 "" H 7550 4000 50  0001 C CNN
+	1    7550 4000
+	1    0    0    -1
+$EndComp
+$Comp
+L GND #PWR037
+U 1 1 5B3CA0DD
+P 3850 3700
+F 0 "#PWR037" H 3850 3450 50  0001 C CNN
+F 1 "GND" H 3850 3550 50  0000 C CNN
+F 2 "" H 3850 3700 50  0001 C CNN
+F 3 "" H 3850 3700 50  0001 C CNN
+	1    3850 3700
+	1    0    0    -1
+$EndComp
+$Comp
+L GND #PWR038
+U 1 1 5B3CA4E0
+P 3650 4600
+F 0 "#PWR038" H 3650 4350 50  0001 C CNN
+F 1 "GND" H 3650 4450 50  0000 C CNN
+F 2 "" H 3650 4600 50  0001 C CNN
+F 3 "" H 3650 4600 50  0001 C CNN
+	1    3650 4600
+	1    0    0    -1
+$EndComp
+$Comp
+L GND #PWR039
+U 1 1 5B3CA54D
+P 5850 3550
+F 0 "#PWR039" H 5850 3300 50  0001 C CNN
+F 1 "GND" H 5850 3400 50  0000 C CNN
+F 2 "" H 5850 3550 50  0001 C CNN
+F 3 "" H 5850 3550 50  0001 C CNN
+	1    5850 3550
+	1    0    0    -1
+$EndComp
 $EndSCHEMATC

Commit message: Update with kicad-helpers files
Parts:
- C11, C15: symbol C_Small -> Device:C_Small
- C16, C17, C18, C20: symbol C -> Device:C
- F2: symbol Fuse_Small -> Device:Fuse_Small
- R23, R25, R26, R27, R33, R34, R53: symbol R -> Device:R
Changed lines of the file:
@@
-EESchema Schematic File Version 2
-LIBS:power
-LIBS:device
-LIBS:transistors
-LIBS:conn
-LIBS:linear
-LIBS:regul
-LIBS:74xx
-LIBS:cmos4000
-LIBS:adc-dac
-LIBS:memory
-LIBS:xilinx
-LIBS:microcontrollers
-LIBS:dsp
-LIBS:microchip
-LIBS:analog_switches
-LIBS:motorola
-LIBS:texas
-LIBS:intel
-LIBS:audio
-LIBS:interface
-LIBS:digital-audio
-LIBS:philips
-LIBS:display
-LIBS:cypress
-LIBS:siliconi
-LIBS:opto
-LIBS:atmel
-LIBS:contrib
-LIBS:valves
-LIBS:sci-bots
-LIBS:dropbot_control_board-cache
-EELAYER 25 0
+EESchema Schematic File Version 4
+EELAYER 30 0
 EELAYER END
 $Descr USLetter 11000 8500
@@
 $EndDescr
 $Comp
-L R R25
+L Device:R R25
 U 1 1 57E388BE
 P 7150 4150
@@
 $EndComp
 $Comp
-L R R26
+L Device:R R26
 U 1 1 57E388BF
 P 7150 4450
@@
 $EndComp
 $Comp
-L C C17
+L Device:C C17
 U 1 1 57E388C0
 P 6900 4450
@@
 $EndComp
 $Comp
-L R R27
+L Device:R R27
 U 1 1 57E388C1
 P 4950 3950
@@
 $EndComp
 $Comp
-L C C16
+L Device:C C16
 U 1 1 57E388C2
 P 4700 3950
@@
 +0.6V
 $Comp
-L C C20
+L Device:C C20
 U 1 1 57E388CA
 P 5850 3400
@@
 first-order low-pass\nanti-aliasing filter
 $Comp
-L C C18
+L Device:C C18
 U 1 1 57E388CC
 P 7550 4450
@@
 CUR_SENSE
 $Comp
-L R R23
+L Device:R R23
 U 1 1 57E5CF28
 P 3650 4450
@@
 $EndComp
 $Comp
-L Fuse_Small F2
+L Device:Fuse_Small F2
 U 1 1 58BC51B6
 P 3450 4100
@@
 Connection ~ 7150 4300
 $Comp
-L C_Small C11
+L Device:C_Small C11
 U 1 1 58C6E481
 P 3900 4100
@@
 Connection ~ 5250 4600
 $Comp
-L R R33
+L Device:R R33
 U 1 1 591D56C4
 P 4950 4350
@@
 	4900 4500 4950 4500
 $Comp
-L R R34
+L Device:R R34
 U 1 1 591D8457
 P 5400 3250
@@
 Connection ~ 5250 3800
 $Comp
-L C_Small C15
+L Device:C_Small C15
 U 1 1 591D89BB
 P 6200 3250
@@
 Connection ~ 5850 3250
 $Comp
-L R R53
+L Device:R R53
 U 1 1 591D8A9A
 P 6500 3400
@@
 	6300 3250 6750 3250
 $Comp
-L +3.3V #PWR035
+L power:+3.3V #PWR035
 U 1 1 5B3C0391
 P 4450 3700
@@
 $EndComp
 $Comp
-L +3.3V #PWR036
+L power:+3.3V #PWR036
 U 1 1 5B3C07F1
 P 7550 4000
@@
 $EndComp
 $Comp
-L GND #PWR037
+L power:GND #PWR037
 U 1 1 5B3CA0DD
 P 3850 3700
@@
 $EndComp
 $Comp
-L GND #PWR038
+L power:GND #PWR038
 U 1 1 5B3CA4E0
 P 3650 4600
@@
 $EndComp
 $Comp
-L GND #PWR039
+L power:GND #PWR039
 U 1 1 5B3CA54D
 P 5850 3550

Commit message: Fix broken symbols and DRC tests
Parts:
- D4: symbol BAV99 -> sci-bots:BAV99
- U11: symbol MCP6022 -> sci-bots:MCP6022
Connections:
- wire segments 17 -> 30
Changed lines of the file:
@@
 $EndComp
 $Comp
-L BAV99 D4
+L sci-bots:BAV99 D4
 U 1 1 58BCBFA7
 P 4150 3700
@@
 $EndComp
 $Comp
-L MCP6022 U11
+L sci-bots:MCP6022 U11
 U 1 1 591D0EAB
 P 5900 4150
@@
 $EndComp
 Wire Wire Line
-	4000 4100 5250 4100
+	4000 4100 4150 4100
 Connection ~ 4950 4100
 Connection ~ 4700 4100
 Wire Wire Line
-	3550 4100 3800 4100
+	3550 4100 3650 4100
 Wire Wire Line
 	3200 4100 3350 4100
@@
 Connection ~ 4150 4100
 Wire Wire Line
-	4700 3800 5250 3800
-Wire Wire Line
-	5250 3250 5250 4000
+	4700 3800 4950 3800
+Wire Wire Line
+	5250 3250 5250 3800
 Connection ~ 4950 3800
 Wire Wire Line
@@
 Connection ~ 6900 4300
 Wire Wire Line
-	3650 4600 7550 4600
+	3650 4600 5250 4600
 Connection ~ 6900 4600
 Wire Wire Line
 	7550 4000 7550 4300
 Wire Wire Line
-	6550 4000 7550 4000
+	6550 4000 7150 4000
 Connection ~ 7150 4000
 Connection ~ 7150 4600
 Wire Wire Line
-	6550 4300 7150 4300
+	6550 4300 6900 4300
 Wire Wire Line
 	5250 4300 5250 4600
@@
 +0.6V
 Wire Wire Line
-	5550 3250 6100 3250
-Wire Wire Line
-	6300 3250 6750 3250
+	5550 3250 5850 3250
+Wire Wire Line
+	6300 3250 6500 3250
 $Comp
 L power:+3.3V #PWR035
@@
 	1    0    0    -1
 $EndComp
+Wire Wire Line
+	4950 4100 5250 4100
+Wire Wire Line
+	4700 4100 4950 4100
+Wire Wire Line
+	3650 4100 3800 4100
+Wire Wire Line
+	4150 4100 4700 4100
+Wire Wire Line
+	4950 3800 5250 3800
+Wire Wire Line
+	6900 4300 7150 4300
+Wire Wire Line
+	6900 4600 7150 4600
+Wire Wire Line
+	7150 4000 7550 4000
+Wire Wire Line
+	7150 4600 7550 4600
+Wire Wire Line
+	5250 4600 6900 4600
+Wire Wire Line
+	5250 3800 5250 4000
+Wire Wire Line
+	5850 3250 6100 3250
+Wire Wire Line
+	6500 3250 6750 3250
 $EndSCHEMATC
