File: feedback.sch (KiCad schematic (older format))
At the start: 16 parts, among them U11 MCP6022

Commit message: Update BOM
Parts:
- C11, C15: MPN (none) -> CC0805KKX7R9BB105; Manufacturer (none) -> Yageo
- C16: MPN (none) -> 08053C154JAT2A; Manufacturer (none) -> KYOCERA AVX
- C17, C18: MPN (none) -> CL21B104KBCNNNC; Manufacturer (none) -> Samsung
- C20: MPN (none) -> CL21C101JECNNWC; Manufacturer (none) -> Samsung
- D4: MPN (none) -> TBAV99,LM; Manufacturer (none) -> Toshiba
- F2: MPN (none) -> B59807A0090A062; Manufacturer (none) -> EPCOS
- R23, R53: MPN (none) -> RC0805FR-071ML; Manufacturer (none) -> Yageo
- R25: MPN (none) -> RC0805FR-0710KL; Manufacturer (none) -> Yageo
- R26: MPN (none) -> RC0805FR-072K2L; Manufacturer (none) -> Yageo
- R27, R33: MPN (none) -> RC0805FR-07100KL; Manufacturer (none) -> Yageo
- R34: MPN (none) -> RC0805FR-075K1L; Manufacturer (none) -> Yageo
- U11: MPN (none) -> ED08DT; Manufacturer (none) -> On Shore Technology

Commit message: Remove "Mfg_Part_No" field (replaced by  "MPN")
Parts:
- C11, C15: Mfg_Part_No CC0805KKX7R9BB105 -> (none)
- C16: Mfg_Part_No 08053C154JAT2A -> (none)
- C17, C18: Mfg_Part_No CL21B104KBCNNNC -> (none)
- C20: Mfg_Part_No CL21C101JECNNWC -> (none)
- D4: Mfg_Part_No TBAV99,LM -> (none)
- F2: Mfg_Part_No B59807A0090A062 -> (none)
- R23, R53: Mfg_Part_No RC0805FR-071ML -> (none)
- R25: Mfg_Part_No RC0805FR-0710KL -> (none)
- R26: Mfg_Part_No RC0805FR-072K2L -> (none)
- R27, R33: Mfg_Part_No RC0805FR-07100KL -> (none)
- R34: Mfg_Part_No RC0805FR-075K1L -> (none)
- U11: Mfg_Part_No ED08DT -> (none)
Changed lines of the file:
@@
 F 4 "RC0805FR-0710KL" H 7300 4250 50 0001 C CNN "MPN"
 F 5 "Yageo" H 7300 4250 50 0001 C CNN "Manufacturer"
-F 6 "RC0805FR-0710KL" H 7150 4150 60 0001 C CNN "Mfg_Part_No"
 	1    7150 4150
 	1    0    0    -1
@@
 F 4 "RC0805FR-072K2L" H 7300 4550 50 0001 C CNN "MPN"
 F 5 "Yageo" H 7300 4550 50 0001 C CNN "Manufacturer"
-F 6 "RC0805FR-072K2L" H 7150 4450 60 0001 C CNN "Mfg_Part_No"
 	1    7150 4450
 	1    0    0    -1
@@
 F 4 "CL21B104KBCNNNC" H 6700 4650 50 0001 C CNN "MPN"
 F 5 "Samsung" H 6700 4650 50 0001 C CNN "Manufacturer"
-F 6 "CL21B104KBCNNNC" H 6900 4450 60 0001 C CNN "Mfg_Part_No"
 	1    6900 4450
 	1    0    0    -1
@@
 F 4 "RC0805FR-07100KL" H 5100 4050 50 0001 C CNN "MPN"
 F 5 "Yageo" H 5100 4050 50 0001 C CNN "Manufacturer"
-F 6 "RC0805FR-07100KL" H 4950 3950 60 0001 C CNN "Mfg_Part_No"
 	1    4950 3950
 	1    0    0    -1
@@
 F 4 "08053C154JAT2A" H 4450 4150 50 0001 C CNN "MPN"
 F 5 "KYOCERA AVX" H 4450 4150 50 0001 C CNN "Manufacturer"
-F 6 "08053C154JAT2A" H 4700 3950 60 0001 C CNN "Mfg_Part_No"
 	1    4700 3950
 	1    0    0    -1
@@
 F 4 "CL21C101JECNNWC" H 5875 3600 50 0001 C CNN "MPN"
 F 5 "Samsung" H 5875 3600 50 0001 C CNN "Manufacturer"
-F 6 "CL21C101JECNNWC" H 5850 3400 60 0001 C CNN "Mfg_Part_No"
 	1    5850 3400
 	-1   0    0    1
@@
 F 4 "CL21B104KBCNNNC" H 7575 4650 50 0001 C CNN "MPN"
 F 5 "Samsung" H 7575 4650 50 0001 C CNN "Manufacturer"
-F 6 "CL21B104KBCNNNC" H 7550 4450 60 0001 C CNN "Mfg_Part_No"
 	1    7550 4450
 	1    0    0    -1
@@
 F 4 "RC0805FR-071ML" H 3550 4550 50 0001 C CNN "MPN"
 F 5 "Yageo" H 3550 4550 50 0001 C CNN "Manufacturer"
-F 6 "RC0805FR-071ML" H 3650 4450 60 0001 C CNN "Mfg_Part_No"
 	1    3650 4450
 	1    0    0    -1
@@
 F 4 "B59807A0090A062" H 3410 4260 50 0001 C CNN "MPN"
 F 5 "EPCOS" H 3410 4260 50 0001 C CNN "Manufacturer"
-F 6 "B59807A0090A062" H 3450 4100 60 0001 C CNN "Mfg_Part_No"
 	1    3450 4100
 	-1   0    0    1
@@
 F 4 "TBAV99,LM" H 4000 3700 50 0001 C CNN "MPN"
 F 5 "Toshiba" H 4000 3700 50 0001 C CNN "Manufacturer"
-F 6 "TBAV99,LM" H 4150 3700 60 0001 C CNN "Mfg_Part_No"
 	1    4150 3700
 	1    0    0    -1
@@
 F 4 "CC0805KKX7R9BB105" H 3750 4150 50 0001 C CNN "MPN"
 F 5 "Yageo" H 3750 4150 50 0001 C CNN "Manufacturer"
-F 6 "CC0805KKX7R9BB105" H 3900 4100 60 0001 C CNN "Mfg_Part_No"
 	1    3900 4100
 	0    -1   -1   0
@@
 F 4 "ED08DT" H 5900 4600 50 0001 C CNN "MPN"
 F 5 "On Shore Technology" H 5900 4600 50 0001 C CNN "Manufacturer"
-F 6 "ED08DT" H 5900 4150 60 0001 C CNN "Mfg_Part_No"
 	1    5900 4150
 	1    0    0    -1
@@
 F 4 "RC0805FR-07100KL" H 5030 4450 50 0001 C CNN "MPN"
 F 5 "Yageo" H 5030 4450 50 0001 C CNN "Manufacturer"
-F 6 "RC0805FR-07100KL" H 4950 4350 60 0001 C CNN "Mfg_Part_No"
 	1    4950 4350
 	-1   0    0    1
@@
 F 4 "RC0805FR-075K1L" H 5480 3350 50 0001 C CNN "MPN"
 F 5 "Yageo" H 5480 3350 50 0001 C CNN "Manufacturer"
-F 6 "RC0805FR-075K1L" H 5400 3250 60 0001 C CNN "Mfg_Part_No"
 	1    5400 3250
 	0    1    1    0
@@
 F 4 "CC0805KKX7R9BB105" H 6050 3300 50 0001 C CNN "MPN"
 F 5 "Yageo" H 6050 3300 50 0001 C CNN "Manufacturer"
-F 6 "CC0805KKX7R9BB105" H 6200 3250 60 0001 C CNN "Mfg_Part_No"
 	1    6200 3250
 	0    -1   -1   0
@@
 F 4 "RC0805FR-071ML" H 6650 3500 50 0001 C CNN "MPN"
 F 5 "Yageo" H 6650 3500 50 0001 C CNN "Manufacturer"
-F 6 "RC0805FR-071ML" H 6500 3400 60 0001 C CNN "Mfg_Part_No"
 	1    6500 3400
 	1    0    0    -1
