File: output-select.sch (KiCad schematic (older format))
At the start: 7 parts, among them U5 DPST (2 Form A), 350V, U9 74AHC1G32

Commit message: Improve layout/stability of boost converter, etc.
* improve layout/stability of boost converter
* enable on board calibration without HVOE
* add decoupling cap to 0.6V reference
* fix footprint for U10
* add programming wire
Parts:
- R11, R12: value 200 -> 150; Mfg_Part_No RC0805FR-07200RL -> RC0805FR-07150RL
Changed lines of the file:
@@
 LIBS:valves
 LIBS:wheelerlab
+LIBS:dropbot_control_board-cache
 EELAYER 25 0
 EELAYER END
@@
 Sheet 7 7
 Title "DropBot control board"
-Date "2017-05-17"
-Rev "3.5"
+Date "2017-06-19"
+Rev "3.6"
 Comp "Sci-Bots Inc."
 Comment1 ""
@@
 P 4750 4050
 F 0 "R12" V 4830 4050 50  0000 C CNN
-F 1 "200" V 4750 4050 50  0000 C CNN
+F 1 "150" V 4750 4050 50  0000 C CNN
 F 2 "Resistors_SMD:R_0805" V 4680 4050 30  0001 C CNN
 F 3 "" H 4750 4050 30  0000 C CNN
-F 4 "RC0805FR-07200RL" H 4750 4050 60  0001 C CNN "Mfg_Part_No"
+F 4 "RC0805FR-07150RL" H 4750 4050 60  0001 C CNN "Mfg_Part_No"
 	1    4750 4050
 	0    -1   -1   0
@@
 P 4850 4550
 F 0 "R11" V 4930 4550 50  0000 C CNN
-F 1 "200" V 4850 4550 50  0000 C CNN
+F 1 "150" V 4850 4550 50  0000 C CNN
 F 2 "Resistors_SMD:R_0805" V 4780 4550 30  0001 C CNN
 F 3 "" H 4850 4550 30  0000 C CNN
-F 4 "RC0805FR-07200RL" H 4850 4550 60  0001 C CNN "Mfg_Part_No"
+F 4 "RC0805FR-07150RL" H 4850 4550 60  0001 C CNN "Mfg_Part_No"
 	1    4850 4550
 	0    -1   -1   0

Commit message: Change EEPROM and swap 150 Ohm resisotors for 100...
Change EEPROM and swap 150 Ohm resisotors for 100 resistors
driving the PhotoMOS switches.
Parts:
- R11, R12: value 150 -> 100; Mfg_Part_No RC0805FR-07150RL -> RC0805FR-07100RL
Changed lines of the file:
@@
 P 4750 4050
 F 0 "R12" V 4830 4050 50  0000 C CNN
-F 1 "150" V 4750 4050 50  0000 C CNN
+F 1 "100" V 4750 4050 50  0000 C CNN
 F 2 "Resistors_SMD:R_0805" V 4680 4050 30  0001 C CNN
 F 3 "" H 4750 4050 30  0000 C CNN
-F 4 "RC0805FR-07150RL" H 4750 4050 60  0001 C CNN "Mfg_Part_No"
+F 4 "RC0805FR-07100RL" H 4750 4050 60  0001 C CNN "Mfg_Part_No"
 	1    4750 4050
 	0    -1   -1   0
@@
 P 4850 4550
 F 0 "R11" V 4930 4550 50  0000 C CNN
-F 1 "150" V 4850 4550 50  0000 C CNN
+F 1 "100" V 4850 4550 50  0000 C CNN
 F 2 "Resistors_SMD:R_0805" V 4780 4550 30  0001 C CNN
 F 3 "" H 4850 4550 30  0000 C CNN
-F 4 "RC0805FR-07150RL" H 4850 4550 60  0001 C CNN "Mfg_Part_No"
+F 4 "RC0805FR-07100RL" H 4850 4550 60  0001 C CNN "Mfg_Part_No"
 	1    4850 4550
 	0    -1   -1   0

Commit message: Update schematic to use power ports
Connections:
- wire segments 13 -> 12
Changed lines of the file:
@@
 	-1   0    0    1
 $EndComp
-Text GLabel 5800 4950 2    60   Input ~ 0
-+3.3V
 $Comp
 L AQW216 U5
@@
 	0    -1   -1   0
 $EndComp
-Text GLabel 4700 4550 0    60   Input ~ 0
-GND
 Text Notes 4200 3150 0    60   ~ 0
 OUTPUT SELECT
 Text GLabel 5800 4650 2    60   Input ~ 0
 A0/SHORT_CHK
-Text GLabel 4550 4050 0    60   Input ~ 0
-+3.3V
 Text GLabel 5800 4050 2    60   Input ~ 0
 HVAC
@@
 Text Notes 4250 3900 0    60   ~ 0
 Both inputs must be\nlow to select HV output
-Text GLabel 5650 3100 2    60   Input ~ 0
-+3.3V
-Text GLabel 5600 3800 0    60   Input ~ 0
-GND
 $Comp
 L R R36
@@
 	5650 3100 5650 3300
 Wire Wire Line
-	5600 3800 5650 3800
-Wire Wire Line
-	5650 3800 5650 3700
-Wire Wire Line
-	4550 4050 4600 4050
+	4100 4050 4600 4050
 Wire Wire Line
 	4900 4050 5000 4050
@@
 Text Notes 6250 4850 0    60   ~ 0
 Short circuit check
+$Comp
+L +3.3V #PWR044
+U 1 1 5B3C0E4E
+P 5650 3100
+F 0 "#PWR044" H 5650 2950 50  0001 C CNN
+F 1 "+3.3V" H 5650 3240 50  0000 C CNN
+F 2 "" H 5650 3100 50  0001 C CNN
+F 3 "" H 5650 3100 50  0001 C CNN
+	1    5650 3100
+	1    0    0    -1
+$EndComp
+$Comp
+L +3.3V #PWR045
+U 1 1 5B3C0EEC
+P 4100 4050
+F 0 "#PWR045" H 4100 3900 50  0001 C CNN
+F 1 "+3.3V" H 4100 4190 50  0000 C CNN
+F 2 "" H 4100 4050 50  0001 C CNN
+F 3 "" H 4100 4050 50  0001 C CNN
+	1    4100 4050
+	1    0    0    -1
+$EndComp
+Connection ~ 4550 4050
+$Comp
+L +3.3V #PWR046
+U 1 1 5B3C10F0
+P 5800 4950
+F 0 "#PWR046" H 5800 4800 50  0001 C CNN
+F 1 "+3.3V" H 5800 5090 50  0000 C CNN
+F 2 "" H 5800 4950 50  0001 C CNN
+F 3 "" H 5800 4950 50  0001 C CNN
+	1    5800 4950
+	-1   0    0    1
+$EndComp
+$Comp
+L GND #PWR047
+U 1 1 5B3CAC28
+P 4400 4550
+F 0 "#PWR047" H 4400 4300 50  0001 C CNN
+F 1 "GND" H 4400 4400 50  0000 C CNN
+F 2 "" H 4400 4550 50  0001 C CNN
+F 3 "" H 4400 4550 50  0001 C CNN
+	1    4400 4550
+	1    0    0    -1
+$EndComp
+Wire Wire Line
+	4700 4550 4400 4550
+$Comp
+L GND #PWR048
+U 1 1 5B3CAFE2
+P 5650 3700
+F 0 "#PWR048" H 5650 3450 50  0001 C CNN
+F 1 "GND" H 5650 3550 50  0000 C CNN
+F 2 "" H 5650 3700 50  0001 C CNN
+F 3 "" H 5650 3700 50  0001 C CNN
+	1    5650 3700
+	1    0    0    -1
+$EndComp
 $EndSCHEMATC

Commit message: Update with kicad-helpers files
Parts:
- R10, R11, R12, R17, R36: symbol R -> Device:R
Changed lines of the file:
@@
-EESchema Schematic File Version 2
-LIBS:power
-LIBS:device
-LIBS:transistors
-LIBS:conn
-LIBS:linear
-LIBS:regul
-LIBS:74xx
-LIBS:cmos4000
-LIBS:adc-dac
-LIBS:memory
-LIBS:xilinx
-LIBS:microcontrollers
-LIBS:dsp
-LIBS:microchip
-LIBS:analog_switches
-LIBS:motorola
-LIBS:texas
-LIBS:intel
-LIBS:audio
-LIBS:interface
-LIBS:digital-audio
-LIBS:philips
-LIBS:display
-LIBS:cypress
-LIBS:siliconi
-LIBS:opto
-LIBS:atmel
-LIBS:contrib
-LIBS:valves
-LIBS:sci-bots
-LIBS:dropbot_control_board-cache
-EELAYER 25 0
+EESchema Schematic File Version 4
+EELAYER 30 0
 EELAYER END
 $Descr USLetter 11000 8500
@@
 $EndDescr
 $Comp
-L R R17
+L Device:R R17
 U 1 1 56C16200
 P 5800 4800
@@
 D8/OUTPUT_SELECT
 $Comp
-L R R10
+L Device:R R10
 U 1 1 56BF2A44
 P 4550 4200
@@
 $EndComp
 $Comp
-L R R12
+L Device:R R12
 U 1 1 56BF2F38
 P 4750 4050
@@
 $EndComp
 $Comp
-L R R11
+L Device:R R11
 U 1 1 56BF3094
 P 4850 4550
@@
 Both inputs must be\nlow to select HV output
 $Comp
-L R R36
+L Device:R R36
 U 1 1 58577F50
 P 5250 3250
@@
 Short circuit check
 $Comp
-L +3.3V #PWR044
+L power:+3.3V #PWR044
 U 1 1 5B3C0E4E
 P 5650 3100
@@
 $EndComp
 $Comp
-L +3.3V #PWR045
+L power:+3.3V #PWR045
 U 1 1 5B3C0EEC
 P 4100 4050
@@
 Connection ~ 4550 4050
 $Comp
-L +3.3V #PWR046
+L power:+3.3V #PWR046
 U 1 1 5B3C10F0
 P 5800 4950
@@
 $EndComp
 $Comp
-L GND #PWR047
+L power:GND #PWR047
 U 1 1 5B3CAC28
 P 4400 4550
@@
 	4700 4550 4400 4550
 $Comp
-L GND #PWR048
+L power:GND #PWR048
 U 1 1 5B3CAFE2
 P 5650 3700

Commit message: Fix broken symbols and DRC tests
Parts:
- U5: symbol AQW216 -> sci-bots:AQW214
- U9: symbol 74AHC1G32 -> sci-bots:74AHC1G32
Connections:
- wire segments 12 -> 15
Changed lines of the file:
@@
 $EndComp
 $Comp
-L AQW216 U5
+L sci-bots:AQW214 U5
 U 1 1 56C16511
 P 5400 4300
@@
 HV_OE
 $Comp
-L 74AHC1G32 U9
+L sci-bots:74AHC1G32 U9
 U 1 1 58517C1B
 P 5850 3500
@@
 	5650 3100 5650 3300
 Wire Wire Line
-	4100 4050 4600 4050
+	4100 4050 4550 4050
 Wire Wire Line
 	4900 4050 5000 4050
 Wire Wire Line
-	4550 4350 5000 4350
+	4550 4350 4950 4350
 Wire Wire Line
-	4950 3950 4950 4350
+	4950 3950 4950 4250
 Connection ~ 4950 4350
 Wire Wire Line
@@
 	1    0    0    -1
 $EndComp
+Wire Wire Line
+	4950 4350 5000 4350
+Wire Wire Line
+	4950 4250 4950 4350
+Wire Wire Line
+	4550 4050 4600 4050
 $EndSCHEMATC
