File: output-select.sch (KiCad schematic (older format))
At the start: 7 parts, among them U5 DPST (2 Form A), 350V, U9 74AHC1G32

Commit message: Update BOM
Parts:
- R10, R36: MPN (none) -> RC0805FR-075K1L; Manufacturer (none) -> Yageo
- R11, R12: MPN (none) -> RC0805FR-07100RL; Manufacturer (none) -> Yageo
- R17: MPN (none) -> RC0805FR-0751KL; Manufacturer (none) -> Yageo
- U5: MPN (none) -> TLP227G-2(TP1,N,F); Manufacturer (none) -> Toshiba
- U9: MPN (none) -> 74AHC1G32GW,125; Manufacturer (none) -> Nexperia
Changed lines of the file:
@@
 U 1 1 56C16200
 P 5800 4800
-F 0 "R17" V 5880 4800 50  0000 C CNN
-F 1 "51k" V 5800 4800 50  0000 C CNN
-F 2 "Resistors_SMD:R_0805" V 5730 4800 30  0001 C CNN
-F 3 "" H 5800 4800 30  0000 C CNN
-F 4 "RC0805FR-0751KL" H 5800 4800 60  0001 C CNN "Mfg_Part_No"
+F 0 "R17" V 5880 4800 50 0000 C CNN
+F 1 "51k" V 5800 4800 50 0000 C CNN
+F 2 "Resistors_SMD:R_0805" V 5730 4800 30 0001 C CNN
+F 3 "" H 5800 4800 30 0000 C CNN
+F 4 "RC0805FR-0751KL" H 5880 4900 50 0001 C CNN "MPN"
+F 5 "Yageo" H 5880 4900 50 0001 C CNN "Manufacturer"
+F 6 "RC0805FR-0751KL" H 5800 4800 60 0001 C CNN "Mfg_Part_No"
 	1    5800 4800
 	-1   0    0    1
@@
 U 1 1 56C16511
 P 5400 4300
-F 0 "U5" H 5400 4550 60  0000 C CNN
-F 1 "DPST (2 Form A), 350V" H 5050 3900 60  0000 C CNN
-F 2 "SMD_Packages:DIP-8_SMD" H 5400 4300 60  0001 C CNN
-F 3 "" H 5400 4300 60  0000 C CNN
-F 4 "TLP227G-2(TP1,N,F)" H 5400 4300 60  0001 C CNN "Mfg_Part_No"
+F 0 "U5" H 5400 4550 60 0000 C CNN
+F 1 "DPST (2 Form A), 350V" H 5050 3900 60 0000 C CNN
+F 2 "SMD_Packages:DIP-8_SMD" H 5400 4300 60 0001 C CNN
+F 3 "" H 5400 4300 60 0000 C CNN
+F 4 "TLP227G-2(TP1,N,F)" H 5400 4650 50 0001 C CNN "MPN"
+F 5 "Toshiba" H 5400 4650 50 0001 C CNN "Manufacturer"
+F 6 "TLP227G-2(TP1,N,F)" H 5400 4300 60 0001 C CNN "Mfg_Part_No"
 	1    5400 4300
+	1    0    0    -1
+$EndComp
+$Comp
+L Device:R R10
+U 1 1 56BF2A44
+P 4550 4200
+F 0 "R10" V 4630 4200 50 0000 C CNN
+F 1 "5.1k" V 4550 4200 50 0000 C CNN
+F 2 "Resistors_SMD:R_0805" V 4480 4200 30 0001 C CNN
+F 3 "" H 4550 4200 30 0000 C CNN
+F 4 "RC0805FR-075K1L" H 4630 4300 50 0001 C CNN "MPN"
+F 5 "Yageo" H 4630 4300 50 0001 C CNN "Manufacturer"
+F 6 "RC0805FR-075K1L" H 4550 4200 60 0001 C CNN "Mfg_Part_No"
+	1    4550 4200
+	1    0    0    -1
+$EndComp
+$Comp
+L Device:R R12
+U 1 1 56BF2F38
+P 4750 4050
+F 0 "R12" V 4830 4050 50 0000 C CNN
+F 1 "100" V 4750 4050 50 0000 C CNN
+F 2 "Resistors_SMD:R_0805" V 4680 4050 30 0001 C CNN
+F 3 "" H 4750 4050 30 0000 C CNN
+F 4 "RC0805FR-07100RL" H 4830 4150 50 0001 C CNN "MPN"
+F 5 "Yageo" H 4830 4150 50 0001 C CNN "Manufacturer"
+F 6 "RC0805FR-07100RL" H 4750 4050 60 0001 C CNN "Mfg_Part_No"
+	1    4750 4050
+	0    -1   -1   0
+$EndComp
+$Comp
+L Device:R R11
+U 1 1 56BF3094
+P 4850 4550
+F 0 "R11" V 4930 4550 50 0000 C CNN
+F 1 "100" V 4850 4550 50 0000 C CNN
+F 2 "Resistors_SMD:R_0805" V 4780 4550 30 0001 C CNN
+F 3 "" H 4850 4550 30 0000 C CNN
+F 4 "RC0805FR-07100RL" H 4930 4650 50 0001 C CNN "MPN"
+F 5 "Yageo" H 4930 4650 50 0001 C CNN "Manufacturer"
+F 6 "RC0805FR-07100RL" H 4850 4550 60 0001 C CNN "Mfg_Part_No"
+	1    4850 4550
+	0    -1   -1   0
+$EndComp
+$Comp
+L sci-bots:74AHC1G32 U9
+U 1 1 58517C1B
+P 5850 3500
+F 0 "U9" H 5850 3550 50 0000 C CNN
+F 1 "74AHC1G32" H 5890 3475 50 0000 C CNN
+F 2 "TO_SOT_Packages_SMD:SOT-353" H 5850 3500 50 0001 C CNN
+F 3 "http://www.nxp.com/documents/data_sheet/74AHC_AHCT1G32.pdf" H 5850 3500 50 0001 C CNN
+F 4 "74AHC1G32GW,125" H 5850 3650 50 0001 C CNN "MPN"
+F 5 "Nexperia" H 5850 3650 50 0001 C CNN "Manufacturer"
+F 6 "74AHC1G32GW,125" H 5850 3500 60 0001 C CNN "Mfg_Part_No"
+	1    5850 3500
+	1    0    0    -1
+$EndComp
+$Comp
+L Device:R R36
+U 1 1 58577F50
+P 5250 3250
+F 0 "R36" V 5330 3250 50 0000 C CNN
+F 1 "5.1k" V 5250 3250 50 0000 C CNN
+F 2 "Resistors_SMD:R_0805" V 5180 3250 30 0001 C CNN
+F 3 "" H 5250 3250 30 0000 C CNN
+F 4 "RC0805FR-075K1L" H 5330 3350 50 0001 C CNN "MPN"
+F 5 "Yageo" H 5330 3350 50 0001 C CNN "Manufacturer"
+F 6 "RC0805FR-075K1L" H 5250 3250 60 0001 C CNN "Mfg_Part_No"
+	1    5250 3250
+	-1   0    0    1
+$EndComp
+$Comp
+L power:+3.3V #PWR044
+U 1 1 5B3C0E4E
+P 5650 3100
+F 0 "#PWR044" H 5650 2950 50 0001 C CNN
+F 1 "+3.3V" H 5650 3240 50 0000 C CNN
+F 2 "" H 5650 3100 50 0001 C CNN
+F 3 "" H 5650 3100 50 0001 C CNN
+	1    5650 3100
+	1    0    0    -1
+$EndComp
+$Comp
+L power:+3.3V #PWR045
+U 1 1 5B3C0EEC
+P 4100 4050
+F 0 "#PWR045" H 4100 3900 50 0001 C CNN
+F 1 "+3.3V" H 4100 4190 50 0000 C CNN
+F 2 "" H 4100 4050 50 0001 C CNN
+F 3 "" H 4100 4050 50 0001 C CNN
+	1    4100 4050
+	1    0    0    -1
+$EndComp
+$Comp
+L power:+3.3V #PWR046
+U 1 1 5B3C10F0
+P 5800 4950
+F 0 "#PWR046" H 5800 4800 50 0001 C CNN
+F 1 "+3.3V" H 5800 5090 50 0000 C CNN
+F 2 "" H 5800 4950 50 0001 C CNN
+F 3 "" H 5800 4950 50 0001 C CNN
+	1    5800 4950
+	-1   0    0    1
+$EndComp
+$Comp
+L power:GND #PWR047
+U 1 1 5B3CAC28
+P 4400 4550
+F 0 "#PWR047" H 4400 4300 50 0001 C CNN
+F 1 "GND" H 4400 4400 50 0000 C CNN
+F 2 "" H 4400 4550 50 0001 C CNN
+F 3 "" H 4400 4550 50 0001 C CNN
+	1    4400 4550
+	1    0    0    -1
+$EndComp
+$Comp
+L power:GND #PWR048
+U 1 1 5B3CAFE2
+P 5650 3700
+F 0 "#PWR048" H 5650 3450 50 0001 C CNN
+F 1 "GND" H 5650 3550 50 0000 C CNN
+F 2 "" H 5650 3700 50 0001 C CNN
+F 3 "" H 5650 3700 50 0001 C CNN
+	1    5650 3700
 	1    0    0    -1
 $EndComp
@@
 Text GLabel 5250 3600 0    60   Input ~ 0
 D8/OUTPUT_SELECT
-$Comp
-L Device:R R10
-U 1 1 56BF2A44
-P 4550 4200
-F 0 "R10" V 4630 4200 50  0000 C CNN
-F 1 "5.1k" V 4550 4200 50  0000 C CNN
-F 2 "Resistors_SMD:R_0805" V 4480 4200 30  0001 C CNN
-F 3 "" H 4550 4200 30  0000 C CNN
-F 4 "RC0805FR-075K1L" H 4550 4200 60  0001 C CNN "Mfg_Part_No"
-	1    4550 4200
-	1    0    0    -1
-$EndComp
-$Comp
-L Device:R R12
-U 1 1 56BF2F38
-P 4750 4050
-F 0 "R12" V 4830 4050 50  0000 C CNN
-F 1 "100" V 4750 4050 50  0000 C CNN
-F 2 "Resistors_SMD:R_0805" V 4680 4050 30  0001 C CNN
-F 3 "" H 4750 4050 30  0000 C CNN
-F 4 "RC0805FR-07100RL" H 4750 4050 60  0001 C CNN "Mfg_Part_No"
-	1    4750 4050
-	0    -1   -1   0
-$EndComp
-$Comp
-L Device:R R11
-U 1 1 56BF3094
-P 4850 4550
-F 0 "R11" V 4930 4550 50  0000 C CNN
-F 1 "100" V 4850 4550 50  0000 C CNN
-F 2 "Resistors_SMD:R_0805" V 4780 4550 30  0001 C CNN
-F 3 "" H 4850 4550 30  0000 C CNN
-F 4 "RC0805FR-07100RL" H 4850 4550 60  0001 C CNN "Mfg_Part_No"
-	1    4850 4550
-	0    -1   -1   0
-$EndComp
 Text Notes 4200 3150 0    60   ~ 0
 OUTPUT SELECT
@@
 Text GLabel 5250 3400 0    60   Input ~ 0
 HV_OE
-$Comp
-L sci-bots:74AHC1G32 U9
-U 1 1 58517C1B
-P 5850 3500
-F 0 "U9" H 5850 3550 50  0000 C CNN
-F 1 "74AHC1G32" H 5890 3475 50  0000 C CNN
-F 2 "TO_SOT_Packages_SMD:SOT-353" H 5850 3500 50  0001 C CNN
-F 3 "http://www.nxp.com/documents/data_sheet/74AHC_AHCT1G32.pdf" H 5850 3500 50  0001 C CNN
-F 4 "74AHC1G32GW,125" H 5850 3500 60  0001 C CNN "Mfg_Part_No"
-	1    5850 3500
-	1    0    0    -1
-$EndComp
 Text Notes 4250 3900 0    60   ~ 0
 Both inputs must be\nlow to select HV output
-$Comp
-L Device:R R36
-U 1 1 58577F50
-P 5250 3250
-F 0 "R36" V 5330 3250 50  0000 C CNN
-F 1 "5.1k" V 5250 3250 50  0000 C CNN
-F 2 "Resistors_SMD:R_0805" V 5180 3250 30  0001 C CNN
-F 3 "" H 5250 3250 30  0000 C CNN
-F 4 "RC0805FR-075K1L" H 5250 3250 60  0001 C CNN "Mfg_Part_No"
-	1    5250 3250
-	-1   0    0    1
-$EndComp
-Wire Wire Line
-	5800 4550 5800 4650
-Wire Wire Line
-	4950 3950 6450 3950
-Wire Wire Line
-	5650 3100 5650 3300
-Wire Wire Line
-	4100 4050 4550 4050
-Wire Wire Line
-	4900 4050 5000 4050
-Wire Wire Line
-	4550 4350 4950 4350
-Wire Wire Line
-	4950 3950 4950 4250
-Connection ~ 4950 4350
-Wire Wire Line
-	5800 4350 5800 4250
-Wire Wire Line
-	6450 3950 6450 3500
-Wire Wire Line
-	5250 3100 5650 3100
-Wire Wire Line
-	5000 4250 4950 4250
-Connection ~ 4950 4250
 Text Notes 6250 4850 0    60   ~ 0
 Short circuit check
-$Comp
-L power:+3.3V #PWR044
-U 1 1 5B3C0E4E
-P 5650 3100
-F 0 "#PWR044" H 5650 2950 50  0001 C CNN
-F 1 "+3.3V" H 5650 3240 50  0000 C CNN
-F 2 "" H 5650 3100 50  0001 C CNN
-F 3 "" H 5650 3100 50  0001 C CNN
-	1    5650 3100
-	1    0    0    -1
-$EndComp
-$Comp
-L power:+3.3V #PWR045
-U 1 1 5B3C0EEC
-P 4100 4050
-F 0 "#PWR045" H 4100 3900 50  0001 C CNN
-F 1 "+3.3V" H 4100 4190 50  0000 C CNN
-F 2 "" H 4100 4050 50  0001 C CNN
-F 3 "" H 4100 4050 50  0001 C CNN
-	1    4100 4050
-	1    0    0    -1
-$EndComp
+Wire Wire Line
+	5800 4550 5800 4650
+Wire Wire Line
+	4950 3950 6450 3950
+Wire Wire Line
+	5650 3100 5650 3300
+Wire Wire Line
+	4100 4050 4550 4050
+Wire Wire Line
+	4900 4050 5000 4050
+Wire Wire Line
+	4550 4350 4950 4350
+Wire Wire Line
+	4950 3950 4950 4250
+Wire Wire Line
+	5800 4350 5800 4250
+Wire Wire Line
+	6450 3950 6450 3500
+Wire Wire Line
+	5250 3100 5650 3100
+Wire Wire Line
+	5000 4250 4950 4250
+Wire Wire Line
+	4700 4550 4400 4550
+Wire Wire Line
+	4950 4350 5000 4350
+Wire Wire Line
+	4950 4250 4950 4350
+Wire Wire Line
+	4550 4050 4600 4050
+Connection ~ 4950 4350
+Connection ~ 4950 4250
 Connection ~ 4550 4050
-$Comp
-L power:+3.3V #PWR046
-U 1 1 5B3C10F0
-P 5800 4950
-F 0 "#PWR046" H 5800 4800 50  0001 C CNN
-F 1 "+3.3V" H 5800 5090 50  0000 C CNN
-F 2 "" H 5800 4950 50  0001 C CNN
-F 3 "" H 5800 4950 50  0001 C CNN
-	1    5800 4950
-	-1   0    0    1
-$EndComp
-$Comp
-L power:GND #PWR047
-U 1 1 5B3CAC28
-P 4400 4550
-F 0 "#PWR047" H 4400 4300 50  0001 C CNN
-F 1 "GND" H 4400 4400 50  0000 C CNN
-F 2 "" H 4400 4550 50  0001 C CNN
-F 3 "" H 4400 4550 50  0001 C CNN
-	1    4400 4550
-	1    0    0    -1
-$EndComp
-Wire Wire Line
-	4700 4550 4400 4550
-$Comp
-L power:GND #PWR048
-U 1 1 5B3CAFE2
-P 5650 3700
-F 0 "#PWR048" H 5650 3450 50  0001 C CNN
-F 1 "GND" H 5650 3550 50  0000 C CNN
-F 2 "" H 5650 3700 50  0001 C CNN
-F 3 "" H 5650 3700 50  0001 C CNN
-	1    5650 3700
-	1    0    0    -1
-$EndComp
-Wire Wire Line
-	4950 4350 5000 4350
-Wire Wire Line
-	4950 4250 4950 4350
-Wire Wire Line
-	4550 4050 4600 4050
 $EndSCHEMATC

Commit message: Remove "Mfg_Part_No" field (replaced by  "MPN")
Parts:
- R10, R36: Mfg_Part_No RC0805FR-075K1L -> (none)
- R11, R12: Mfg_Part_No RC0805FR-07100RL -> (none)
- R17: Mfg_Part_No RC0805FR-0751KL -> (none)
- U5: Mfg_Part_No TLP227G-2(TP1,N,F) -> (none)
- U9: Mfg_Part_No 74AHC1G32GW,125 -> (none)
Changed lines of the file:
@@
 F 4 "RC0805FR-0751KL" H 5880 4900 50 0001 C CNN "MPN"
 F 5 "Yageo" H 5880 4900 50 0001 C CNN "Manufacturer"
-F 6 "RC0805FR-0751KL" H 5800 4800 60 0001 C CNN "Mfg_Part_No"
 	1    5800 4800
 	-1   0    0    1
@@
 F 4 "TLP227G-2(TP1,N,F)" H 5400 4650 50 0001 C CNN "MPN"
 F 5 "Toshiba" H 5400 4650 50 0001 C CNN "Manufacturer"
-F 6 "TLP227G-2(TP1,N,F)" H 5400 4300 60 0001 C CNN "Mfg_Part_No"
 	1    5400 4300
 	1    0    0    -1
@@
 F 4 "RC0805FR-075K1L" H 4630 4300 50 0001 C CNN "MPN"
 F 5 "Yageo" H 4630 4300 50 0001 C CNN "Manufacturer"
-F 6 "RC0805FR-075K1L" H 4550 4200 60 0001 C CNN "Mfg_Part_No"
 	1    4550 4200
 	1    0    0    -1
@@
 F 4 "RC0805FR-07100RL" H 4830 4150 50 0001 C CNN "MPN"
 F 5 "Yageo" H 4830 4150 50 0001 C CNN "Manufacturer"
-F 6 "RC0805FR-07100RL" H 4750 4050 60 0001 C CNN "Mfg_Part_No"
 	1    4750 4050
 	0    -1   -1   0
@@
 F 4 "RC0805FR-07100RL" H 4930 4650 50 0001 C CNN "MPN"
 F 5 "Yageo" H 4930 4650 50 0001 C CNN "Manufacturer"
-F 6 "RC0805FR-07100RL" H 4850 4550 60 0001 C CNN "Mfg_Part_No"
 	1    4850 4550
 	0    -1   -1   0
@@
 F 4 "74AHC1G32GW,125" H 5850 3650 50 0001 C CNN "MPN"
 F 5 "Nexperia" H 5850 3650 50 0001 C CNN "Manufacturer"
-F 6 "74AHC1G32GW,125" H 5850 3500 60 0001 C CNN "Mfg_Part_No"
 	1    5850 3500
 	1    0    0    -1
@@
 F 4 "RC0805FR-075K1L" H 5330 3350 50 0001 C CNN "MPN"
 F 5 "Yageo" H 5330 3350 50 0001 C CNN "Manufacturer"
-F 6 "RC0805FR-075K1L" H 5250 3250 60 0001 C CNN "Mfg_Part_No"
 	1    5250 3250
 	-1   0    0    1
